File: Old2/Krokovka2.sch (KiCad schematic (older format))
At the start: 9 parts, among them J10 Conn_01x01_Female, J12 Conn_01x02_Female, J13 Conn_01x08_Female, J14 Conn_01x04_Male, J8 Conn_01x08_Female

Commit message: Verze 0.2, Indexy
Parts:
- added J11: Conn_01x02_Female, symbol Connector:Conn_01x02_Female
- added J9: Conn_01x01_Female, symbol Connector:Conn_01x01_Female
Connections:
- net labels added: M1A, M1B, M2A, M2B, PDN_UART2, SPREAD, VIO
- net labels removed: +10V, +3V3, A1, A2, B1, B2, CLK, INDEX_2, VDD
- wire segments 33 -> 32
Changed lines of the file:
@@
 MS2
 Text Label 1350 4300 0    50   ~ 0
-PDN_UART
+SPREAD
 Text Label 1350 4400 0    50   ~ 0
 PDN_UART
 Text Label 1350 4500 0    50   ~ 0
-CLK
+PDN_UART2
 Text Label 1350 4600 0    50   ~ 0
 STEP
@@
 AR Path="/601BF914/6020C1B3" Ref="J?"  Part="1"
 AR Path="/601E7BA1/6020C1B3" Ref="J8"  Part="1"
-F 0 "J8" V 2050 4250 50  0000 L CNN
-F 1 "Conn_01x08_Female" V 1950 3900 50  0000 L CNN
+F 0 "J8" H 1928 4276 50  0000 L CNN
+F 1 "Conn_01x08_Female" H 1928 4185 50  0000 L CNN
 F 2 "" H 1900 4300 50  0001 C CNN
 F 3 "~" H 1900 4300 50  0001 C CNN
@@
 AR Path="/601BF914/6020C1C0" Ref="J?"  Part="1"
 AR Path="/601E7BA1/6020C1C0" Ref="J13"  Part="1"
-F 0 "J13" V 2450 4300 50  0000 C CNN
-F 1 "Conn_01x08_Female" V 2350 4250 50  0000 C CNN
+F 0 "J13" H 2192 4785 50  0000 C CNN
+F 1 "Conn_01x08_Female" H 2192 4694 50  0000 C CNN
 F 2 "" H 2300 4300 50  0001 C CNN
 F 3 "~" H 2300 4300 50  0001 C CNN
@@
 GND
 Text Label 2550 4200 0    50   ~ 0
-A2
+M2B
 Text Label 2550 4300 0    50   ~ 0
-A1
+M2A
 Text Label 2550 4400 0    50   ~ 0
-B1
+M1A
 Text Label 2550 4500 0    50   ~ 0
-B2
+M1B
 Text Label 2550 4600 0    50   ~ 0
-VDD
+VIO
 Text Label 2550 4700 0    50   ~ 0
 GND
@@
 AR Path="/601BF914/6020C1CE" Ref="J?"  Part="1"
 AR Path="/601E7BA1/6020C1CE" Ref="J10"  Part="1"
-F 0 "J10" H 1750 3800 50  0000 L CNN
-F 1 "Conn_01x01_Female" H 1200 3850 50  0000 L CNN
+F 0 "J10" V 1796 3998 50  0000 L CNN
+F 1 "Conn_01x01_Female" V 1887 3998 50  0000 L CNN
 F 2 "" H 1950 3950 50  0001 C CNN
 F 3 "~" H 1950 3950 50  0001 C CNN
@@
 AR Path="/601BF914/6020C1D4" Ref="J?"  Part="1"
 AR Path="/601E7BA1/6020C1D4" Ref="J12"  Part="1"
-F 0 "J12" V 2200 3900 50  0000 L CNN
-F 1 "Conn_01x02_Female" H 1350 4000 50  0000 L CNN
+F 0 "J12" V 1996 3998 50  0000 L CNN
+F 1 "Conn_01x02_Female" V 2087 3998 50  0000 L CNN
 F 2 "" H 2150 3950 50  0001 C CNN
 F 3 "~" H 2150 3950 50  0001 C CNN
@@
 Text HLabel 1300 4700 0    50   Input ~ 0
 DIR2
+NoConn ~ 1300 4500
 $Comp
 L power:GND #PWR?
@@
 	1    2950 4100
 	0    -1   -1   0
+$EndComp
+$Comp
+L Connector:Conn_01x01_Female J?
+U 1 1 6020C245
+P 1950 3050
+AR Path="/601BF914/6020C245" Ref="J?"  Part="1"
+AR Path="/601E7BA1/6020C245" Ref="J9"  Part="1"
+F 0 "J9" V 1888 2962 50  0000 R CNN
+F 1 "Conn_01x01_Female" V 1797 2962 50  0000 R CNN
+F 2 "" H 1950 3050 50  0001 C CNN
+F 3 "~" H 1950 3050 50  0001 C CNN
+	1    1950 3050
+	0    -1   -1   0
+$EndComp
+$Comp
+L Connector:Conn_01x02_Female J?
+U 1 1 6020C24B
+P 2050 3050
+AR Path="/601BF914/6020C24B" Ref="J?"  Part="1"
+AR Path="/601E7BA1/6020C24B" Ref="J11"  Part="1"
+F 0 "J11" V 1988 2862 50  0000 R CNN
+F 1 "Conn_01x02_Female" V 1897 2862 50  0000 R CNN
+F 2 "" H 2050 3050 50  0001 C CNN
+F 3 "~" H 2050 3050 50  0001 C CNN
+	1    2050 3050
+	0    -1   -1   0
+$EndComp
+NoConn ~ 2950 4600
+NoConn ~ 1300 4300
+$Comp
+L power:VCC #PWR?
+U 1 1 60243DD1
+P 2650 4000
+AR Path="/601BF914/60243DD1" Ref="#PWR?"  Part="1"
+AR Path="/601E7BA1/60243DD1" Ref="#PWR0103"  Part="1"
+F 0 "#PWR0103" H 2650 3850 50  0001 C CNN
+F 1 "VCC" V 2665 4127 50  0000 L CNN
+F 2 "" H 2650 4000 50  0001 C CNN
+F 3 "" H 2650 4000 50  0001 C CNN
+	1    2650 4000
+	0    1    1    0
 $EndComp
 Wire Wire Line
@@
 	0    1    1    0
 $EndComp
-$Comp
-L power:+10V #PWR?
-U 1 1 601A68DF
-P 2650 4000
-F 0 "#PWR?" H 2650 3850 50  0001 C CNN
-F 1 "+10V" V 2665 4128 50  0000 L CNN
-F 2 "" H 2650 4000 50  0001 C CNN
-F 3 "" H 2650 4000 50  0001 C CNN
-	1    2650 4000
-	0    1    1    0
-$EndComp
-$Comp
-L power:+3V3 #PWR?
-U 1 1 601A7076
-P 2950 4600
-F 0 "#PWR?" H 2950 4450 50  0001 C CNN
-F 1 "+3V3" V 2965 4728 50  0000 L CNN
-F 2 "" H 2950 4600 50  0001 C CNN
-F 3 "" H 2950 4600 50  0001 C CNN
-	1    2950 4600
-	0    1    1    0
-$EndComp
-NoConn ~ 1300 4500
-Wire Wire Line
-	1300 4300 1300 4400
-Text HLabel 2150 3250 1    50   Input ~ 0
-INDEX_2
-NoConn ~ 2050 3250
-NoConn ~ 1950 3250
 $EndSCHEMATC
