File: Old2/Napajeni.sch (KiCad schematic (older format))
At the start: 16 parts, among them Q1 BS250, Q2 NTR2101P, Q3 NTR2101P, Q4 BS250, Q5 NTR2101P, SW1 SW_MEC_5G, SW2 SW_MEC_5G

Commit message: Verze 0.2, Indexy
Connections:
- net labels added: VCC
- net labels removed: +10V, +3V3
- wire segments 42 -> 40
Changed lines of the file:
@@
 	5000 2950 5300 2950
 Wire Wire Line
-	5300 2950 5300 3550
+	5300 2950 5300 4000
 Wire Wire Line
 	5750 2950 5750 4000
@@
 	5950 2650 6300 2650
 $Comp
+L power:VCC #PWR012
+U 1 1 6019520F
+P 7950 2200
+F 0 "#PWR012" H 7950 2050 50  0001 C CNN
+F 1 "VCC" H 7965 2373 50  0000 C CNN
+F 2 "" H 7950 2200 50  0001 C CNN
+F 3 "" H 7950 2200 50  0001 C CNN
+	1    7950 2200
+	1    0    0    -1
+$EndComp
+$Comp
 L Device:R R3
 U 1 1 60196125
@@
 $EndComp
 $Comp
+L power:VCC #PWR05
+U 1 1 6019987E
+P 6150 2800
+F 0 "#PWR05" H 6150 2650 50  0001 C CNN
+F 1 "VCC" H 6165 2973 50  0000 C CNN
+F 2 "" H 6150 2800 50  0001 C CNN
+F 3 "" H 6150 2800 50  0001 C CNN
+	1    6150 2800
+	1    0    0    -1
+$EndComp
+$Comp
 L Device:Polyfuse F1
 U 1 1 6019A463
@@
 	7450 2650 7950 2650
 Wire Wire Line
-	7950 2650 7950 2250
+	7950 2650 7950 2200
 Wire Wire Line
 	6100 3200 6150 3200
@@
 $EndComp
 $Comp
+L power:VCC #PWR010
+U 1 1 601BC34A
+P 7650 2950
+F 0 "#PWR010" H 7650 2800 50  0001 C CNN
+F 1 "VCC" H 7665 3123 50  0000 C CNN
+F 2 "" H 7650 2950 50  0001 C CNN
+F 3 "" H 7650 2950 50  0001 C CNN
+	1    7650 2950
+	1    0    0    -1
+$EndComp
+$Comp
 L power:GND #PWR011
 U 1 1 601BC6CA
@@
 	7650 3550 7650 3400
 Connection ~ 7650 3550
+Wire Wire Line
+	7650 3100 7650 2950
 Text HLabel 8050 3550 2    50   Input ~ 0
 SW_OFF
 Wire Wire Line
 	8050 3550 7650 3550
-$Comp
-L power:PWR_FLAG #FLG?
-U 1 1 601A02E3
-P 7950 2250
-F 0 "#FLG?" H 7950 2325 50  0001 C CNN
-F 1 "PWR_FLAG" V 7950 2378 50  0000 L CNN
-F 2 "" H 7950 2250 50  0001 C CNN
-F 3 "~" H 7950 2250 50  0001 C CNN
-	1    7950 2250
-	0    1    1    0
-$EndComp
-Connection ~ 7950 2250
-Wire Wire Line
-	7950 2250 7950 2200
-$Comp
-L power:PWR_FLAG #FLG?
-U 1 1 601A083D
-P 5300 3550
-F 0 "#FLG?" H 5300 3625 50  0001 C CNN
-F 1 "PWR_FLAG" V 5300 3677 50  0000 L CNN
-F 2 "" H 5300 3550 50  0001 C CNN
-F 3 "~" H 5300 3550 50  0001 C CNN
-	1    5300 3550
-	0    -1   -1   0
-$EndComp
-Connection ~ 5300 3550
-Wire Wire Line
-	5300 3550 5300 4000
-$Comp
-L power:+10V #PWR?
-U 1 1 601A14D9
-P 7950 2200
-F 0 "#PWR?" H 7950 2050 50  0001 C CNN
-F 1 "+10V" H 7965 2373 50  0000 C CNN
-F 2 "" H 7950 2200 50  0001 C CNN
-F 3 "" H 7950 2200 50  0001 C CNN
-	1    7950 2200
-	1    0    0    -1
-$EndComp
-Wire Wire Line
-	7650 3100 7650 2950
-$Comp
-L power:+3V3 #PWR?
-U 1 1 601A3014
-P 7650 2950
-F 0 "#PWR?" H 7650 2800 50  0001 C CNN
-F 1 "+3V3" H 7665 3123 50  0000 C CNN
-F 2 "" H 7650 2950 50  0001 C CNN
-F 3 "" H 7650 2950 50  0001 C CNN
-	1    7650 2950
-	1    0    0    -1
-$EndComp
-$Comp
-L power:+3V3 #PWR?
-U 1 1 601A5073
-P 6150 2800
-F 0 "#PWR?" H 6150 2650 50  0001 C CNN
-F 1 "+3V3" H 6165 2973 50  0000 C CNN
-F 2 "" H 6150 2800 50  0001 C CNN
-F 3 "" H 6150 2800 50  0001 C CNN
-	1    6150 2800
-	1    0    0    -1
-$EndComp
 $EndSCHEMATC
