File: Old2/Základní deska II.sch (KiCad schematic (older format))
At the start: 2 parts, among them U1 ESP32-WROOM-32

Commit message: Verze 0.2, Indexy
Connections:
- net labels added: VCC
- net labels removed: +3V3
Changed lines of the file:
@@
 F4 "STEP1" I L 9500 2750 50
 F5 "DIR1" I L 9500 2850 50
-F6 "INDEX_1" I L 9500 2950 50
 $EndSheet
 $Sheet
@@
 F4 "STEP2" I L 9500 3950 50
 F5 "DIR2" I L 9500 4100 50
-F6 "INDEX_2" I L 9500 3850 50
 $EndSheet
 $Sheet
@@
 F4 "STEP3" I L 9500 5050 50
 F5 "DIR3" I L 9500 5200 50
-F6 "INDEX_3" I L 9500 4650 50
 $EndSheet
 $Sheet
@@
 F4 "STEP4" I L 9500 6000 50
 F5 "DIR4" I L 9500 6150 50
-F6 "INDEX_4" I L 9500 6250 50
 $EndSheet
 $Comp
@@
 	1    0    0    -1
 $EndComp
+$Comp
+L power:VCC #PWR0112
+U 1 1 6024E04F
+P 2950 1000
+F 0 "#PWR0112" H 2950 850 50  0001 C CNN
+F 1 "VCC" H 2965 1173 50  0000 C CNN
+F 2 "" H 2950 1000 50  0001 C CNN
+F 3 "" H 2950 1000 50  0001 C CNN
+	1    2950 1000
+	1    0    0    -1
+$EndComp
 Wire Wire Line
 	2950 1400 2950 1000
@@
 NoConn ~ 3550 3800
 NoConn ~ 3550 3900
-$Comp
-L power:+3V3 #PWR?
-U 1 1 601B583E
-P 2950 1000
-F 0 "#PWR?" H 2950 850 50  0001 C CNN
-F 1 "+3V3" H 2965 1173 50  0000 C CNN
-F 2 "" H 2950 1000 50  0001 C CNN
-F 3 "" H 2950 1000 50  0001 C CNN
-	1    2950 1000
-	1    0    0    -1
-$EndComp
 $EndSCHEMATC
