File: Krokovka 4.sch (KiCad schematic (older format))
At the start: 9 parts, among them J22 Conn_01x08_Female, J24 Conn_01x01_Female, J26 Conn_01x02_Female, J27 Conn_01x08_Female, J28 Conn_01x04_Male

Commit message: Deska 0.5
Parts:
- removed J22, J27: Conn_01x08_Female, symbol Connector:Conn_01x08_Female
- removed J24: Conn_01x01_Female, symbol Connector:Conn_01x01_Female
- removed J26: Conn_01x02_Female, symbol Connector:Conn_01x02_Female
- added 2209Br4: TMC2209BreaoutBoard, symbol Tmc2209BreakoutBoard:TMC2209BreaoutBoard
Connections:
- net labels removed: A1, A2, B1, B2, CLK, DIAG, DIR, EN, INDEX, MS1, MS2, PDN_UART, STEP, VCC, VDD, VM, VREF
- wire segments 35 -> 18
Other:
- moved on the sheet: C14, C15, C16, C17, J28
