File: Krokovka 4.sch (KiCad schematic (older format))
At the start: 6 parts, among them J28 Conn_01x04_Male

Commit message: Doplnen reset
Parts:
- added C?: 10nF, symbol Device:C
Connections:
- net labels added: VDD_4
- wire segments 18 -> 23
Changed lines of the file:
@@
-$EndComp
-$Comp
-L power:+3V3 #PWR0123
-U 1 1 601BA865
-P 3100 5800
-F 0 "#PWR0123" H 3100 5650 50  0001 C CNN
-F 1 "+3V3" V 3115 5928 50  0000 L CNN
-F 2 "" H 3100 5800 50  0001 C CNN
-F 3 "" H 3100 5800 50  0001 C CNN
-	1    3100 5800
-	0    1    1    0
 $EndComp
 $Comp
@@
 F 3 "" H 2250 5300 50  0001 C CNN
 	1    2250 5300
-	0    -1   -1   0
-$EndComp
-$Comp
-L power:GND #PWR?
-U 1 1 60284C80
-P 3100 5900
-AR Path="/601BF914/60284C80" Ref="#PWR?"  Part="1"
-AR Path="/601E7BA1/60284C80" Ref="#PWR?"  Part="1"
-AR Path="/60210E5F/60284C80" Ref="#PWR?"  Part="1"
-AR Path="/60218F69/60284C80" Ref="#PWR013"  Part="1"
-F 0 "#PWR013" H 3100 5650 50  0001 C CNN
-F 1 "GND" V 3105 5772 50  0000 R CNN
-F 2 "" H 3100 5900 50  0001 C CNN
-F 3 "" H 3100 5900 50  0001 C CNN
-	1    3100 5900
 	0    -1   -1   0
 $EndComp
@@
 	1    0    0    -1
 $EndComp
+$Comp
+L power:GND #PWR?
+U 1 1 602430E4
+P 3350 6100
+AR Path="/601BF914/602430E4" Ref="#PWR?"  Part="1"
+AR Path="/601E7BA1/602430E4" Ref="#PWR?"  Part="1"
+AR Path="/60210E5F/602430E4" Ref="#PWR?"  Part="1"
+F 0 "#PWR?" H 3350 5850 50  0001 C CNN
+F 1 "GND" V 3355 5972 50  0000 R CNN
+F 2 "" H 3350 6100 50  0001 C CNN
+F 3 "" H 3350 6100 50  0001 C CNN
+	1    3350 6100
+	0    -1   -1   0
+$EndComp
+$Comp
+L Device:C C?
+U 1 1 602430EA
+P 3250 5950
+AR Path="/601BF914/602430EA" Ref="C?"  Part="1"
+AR Path="/601E7BA1/602430EA" Ref="C?"  Part="1"
+AR Path="/60210E5F/602430EA" Ref="C?"  Part="1"
+F 0 "C?" H 3200 6350 50  0000 L CNN
+F 1 "10nF" H 3150 6250 50  0000 L CNN
+F 2 "" H 3288 5800 50  0001 C CNN
+F 3 "~" H 3250 5950 50  0001 C CNN
+	1    3250 5950
+	-1   0    0    1
+$EndComp
+Wire Wire Line
+	3100 6100 3250 6100
+Wire Wire Line
+	3350 6100 3250 6100
+Connection ~ 3250 6100
+Text HLabel 3400 5800 2    50   Input ~ 0
+VDD_4
+Wire Wire Line
+	3400 5800 3250 5800
+Wire Wire Line
+	3250 5800 3100 5800
+Connection ~ 3250 5800
+Wire Wire Line
+	3100 5900 3100 6100
 $EndSCHEMATC

Commit message: Mosfet
Parts:
- gave numbers to parts that had none: 1
Changed lines of the file:
@@
 AR Path="/601E7BA1/602430E4" Ref="#PWR?"  Part="1"
 AR Path="/60210E5F/602430E4" Ref="#PWR?"  Part="1"
-F 0 "#PWR?" H 3350 5850 50  0001 C CNN
+AR Path="/60218F69/602430E4" Ref="#PWR05"  Part="1"
+F 0 "#PWR05" H 3350 5850 50  0001 C CNN
 F 1 "GND" V 3355 5972 50  0000 R CNN
 F 2 "" H 3350 6100 50  0001 C CNN
@@
 AR Path="/601E7BA1/602430EA" Ref="C?"  Part="1"
 AR Path="/60210E5F/602430EA" Ref="C?"  Part="1"
-F 0 "C?" H 3200 6350 50  0000 L CNN
+AR Path="/60218F69/602430EA" Ref="C19"  Part="1"
+F 0 "C19" H 3200 6350 50  0000 L CNN
 F 1 "10nF" H 3150 6250 50  0000 L CNN
 F 2 "" H 3288 5800 50  0001 C CNN

Commit message: Jirka upravy
Parts:
- removed C14, C15, C16, C17: 470pF, symbol Device:C
- added R? (x2): 1k, symbol Device:R
- C19: value 10nF -> 100nF
Connections:
- wire segments 23 -> 10
Changed lines of the file:
@@
 $EndDescr
-$Comp
-L Device:C C?
-U 1 1 6021D36B
-P 3950 6250
-AR Path="/601BF914/6021D36B" Ref="C?"  Part="1"
-AR Path="/601E7BA1/6021D36B" Ref="C?"  Part="1"
-AR Path="/60210E5F/6021D36B" Ref="C?"  Part="1"
-AR Path="/60218F69/6021D36B" Ref="C14"  Part="1"
-F 0 "C14" H 4065 6296 50  0000 L CNN
-F 1 "470pF" H 4065 6205 50  0000 L CNN
-F 2 "" H 3988 6100 50  0001 C CNN
-F 3 "~" H 3950 6250 50  0001 C CNN
-	1    3950 6250
-	1    0    0    -1
-$EndComp
-$Comp
-L Device:C C?
-U 1 1 6021D371
-P 4650 6250
-AR Path="/601BF914/6021D371" Ref="C?"  Part="1"
-AR Path="/601E7BA1/6021D371" Ref="C?"  Part="1"
-AR Path="/60210E5F/6021D371" Ref="C?"  Part="1"
-AR Path="/60218F69/6021D371" Ref="C16"  Part="1"
-F 0 "C16" H 4765 6296 50  0000 L CNN
-F 1 "470pF" H 4765 6205 50  0000 L CNN
-F 2 "" H 4688 6100 50  0001 C CNN
-F 3 "~" H 4650 6250 50  0001 C CNN
-	1    4650 6250
-	1    0    0    -1
-$EndComp
-$Comp
-L Device:C C?
-U 1 1 6021D377
-P 5000 6250
-AR Path="/601BF914/6021D377" Ref="C?"  Part="1"
-AR Path="/601E7BA1/6021D377" Ref="C?"  Part="1"
-AR Path="/60210E5F/6021D377" Ref="C?"  Part="1"
-AR Path="/60218F69/6021D377" Ref="C17"  Part="1"
-F 0 "C17" H 5115 6296 50  0000 L CNN
-F 1 "470pF" H 5115 6205 50  0000 L CNN
-F 2 "" H 5038 6100 50  0001 C CNN
-F 3 "~" H 5000 6250 50  0001 C CNN
-	1    5000 6250
-	1    0    0    -1
-$EndComp
 $Comp
 L Connector:Conn_01x04_Male J?
@@
 	-1   0    0    1
 $EndComp
-Wire Wire Line
-	3100 5700 3950 5700
-Wire Wire Line
-	3100 5600 4300 5600
-Wire Wire Line
-	3950 6100 3950 5700
-Connection ~ 3950 5700
-Wire Wire Line
-	3950 5700 5100 5700
-Connection ~ 4300 5600
-Wire Wire Line
-	4300 5600 5100 5600
-Wire Wire Line
-	4650 6100 4650 5500
-Connection ~ 4650 5500
-Wire Wire Line
-	4650 5500 5100 5500
-Wire Wire Line
-	5000 6100 5000 5400
-Connection ~ 5000 5400
-Wire Wire Line
-	5000 5400 5100 5400
-$Comp
-L power:GND #PWR?
-U 1 1 6021D399
-P 3950 6500
-AR Path="/601BF914/6021D399" Ref="#PWR?"  Part="1"
-AR Path="/601E7BA1/6021D399" Ref="#PWR?"  Part="1"
-AR Path="/60210E5F/6021D399" Ref="#PWR?"  Part="1"
-AR Path="/60218F69/6021D399" Ref="#PWR045"  Part="1"
-F 0 "#PWR045" H 3950 6250 50  0001 C CNN
-F 1 "GND" H 3955 6327 50  0000 C CNN
-F 2 "" H 3950 6500 50  0001 C CNN
-F 3 "" H 3950 6500 50  0001 C CNN
-	1    3950 6500
-	1    0    0    -1
-$EndComp
-$Comp
-L power:GND #PWR?
-U 1 1 6021D39F
-P 4300 6500
-AR Path="/601BF914/6021D39F" Ref="#PWR?"  Part="1"
-AR Path="/601E7BA1/6021D39F" Ref="#PWR?"  Part="1"
-AR Path="/60210E5F/6021D39F" Ref="#PWR?"  Part="1"
-AR Path="/60218F69/6021D39F" Ref="#PWR046"  Part="1"
-F 0 "#PWR046" H 4300 6250 50  0001 C CNN
-F 1 "GND" H 4305 6327 50  0000 C CNN
-F 2 "" H 4300 6500 50  0001 C CNN
-F 3 "" H 4300 6500 50  0001 C CNN
-	1    4300 6500
-	1    0    0    -1
-$EndComp
-$Comp
-L power:GND #PWR?
-U 1 1 6021D3A5
-P 4650 6500
-AR Path="/601BF914/6021D3A5" Ref="#PWR?"  Part="1"
-AR Path="/601E7BA1/6021D3A5" Ref="#PWR?"  Part="1"
-AR Path="/60210E5F/6021D3A5" Ref="#PWR?"  Part="1"
-AR Path="/60218F69/6021D3A5" Ref="#PWR047"  Part="1"
-F 0 "#PWR047" H 4650 6250 50  0001 C CNN
-F 1 "GND" H 4655 6327 50  0000 C CNN
-F 2 "" H 4650 6500 50  0001 C CNN
-F 3 "" H 4650 6500 50  0001 C CNN
-	1    4650 6500
-	1    0    0    -1
-$EndComp
-Wire Wire Line
-	3950 6400 3950 6500
-Wire Wire Line
-	4650 6400 4650 6500
-Wire Wire Line
-	4300 6400 4300 6500
-Wire Wire Line
-	4300 6100 4300 5600
-$Comp
-L Device:C C?
-U 1 1 6021D3B6
-P 4300 6250
-AR Path="/601BF914/6021D3B6" Ref="C?"  Part="1"
-AR Path="/601E7BA1/6021D3B6" Ref="C?"  Part="1"
-AR Path="/60210E5F/6021D3B6" Ref="C?"  Part="1"
-AR Path="/60218F69/6021D3B6" Ref="C15"  Part="1"
-F 0 "C15" H 4415 6296 50  0000 L CNN
-F 1 "470pF" H 4415 6205 50  0000 L CNN
-F 2 "" H 4338 6100 50  0001 C CNN
-F 3 "~" H 4300 6250 50  0001 C CNN
-	1    4300 6250
-	1    0    0    -1
-$EndComp
 Text HLabel 2250 5200 0    50   Input ~ 0
 EN4
-Text HLabel 2250 5600 0    50   Input ~ 0
-PDN_4
-$Comp
-L power:GND #PWR?
-U 1 1 6021D3CD
-P 3100 5300
-AR Path="/601BF914/6021D3CD" Ref="#PWR?"  Part="1"
-AR Path="/601E7BA1/6021D3CD" Ref="#PWR?"  Part="1"
-AR Path="/60210E5F/6021D3CD" Ref="#PWR?"  Part="1"
-AR Path="/60218F69/6021D3CD" Ref="#PWR043"  Part="1"
-F 0 "#PWR043" H 3100 5050 50  0001 C CNN
-F 1 "GND" V 3105 5172 50  0000 R CNN
-F 2 "" H 3100 5300 50  0001 C CNN
-F 3 "" H 3100 5300 50  0001 C CNN
-	1    3100 5300
-	0    -1   -1   0
-$EndComp
-$Comp
-L power:GND #PWR?
-U 1 1 60251790
-P 5000 6500
-AR Path="/601BF914/60251790" Ref="#PWR?"  Part="1"
-AR Path="/601E7BA1/60251790" Ref="#PWR?"  Part="1"
-AR Path="/60210E5F/60251790" Ref="#PWR?"  Part="1"
-AR Path="/60218F69/60251790" Ref="#PWR0108"  Part="1"
-F 0 "#PWR0108" H 5000 6250 50  0001 C CNN
-F 1 "GND" H 5005 6327 50  0000 C CNN
-F 2 "" H 5000 6500 50  0001 C CNN
-F 3 "" H 5000 6500 50  0001 C CNN
-	1    5000 6500
-	1    0    0    -1
-$EndComp
-Wire Wire Line
-	5000 6500 5000 6400
 Text HLabel 2600 4800 1    50   Input ~ 0
 INDEX_4
-$Comp
-L power:+10V #PWR0122
-U 1 1 601B9CD6
-P 3100 5200
-F 0 "#PWR0122" H 3100 5050 50  0001 C CNN
-F 1 "+10V" V 3115 5328 50  0000 L CNN
-F 2 "" H 3100 5200 50  0001 C CNN
-F 3 "" H 3100 5200 50  0001 C CNN
-	1    3100 5200
-	0    1    1    0
-$EndComp
-$Comp
-L power:+3V3 #PWR0106
-U 1 1 601B673B
-P 2250 5300
-F 0 "#PWR0106" H 2250 5150 50  0001 C CNN
-F 1 "+3V3" V 2265 5428 50  0000 L CNN
-F 2 "" H 2250 5300 50  0001 C CNN
-F 3 "" H 2250 5300 50  0001 C CNN
-	1    2250 5300
-	0    -1   -1   0
-$EndComp
-Wire Wire Line
-	2250 5600 2250 5500
-NoConn ~ 2250 5700
-NoConn ~ 2500 4800
-NoConn ~ 2700 4800
-Wire Wire Line
-	2250 5400 2250 5300
-NoConn ~ 2250 5900
-NoConn ~ 2250 5800
-Wire Wire Line
-	3100 5500 4650 5500
-Wire Wire Line
-	3100 5400 5000 5400
-Connection ~ 2250 5300
-$Comp
-L Základní-deska-II-rescue:TMC2209BreaoutBoard-Tmc2209BreakoutBoard 2209Br4
-U 1 1 6027E2D2
-P 2700 5450
-F 0 "2209Br4" H 2675 4877 50  0000 C CNN
-F 1 "TMC2209BreaoutBoard" H 2675 4786 50  0000 C CNN
-F 2 "" H 2450 5450 50  0001 C CNN
-F 3 "" H 2450 5450 50  0001 C CNN
-	1    2700 5450
-	1    0    0    -1
-$EndComp
 $Comp
 L power:GND #PWR?
@@
 AR Path="/60218F69/602430EA" Ref="C19"  Part="1"
 F 0 "C19" H 3200 6350 50  0000 L CNN
-F 1 "10nF" H 3150 6250 50  0000 L CNN
+F 1 "100nF" H 3150 6250 50  0000 L CNN
 F 2 "" H 3288 5800 50  0001 C CNN
 F 3 "~" H 3250 5950 50  0001 C CNN
@@
 Wire Wire Line
 	3400 5800 3250 5800
+Connection ~ 3250 5800
+Text HLabel 2250 5600 0    50   Input ~ 0
+PDN_4
+Wire Wire Line
+	3100 5900 3100 6100
+NoConn ~ 2250 5900
+NoConn ~ 2250 5800
+NoConn ~ 2250 5700
+Wire Wire Line
+	2250 5600 2250 5500
+NoConn ~ 2700 4800
+NoConn ~ 2500 4800
+$Comp
+L power:+10V #PWR0122
+U 1 1 601B9CD6
+P 3100 5200
+F 0 "#PWR0122" H 3100 5050 50  0001 C CNN
+F 1 "+10V" V 3115 5328 50  0000 L CNN
+F 2 "" H 3100 5200 50  0001 C CNN
+F 3 "" H 3100 5200 50  0001 C CNN
+	1    3100 5200
+	0    1    1    0
+$EndComp
+$Comp
+L power:GND #PWR?
+U 1 1 6021D3CD
+P 3100 5300
+AR Path="/601BF914/6021D3CD" Ref="#PWR?"  Part="1"
+AR Path="/601E7BA1/6021D3CD" Ref="#PWR?"  Part="1"
+AR Path="/60210E5F/6021D3CD" Ref="#PWR?"  Part="1"
+AR Path="/60218F69/6021D3CD" Ref="#PWR043"  Part="1"
+F 0 "#PWR043" H 3100 5050 50  0001 C CNN
+F 1 "GND" V 3105 5172 50  0000 R CNN
+F 2 "" H 3100 5300 50  0001 C CNN
+F 3 "" H 3100 5300 50  0001 C CNN
+	1    3100 5300
+	0    -1   -1   0
+$EndComp
+Wire Wire Line
+	3100 5400 5100 5400
+Wire Wire Line
+	3100 5500 5100 5500
+Wire Wire Line
+	3100 5600 5100 5600
+Wire Wire Line
+	3100 5700 5100 5700
 Wire Wire Line
 	3250 5800 3100 5800
-Connection ~ 3250 5800
-Wire Wire Line
-	3100 5900 3100 6100
+$Comp
+L Základní-deska-II-rescue:TMC2209BreaoutBoard-Tmc2209BreakoutBoard 2209Br4
+U 1 1 6027E2D2
+P 2700 5450
+F 0 "2209Br4" H 2675 4877 50  0000 C CNN
+F 1 "TMC2209BreaoutBoard" H 2675 4786 50  0000 C CNN
+F 2 "" H 2450 5450 50  0001 C CNN
+F 3 "" H 2450 5450 50  0001 C CNN
+	1    2700 5450
+	1    0    0    -1
+$EndComp
+$Comp
+L power:+3V3 #PWR0106
+U 1 1 601B673B
+P 1950 5300
+F 0 "#PWR0106" H 1950 5150 50  0001 C CNN
+F 1 "+3V3" V 1950 5500 50  0000 L CNN
+F 2 "" H 1950 5300 50  0001 C CNN
+F 3 "" H 1950 5300 50  0001 C CNN
+	1    1950 5300
+	0    -1   -1   0
+$EndComp
+$Comp
+L Device:R R?
+U 1 1 6025F32C
+P 2100 5300
+F 0 "R?" V 1893 5300 50  0000 C CNN
+F 1 "1k" V 1984 5300 50  0000 C CNN
+F 2 "" V 2030 5300 50  0001 C CNN
+F 3 "~" H 2100 5300 50  0001 C CNN
+	1    2100 5300
+	0    1    1    0
+$EndComp
+$Comp
+L Device:R R?
+U 1 1 6025F620
+P 2100 5400
+F 0 "R?" V 1893 5400 50  0000 C CNN
+F 1 "1k" V 1984 5400 50  0000 C CNN
+F 2 "" V 2030 5400 50  0001 C CNN
+F 3 "~" H 2100 5400 50  0001 C CNN
+	1    2100 5400
+	0    1    1    0
+$EndComp
+$Comp
+L power:+3V3 #PWR?
+U 1 1 6025F823
+P 1950 5400
+F 0 "#PWR?" H 1950 5250 50  0001 C CNN
+F 1 "+3V3" V 1950 5600 50  0000 L CNN
+F 2 "" H 1950 5400 50  0001 C CNN
+F 3 "" H 1950 5400 50  0001 C CNN
+	1    1950 5400
+	0    -1   -1   0
+$EndComp
 $EndSCHEMATC

Commit message: Hotové schéma
Parts:
- 2209Br4: LCSC (none) -> -
- C19: footprint (none) -> Capacitor_SMD:C_0402_1005Metric_Pad0.74x0.62mm_HandSolder; LCSC (none) -> C14663
- J28: footprint (none) -> Connector_PinHeader_2.54mm:PinHeader_1x04_P2.54mm_Vertical; LCSC (none) -> -
- R12, R13: renamed from R?; footprint (none) -> Resistor_SMD:R_0805_2012Metric_Pad1.20x1.40mm_HandSolder; LCSC (none) -> C17513
Connections:
- wire segments 10 -> 14
Other:
- moved on the sheet: J28, R12, R13
Changed lines of the file:
@@
 Comment4 ""
 $EndDescr
-$Comp
-L Connector:Conn_01x04_Male J?
-U 1 1 6021D37D
-P 5300 5600
-AR Path="/601BF914/6021D37D" Ref="J?"  Part="1"
-AR Path="/601E7BA1/6021D37D" Ref="J?"  Part="1"
-AR Path="/60210E5F/6021D37D" Ref="J?"  Part="1"
-AR Path="/60218F69/6021D37D" Ref="J28"  Part="1"
-F 0 "J28" H 5272 5482 50  0000 R CNN
-F 1 "Conn_01x04_Male" H 5272 5573 50  0000 R CNN
-F 2 "" H 5300 5600 50  0001 C CNN
-F 3 "~" H 5300 5600 50  0001 C CNN
-	1    5300 5600
-	-1   0    0    1
-$EndComp
 Text HLabel 2250 5200 0    50   Input ~ 0
 EN4
@@
 F 0 "C19" H 3200 6350 50  0000 L CNN
 F 1 "100nF" H 3150 6250 50  0000 L CNN
-F 2 "" H 3288 5800 50  0001 C CNN
+F 2 "Capacitor_SMD:C_0402_1005Metric_Pad0.74x0.62mm_HandSolder" H 3288 5800 50  0001 C CNN
 F 3 "~" H 3250 5950 50  0001 C CNN
+F 4 "C14663" H 3250 5950 50  0001 C CNN "LCSC"
 	1    3250 5950
 	-1   0    0    1
@@
 $EndComp
 Wire Wire Line
-	3100 5400 5100 5400
-Wire Wire Line
-	3100 5500 5100 5500
-Wire Wire Line
-	3100 5600 5100 5600
-Wire Wire Line
-	3100 5700 5100 5700
-Wire Wire Line
 	3250 5800 3100 5800
 $Comp
@@
 F 2 "" H 2450 5450 50  0001 C CNN
 F 3 "" H 2450 5450 50  0001 C CNN
+F 4 "-" H 2700 5450 50  0001 C CNN "LCSC"
 	1    2700 5450
 	1    0    0    -1
@@
 L power:+3V3 #PWR0106
 U 1 1 601B673B
+P 1550 5300
+F 0 "#PWR0106" H 1550 5150 50  0001 C CNN
+F 1 "+3V3" V 1550 5500 50  0000 L CNN
+F 2 "" H 1550 5300 50  0001 C CNN
+F 3 "" H 1550 5300 50  0001 C CNN
+	1    1550 5300
+	0    -1   -1   0
+$EndComp
+$Comp
+L Device:R R12
+U 1 1 6025F32C
+P 1700 5300
+F 0 "R12" V 1600 5300 50  0000 C CNN
+F 1 "1k" V 1700 5300 50  0000 C CNN
+F 2 "Resistor_SMD:R_0805_2012Metric_Pad1.20x1.40mm_HandSolder" V 1630 5300 50  0001 C CNN
+F 3 "~" H 1700 5300 50  0001 C CNN
+F 4 "C17513" H 1700 5300 50  0001 C CNN "LCSC"
+	1    1700 5300
+	0    1    1    0
+$EndComp
+$Comp
+L Device:R R13
+U 1 1 6025F620
+P 1700 5400
+F 0 "R13" V 1800 5400 50  0000 C CNN
+F 1 "1k" V 1700 5400 50  0000 C CNN
+F 2 "Resistor_SMD:R_0805_2012Metric_Pad1.20x1.40mm_HandSolder" V 1630 5400 50  0001 C CNN
+F 3 "~" H 1700 5400 50  0001 C CNN
+F 4 "C17513" H 1700 5400 50  0001 C CNN "LCSC"
+	1    1700 5400
+	0    1    1    0
+$EndComp
+$Comp
+L power:+3V3 #PWR013
+U 1 1 6025F823
+P 1550 5400
+F 0 "#PWR013" H 1550 5250 50  0001 C CNN
+F 1 "+3V3" V 1550 5600 50  0000 L CNN
+F 2 "" H 1550 5400 50  0001 C CNN
+F 3 "" H 1550 5400 50  0001 C CNN
+	1    1550 5400
+	0    -1   -1   0
+$EndComp
+Wire Wire Line
+	3100 5400 3450 5400
+Wire Wire Line
+	3100 5500 3450 5500
+Wire Wire Line
+	3100 5600 3450 5600
+Wire Wire Line
+	3100 5700 3450 5700
+$Comp
+L Connector:Conn_01x04_Male J?
+U 1 1 6021D37D
+P 3650 5600
+AR Path="/601BF914/6021D37D" Ref="J?"  Part="1"
+AR Path="/601E7BA1/6021D37D" Ref="J?"  Part="1"
+AR Path="/60210E5F/6021D37D" Ref="J?"  Part="1"
+AR Path="/60218F69/6021D37D" Ref="J28"  Part="1"
+F 0 "J28" H 3622 5482 50  0000 R CNN
+F 1 "Conn_01x04_Male" H 3622 5573 50  0000 R CNN
+F 2 "Connector_PinHeader_2.54mm:PinHeader_1x04_P2.54mm_Vertical" H 3650 5600 50  0001 C CNN
+F 3 "~" H 3650 5600 50  0001 C CNN
+F 4 "-" H 3650 5600 50  0001 C CNN "LCSC"
+	1    3650 5600
+	-1   0    0    1
+$EndComp
+Wire Wire Line
+	1850 5300 1950 5300
+Wire Wire Line
+	2250 5400 1950 5400
+$Comp
+L power:PWR_FLAG #FLG0104
+U 1 1 6022C389
+P 1950 5400
+F 0 "#FLG0104" H 1950 5475 50  0001 C CNN
+F 1 "PWR_FLAG" V 2050 5600 50  0000 C CNN
+F 2 "" H 1950 5400 50  0001 C CNN
+F 3 "~" H 1950 5400 50  0001 C CNN
+	1    1950 5400
+	-1   0    0    1
+$EndComp
+Connection ~ 1950 5400
+Wire Wire Line
+	1950 5400 1850 5400
+$Comp
+L power:PWR_FLAG #FLG0105
+U 1 1 6022C9EA
 P 1950 5300
-F 0 "#PWR0106" H 1950 5150 50  0001 C CNN
-F 1 "+3V3" V 1950 5500 50  0000 L CNN
+F 0 "#FLG0105" H 1950 5375 50  0001 C CNN
+F 1 "PWR_FLAG" V 1850 5500 50  0000 C CNN
 F 2 "" H 1950 5300 50  0001 C CNN
-F 3 "" H 1950 5300 50  0001 C CNN
+F 3 "~" H 1950 5300 50  0001 C CNN
 	1    1950 5300
-	0    -1   -1   0
-$EndComp
-$Comp
-L Device:R R?
-U 1 1 6025F32C
-P 2100 5300
-F 0 "R?" V 1893 5300 50  0000 C CNN
-F 1 "1k" V 1984 5300 50  0000 C CNN
-F 2 "" V 2030 5300 50  0001 C CNN
-F 3 "~" H 2100 5300 50  0001 C CNN
-	1    2100 5300
-	0    1    1    0
-$EndComp
-$Comp
-L Device:R R?
-U 1 1 6025F620
-P 2100 5400
-F 0 "R?" V 1893 5400 50  0000 C CNN
-F 1 "1k" V 1984 5400 50  0000 C CNN
-F 2 "" V 2030 5400 50  0001 C CNN
-F 3 "~" H 2100 5400 50  0001 C CNN
-	1    2100 5400
-	0    1    1    0
-$EndComp
-$Comp
-L power:+3V3 #PWR?
-U 1 1 6025F823
-P 1950 5400
-F 0 "#PWR?" H 1950 5250 50  0001 C CNN
-F 1 "+3V3" V 1950 5600 50  0000 L CNN
-F 2 "" H 1950 5400 50  0001 C CNN
-F 3 "" H 1950 5400 50  0001 C CNN
-	1    1950 5400
-	0    -1   -1   0
-$EndComp
+	1    0    0    -1
+$EndComp
+Connection ~ 1950 5300
+Wire Wire Line
+	1950 5300 2250 5300
 $EndSCHEMATC

Commit message: Hotová deska
Parts:
- 2209Br4: footprint (none) -> FinalExamThesis:TMC_2209_Breaout_Board
Changed lines of the file:
@@
 F 0 "2209Br4" H 2675 4877 50  0000 C CNN
 F 1 "TMC2209BreaoutBoard" H 2675 4786 50  0000 C CNN
-F 2 "" H 2450 5450 50  0001 C CNN
+F 2 "FinalExamThesis:TMC_2209_Breaout_Board" H 2450 5450 50  0001 C CNN
 F 3 "" H 2450 5450 50  0001 C CNN
 F 4 "-" H 2700 5450 50  0001 C CNN "LCSC"

Commit message: Nová Deska
Parts:
- added C4: 2,2mF, Capacitor_THT:CP_Radial_D10.0mm_P2.50mm, symbol Device:C
- 2209Br4: symbol Základní-deska-II-rescue:TMC2209BreaoutBoard-Tmc2209BreakoutBoard -> Základní-deska-II-rescue:TMC2209BreaoutBoard-Tmc2209BreakoutBoard-Základní-deska-II-rescue
Connections:
- wire segments 14 -> 17
Changed lines of the file:
@@
 L power:+10V #PWR0122
 U 1 1 601B9CD6
-P 3100 5200
-F 0 "#PWR0122" H 3100 5050 50  0001 C CNN
-F 1 "+10V" V 3115 5328 50  0000 L CNN
-F 2 "" H 3100 5200 50  0001 C CNN
-F 3 "" H 3100 5200 50  0001 C CNN
-	1    3100 5200
+P 3250 5000
+F 0 "#PWR0122" H 3250 4850 50  0001 C CNN
+F 1 "+10V" V 3265 5128 50  0000 L CNN
+F 2 "" H 3250 5000 50  0001 C CNN
+F 3 "" H 3250 5000 50  0001 C CNN
+	1    3250 5000
 	0    1    1    0
 $EndComp
@@
 L power:GND #PWR?
 U 1 1 6021D3CD
-P 3100 5300
+P 3250 5300
 AR Path="/601BF914/6021D3CD" Ref="#PWR?"  Part="1"
 AR Path="/601E7BA1/6021D3CD" Ref="#PWR?"  Part="1"
 AR Path="/60210E5F/6021D3CD" Ref="#PWR?"  Part="1"
 AR Path="/60218F69/6021D3CD" Ref="#PWR043"  Part="1"
-F 0 "#PWR043" H 3100 5050 50  0001 C CNN
-F 1 "GND" V 3105 5172 50  0000 R CNN
-F 2 "" H 3100 5300 50  0001 C CNN
-F 3 "" H 3100 5300 50  0001 C CNN
-	1    3100 5300
+F 0 "#PWR043" H 3250 5050 50  0001 C CNN
+F 1 "GND" V 3255 5172 50  0000 R CNN
+F 2 "" H 3250 5300 50  0001 C CNN
+F 3 "" H 3250 5300 50  0001 C CNN
+	1    3250 5300
 	0    -1   -1   0
 $EndComp
@@
 	3250 5800 3100 5800
 $Comp
-L Základní-deska-II-rescue:TMC2209BreaoutBoard-Tmc2209BreakoutBoard 2209Br4
+L Základní-deska-II-rescue:TMC2209BreaoutBoard-Tmc2209BreakoutBoard-Základní-deska-II-rescue 2209Br4
 U 1 1 6027E2D2
 P 2700 5450
@@
 Wire Wire Line
 	1950 5300 2250 5300
+$Comp
+L Device:C C?
+U 1 1 602BB06A
+P 3250 5150
+AR Path="/601BF914/602BB06A" Ref="C?"  Part="1"
+AR Path="/60218F69/602BB06A" Ref="C4"  Part="1"
+F 0 "C4" H 3365 5196 50  0000 L CNN
+F 1 "2,2mF" H 3365 5105 50  0000 L CNN
+F 2 "Capacitor_THT:CP_Radial_D10.0mm_P2.50mm" H 3288 5000 50  0001 C CNN
+F 3 "~" H 3250 5150 50  0001 C CNN
+F 4 "C138489" H 3250 5150 50  0001 C CNN "LCSC"
+	1    3250 5150
+	1    0    0    -1
+$EndComp
+Wire Wire Line
+	3100 5300 3250 5300
+Connection ~ 3250 5300
+Wire Wire Line
+	3100 5200 3100 5000
+Wire Wire Line
+	3100 5000 3250 5000
+Connection ~ 3250 5000
 $EndSCHEMATC

Commit message: Deska 1.1
Parts:
- C4: value 2,2mF -> 470uF; LCSC C138489 -> C34642
Changed lines of the file:
@@
 AR Path="/60218F69/602BB06A" Ref="C4"  Part="1"
 F 0 "C4" H 3365 5196 50  0000 L CNN
-F 1 "2,2mF" H 3365 5105 50  0000 L CNN
+F 1 "470uF" H 3365 5105 50  0000 L CNN
 F 2 "Capacitor_THT:CP_Radial_D10.0mm_P2.50mm" H 3288 5000 50  0001 C CNN
 F 3 "~" H 3250 5150 50  0001 C CNN
-F 4 "C138489" H 3250 5150 50  0001 C CNN "LCSC"
+F 4 "C34642" H 3250 5150 50  0001 C CNN "LCSC"
 	1    3250 5150
 	1    0    0    -1

Commit message: release candidate
Parts:
- C19: LCSC C14663 -> C1525
Changed lines of the file:
@@
 F 2 "Capacitor_SMD:C_0402_1005Metric_Pad0.74x0.62mm_HandSolder" H 3288 5800 50  0001 C CNN
 F 3 "~" H 3250 5950 50  0001 C CNN
-F 4 "C14663" H 3250 5950 50  0001 C CNN "LCSC"
+F 4 "C1525" H 3250 5950 50  0001 C CNN "LCSC"
 	1    3250 5950
 	-1   0    0    1
