File: Krokovka 4.sch (KiCad schematic (older format))
At the start: 6 parts, among them J28 Conn_01x04_Male

Commit message: Ordered
Parts:
- 2209Br4: symbol Základní-deska-II-rescue:TMC2209BreaoutBoard-Tmc2209BreakoutBoard-Základní-deska-II-rescue -> Zakladni_deska_II-rescue:TMC2209BreaoutBoard; JLCPCB_IGNORE (none) -> 1
- J28: JLCPCB_IGNORE (none) -> 1
- R12, R13: LCSC C17513 -> C17379
Changed lines of the file:
@@
 	3250 5800 3100 5800
 $Comp
-L Základní-deska-II-rescue:TMC2209BreaoutBoard-Tmc2209BreakoutBoard-Základní-deska-II-rescue 2209Br4
+L Zakladni_deska_II-rescue:TMC2209BreaoutBoard 2209Br4
 U 1 1 6027E2D2
 P 2700 5450
@@
 F 3 "" H 2450 5450 50  0001 C CNN
 F 4 "-" H 2700 5450 50  0001 C CNN "LCSC"
+F 5 "1" H 2700 5450 50  0001 C CNN "JLCPCB_IGNORE"
 	1    2700 5450
 	1    0    0    -1
@@
 F 2 "Resistor_SMD:R_0805_2012Metric_Pad1.20x1.40mm_HandSolder" V 1630 5300 50  0001 C CNN
 F 3 "~" H 1700 5300 50  0001 C CNN
-F 4 "C17513" H 1700 5300 50  0001 C CNN "LCSC"
+F 4 "C17379" H 1700 5300 50  0001 C CNN "LCSC"
 	1    1700 5300
 	0    1    1    0
@@
 F 2 "Resistor_SMD:R_0805_2012Metric_Pad1.20x1.40mm_HandSolder" V 1630 5400 50  0001 C CNN
 F 3 "~" H 1700 5400 50  0001 C CNN
-F 4 "C17513" H 1700 5400 50  0001 C CNN "LCSC"
+F 4 "C17379" H 1700 5400 50  0001 C CNN "LCSC"
 	1    1700 5400
 	0    1    1    0
@@
 F 3 "~" H 3650 5600 50  0001 C CNN
 F 4 "-" H 3650 5600 50  0001 C CNN "LCSC"
+F 5 "1" H 3650 5600 50  0001 C CNN "JLCPCB_IGNORE"
 	1    3650 5600
 	-1   0    0    1
