File: Krokovka1.sch (KiCad schematic (older format))
At the start: 9 parts, among them J1 Conn_01x08_Female, J2 Conn_01x01_Female, J3 Conn_01x02_Female, J4 Conn_01x08_Female, J7 Conn_01x04_Male

Commit message: Deska 0.5
Parts:
- removed J1, J4: Conn_01x08_Female, symbol Connector:Conn_01x08_Female
- removed J2: Conn_01x01_Female, symbol Connector:Conn_01x01_Female
- removed J3: Conn_01x02_Female, symbol Connector:Conn_01x02_Female
- added 2209Br1: TMC2209BreaoutBoard, symbol Tmc2209BreakoutBoard:TMC2209BreaoutBoard
Connections:
- net labels removed: A1, A2, B1, B2, CLK, DIAG, DIR, EN, INDEX, MS1, MS2, PDN_UART, STEP, VDD, VM, VREF
- wire segments 33 -> 18
Other:
- moved on the sheet: C2, C3, C4, C5, J7
