File: Krokovka1.sch (KiCad schematic (older format))
At the start: 6 parts, among them J7 Conn_01x04_Male

Commit message: Doplnen reset
Parts:
- added C1: 10nF, symbol Device:C
Connections:
- net labels added: VDD_1
- net labels removed: +3V3
- wire segments 18 -> 23
Changed lines of the file:
@@
 $EndComp
-Wire Wire Line
-	8000 3850 8850 3850
-Wire Wire Line
-	8000 3750 9200 3750
-Wire Wire Line
-	8000 3650 9550 3650
-Wire Wire Line
-	8000 3550 9900 3550
 Wire Wire Line
 	8850 4250 8850 3850
@@
 Text HLabel 7150 3350 0    50   Input ~ 0
 EN1
-Text HLabel 7150 3650 0    50   Input ~ 0
-PDN_1
 $Comp
 L power:GND #PWR0109
@@
 Wire Wire Line
 	9900 4550 9900 4650
+Text HLabel 7500 2850 1    50   Input ~ 0
+INDEX_1
 $Comp
-L power:GND #PWR0107
-U 1 1 6024BF79
-P 8000 4050
-F 0 "#PWR0107" H 8000 3800 50  0001 C CNN
-F 1 "GND" V 8000 3850 50  0000 C CNN
-F 2 "" H 8000 4050 50  0001 C CNN
-F 3 "" H 8000 4050 50  0001 C CNN
-	1    8000 4050
-	0    -1   -1   0
+L Device:C C1
+U 1 1 601DF858
+P 8100 4100
+F 0 "C1" H 8215 4146 50  0000 L CNN
+F 1 "10nF" H 8215 4055 50  0000 L CNN
+F 2 "" H 8138 3950 50  0001 C CNN
+F 3 "~" H 8100 4100 50  0001 C CNN
+	1    8100 4100
+	1    0    0    -1
 $EndComp
-$Comp
-L power:+3V3 #PWR0112
-U 1 1 6024C39B
-P 8000 3950
-F 0 "#PWR0112" H 8000 3800 50  0001 C CNN
-F 1 "+3V3" V 8015 4078 50  0000 L CNN
-F 2 "" H 8000 3950 50  0001 C CNN
-F 3 "" H 8000 3950 50  0001 C CNN
-	1    8000 3950
-	0    1    1    0
-$EndComp
-$Comp
-L power:GND #PWR0113
-U 1 1 60253955
-P 8000 3450
-F 0 "#PWR0113" H 8000 3200 50  0001 C CNN
-F 1 "GND" V 8005 3322 50  0000 R CNN
-F 2 "" H 8000 3450 50  0001 C CNN
-F 3 "" H 8000 3450 50  0001 C CNN
-	1    8000 3450
-	0    -1   -1   0
-$EndComp
-$Comp
-L power:+10V #PWR0114
-U 1 1 60254170
-P 8000 3350
-F 0 "#PWR0114" H 8000 3200 50  0001 C CNN
-F 1 "+10V" V 8015 3478 50  0000 L CNN
-F 2 "" H 8000 3350 50  0001 C CNN
-F 3 "" H 8000 3350 50  0001 C CNN
-	1    8000 3350
-	0    1    1    0
-$EndComp
+Text HLabel 7150 3650 0    50   Input ~ 0
+PDN_1
+NoConn ~ 7150 4050
+NoConn ~ 7150 3950
+NoConn ~ 7150 3850
 Wire Wire Line
 	7150 3750 7150 3650
-NoConn ~ 7150 3850
 $Comp
 L power:GND #PWR0126
@@
 	0    1    1    0
 $EndComp
+NoConn ~ 7600 2950
+Wire Wire Line
+	7500 2950 7500 2850
 NoConn ~ 7400 2950
-NoConn ~ 7600 2950
-Text HLabel 7500 2850 1    50   Input ~ 0
-INDEX_1
+$Comp
+L power:+10V #PWR0114
+U 1 1 60254170
+P 8000 3350
+F 0 "#PWR0114" H 8000 3200 50  0001 C CNN
+F 1 "+10V" V 8015 3478 50  0000 L CNN
+F 2 "" H 8000 3350 50  0001 C CNN
+F 3 "" H 8000 3350 50  0001 C CNN
+	1    8000 3350
+	0    1    1    0
+$EndComp
+$Comp
+L power:GND #PWR0113
+U 1 1 60253955
+P 8000 3450
+F 0 "#PWR0113" H 8000 3200 50  0001 C CNN
+F 1 "GND" V 8005 3322 50  0000 R CNN
+F 2 "" H 8000 3450 50  0001 C CNN
+F 3 "" H 8000 3450 50  0001 C CNN
+	1    8000 3450
+	0    -1   -1   0
+$EndComp
+Wire Wire Line
+	8000 3550 9900 3550
+Wire Wire Line
+	8000 3650 9550 3650
+Wire Wire Line
+	8000 3750 9200 3750
+Wire Wire Line
+	8000 3850 8850 3850
 $Comp
 L Základní-deska-II-rescue:TMC2209BreaoutBoard-Tmc2209BreakoutBoard 2209Br1
@@
 	1    0    0    -1
 $EndComp
+$Comp
+L power:GND #PWR0107
+U 1 1 6024BF79
+P 8150 4250
+F 0 "#PWR0107" H 8150 4000 50  0001 C CNN
+F 1 "GND" V 8150 4050 50  0000 C CNN
+F 2 "" H 8150 4250 50  0001 C CNN
+F 3 "" H 8150 4250 50  0001 C CNN
+	1    8150 4250
+	0    -1   -1   0
+$EndComp
 Wire Wire Line
-	7500 2950 7500 2850
-NoConn ~ 7150 3950
-NoConn ~ 7150 4050
+	8000 3950 8100 3950
+Wire Wire Line
+	8000 4050 8000 4250
+Wire Wire Line
+	8000 4250 8100 4250
+Wire Wire Line
+	8100 4250 8150 4250
+Connection ~ 8100 4250
+Text HLabel 8300 3950 2    50   Input ~ 0
+VDD_1
+Wire Wire Line
+	8100 3950 8300 3950
+Connection ~ 8100 3950
 $EndSCHEMATC

Commit message: Jirka upravy
Parts:
- removed C2, C3, C4, C5: 470pF, symbol Device:C
- added R? (x2): 1k, symbol Device:R
- C1: value 10nF -> 100nF
Connections:
- wire segments 23 -> 11
Changed lines of the file:
@@
 $EndDescr
-$Comp
-L Device:C C2
-U 1 1 601E9834
-P 8850 4400
-F 0 "C2" H 8965 4446 50  0000 L CNN
-F 1 "470pF" H 8965 4355 50  0000 L CNN
-F 2 "" H 8888 4250 50  0001 C CNN
-F 3 "~" H 8850 4400 50  0001 C CNN
-	1    8850 4400
-	1    0    0    -1
-$EndComp
-$Comp
-L Device:C C4
-U 1 1 601EAB50
-P 9550 4400
-F 0 "C4" H 9665 4446 50  0000 L CNN
-F 1 "470pF" H 9665 4355 50  0000 L CNN
-F 2 "" H 9588 4250 50  0001 C CNN
-F 3 "~" H 9550 4400 50  0001 C CNN
-	1    9550 4400
-	1    0    0    -1
-$EndComp
-$Comp
-L Device:C C5
-U 1 1 601EAE47
-P 9900 4400
-F 0 "C5" H 10015 4446 50  0000 L CNN
-F 1 "470pF" H 10015 4355 50  0000 L CNN
-F 2 "" H 9938 4250 50  0001 C CNN
-F 3 "~" H 9900 4400 50  0001 C CNN
-	1    9900 4400
-	1    0    0    -1
-$EndComp
 $Comp
 L Connector:Conn_01x04_Male J7
@@
 	-1   0    0    1
 $EndComp
-Wire Wire Line
-	8850 4250 8850 3850
-Connection ~ 8850 3850
-Wire Wire Line
-	8850 3850 10000 3850
-Connection ~ 9200 3750
-Wire Wire Line
-	9200 3750 10000 3750
-Wire Wire Line
-	9550 4250 9550 3650
-Connection ~ 9550 3650
-Wire Wire Line
-	9550 3650 10000 3650
-Wire Wire Line
-	9900 4250 9900 3550
-Connection ~ 9900 3550
-Wire Wire Line
-	9900 3550 10000 3550
-$Comp
-L power:GND #PWR018
-U 1 1 601F09F4
-P 8850 4650
-F 0 "#PWR018" H 8850 4400 50  0001 C CNN
-F 1 "GND" H 8855 4477 50  0000 C CNN
-F 2 "" H 8850 4650 50  0001 C CNN
-F 3 "" H 8850 4650 50  0001 C CNN
-	1    8850 4650
-	1    0    0    -1
-$EndComp
-Wire Wire Line
-	8850 4550 8850 4650
-Wire Wire Line
-	9200 4250 9200 3750
-$Comp
-L Device:C C3
-U 1 1 601EA13D
-P 9200 4400
-F 0 "C3" H 9315 4446 50  0000 L CNN
-F 1 "470pF" H 9315 4355 50  0000 L CNN
-F 2 "" H 9238 4250 50  0001 C CNN
-F 3 "~" H 9200 4400 50  0001 C CNN
-	1    9200 4400
-	1    0    0    -1
-$EndComp
 Text HLabel 7150 3350 0    50   Input ~ 0
 EN1
-$Comp
-L power:GND #PWR0109
-U 1 1 60244E14
-P 9200 4650
-F 0 "#PWR0109" H 9200 4400 50  0001 C CNN
-F 1 "GND" H 9205 4477 50  0000 C CNN
-F 2 "" H 9200 4650 50  0001 C CNN
-F 3 "" H 9200 4650 50  0001 C CNN
-	1    9200 4650
-	1    0    0    -1
-$EndComp
-Wire Wire Line
-	9200 4650 9200 4550
-$Comp
-L power:GND #PWR0110
-U 1 1 6024567B
-P 9550 4650
-F 0 "#PWR0110" H 9550 4400 50  0001 C CNN
-F 1 "GND" H 9555 4477 50  0000 C CNN
-F 2 "" H 9550 4650 50  0001 C CNN
-F 3 "" H 9550 4650 50  0001 C CNN
-	1    9550 4650
-	1    0    0    -1
-$EndComp
-Wire Wire Line
-	9550 4550 9550 4650
-$Comp
-L power:GND #PWR0111
-U 1 1 6024653E
-P 9900 4650
-F 0 "#PWR0111" H 9900 4400 50  0001 C CNN
-F 1 "GND" H 9905 4477 50  0000 C CNN
-F 2 "" H 9900 4650 50  0001 C CNN
-F 3 "" H 9900 4650 50  0001 C CNN
-	1    9900 4650
-	1    0    0    -1
-$EndComp
-Wire Wire Line
-	9900 4550 9900 4650
 Text HLabel 7500 2850 1    50   Input ~ 0
 INDEX_1
@@
 P 8100 4100
 F 0 "C1" H 8215 4146 50  0000 L CNN
-F 1 "10nF" H 8215 4055 50  0000 L CNN
+F 1 "100nF" H 8215 4055 50  0000 L CNN
 F 2 "" H 8138 3950 50  0001 C CNN
 F 3 "~" H 8100 4100 50  0001 C CNN
@@
 L power:GND #PWR0126
 U 1 1 60256C31
-P 7150 3550
-F 0 "#PWR0126" H 7150 3300 50  0001 C CNN
-F 1 "GND" V 7155 3422 50  0000 R CNN
-F 2 "" H 7150 3550 50  0001 C CNN
-F 3 "" H 7150 3550 50  0001 C CNN
-	1    7150 3550
+P 6850 3550
+F 0 "#PWR0126" H 6850 3300 50  0001 C CNN
+F 1 "GND" V 6855 3422 50  0000 R CNN
+F 2 "" H 6850 3550 50  0001 C CNN
+F 3 "" H 6850 3550 50  0001 C CNN
+	1    6850 3550
 	0    1    1    0
 $EndComp
@@
 L power:GND #PWR0127
 U 1 1 602572F0
-P 7150 3450
-F 0 "#PWR0127" H 7150 3200 50  0001 C CNN
-F 1 "GND" V 7155 3322 50  0000 R CNN
-F 2 "" H 7150 3450 50  0001 C CNN
-F 3 "" H 7150 3450 50  0001 C CNN
-	1    7150 3450
+P 6850 3450
+F 0 "#PWR0127" H 6850 3200 50  0001 C CNN
+F 1 "GND" V 6855 3322 50  0000 R CNN
+F 2 "" H 6850 3450 50  0001 C CNN
+F 3 "" H 6850 3450 50  0001 C CNN
+	1    6850 3450
 	0    1    1    0
 $EndComp
@@
 	0    -1   -1   0
 $EndComp
-Wire Wire Line
-	8000 3550 9900 3550
-Wire Wire Line
-	8000 3650 9550 3650
-Wire Wire Line
-	8000 3750 9200 3750
-Wire Wire Line
-	8000 3850 8850 3850
 $Comp
 L Základní-deska-II-rescue:TMC2209BreaoutBoard-Tmc2209BreakoutBoard 2209Br1
@@
 	8100 3950 8300 3950
 Connection ~ 8100 3950
+Wire Wire Line
+	8000 3850 10000 3850
+Wire Wire Line
+	8000 3650 10000 3650
+Wire Wire Line
+	8000 3550 10000 3550
+Wire Wire Line
+	8000 3750 10000 3750
+$Comp
+L Device:R R?
+U 1 1 60259AC4
+P 7000 3450
+F 0 "R?" V 6793 3450 50  0000 C CNN
+F 1 "1k" V 6884 3450 50  0000 C CNN
+F 2 "" V 6930 3450 50  0001 C CNN
+F 3 "~" H 7000 3450 50  0001 C CNN
+	1    7000 3450
+	0    1    1    0
+$EndComp
+$Comp
+L Device:R R?
+U 1 1 6025A673
+P 7000 3550
+F 0 "R?" V 6793 3550 50  0000 C CNN
+F 1 "1k" V 6884 3550 50  0000 C CNN
+F 2 "" V 6930 3550 50  0001 C CNN
+F 3 "~" H 7000 3550 50  0001 C CNN
+	1    7000 3550
+	0    1    1    0
+$EndComp
 $EndSCHEMATC

Commit message: Hotové schéma
Parts:
- removed R? (x2): 1k, symbol Device:R
- 2209Br1: LCSC (none) -> -
- C1: footprint (none) -> Capacitor_SMD:C_0402_1005Metric_Pad0.74x0.62mm_HandSolder; LCSC (none) -> C14663
- J7: footprint (none) -> Connector_PinHeader_2.54mm:PinHeader_1x04_P2.54mm_Vertical; LCSC (none) -> -
Other:
- moved on the sheet: J7
Changed lines of the file:
@@
 L Connector:Conn_01x04_Male J7
 U 1 1 601ECA06
-P 10200 3750
-F 0 "J7" H 10172 3632 50  0000 R CNN
-F 1 "Conn_01x04_Male" H 10172 3723 50  0000 R CNN
-F 2 "" H 10200 3750 50  0001 C CNN
-F 3 "~" H 10200 3750 50  0001 C CNN
-	1    10200 3750
+P 8450 3750
+F 0 "J7" H 8422 3632 50  0000 R CNN
+F 1 "Conn_01x04_Male" H 8422 3723 50  0000 R CNN
+F 2 "Connector_PinHeader_2.54mm:PinHeader_1x04_P2.54mm_Vertical" H 8450 3750 50  0001 C CNN
+F 3 "~" H 8450 3750 50  0001 C CNN
+F 4 "-" H 8450 3750 50  0001 C CNN "LCSC"
+	1    8450 3750
 	-1   0    0    1
 $EndComp
@@
 F 0 "C1" H 8215 4146 50  0000 L CNN
 F 1 "100nF" H 8215 4055 50  0000 L CNN
-F 2 "" H 8138 3950 50  0001 C CNN
+F 2 "Capacitor_SMD:C_0402_1005Metric_Pad0.74x0.62mm_HandSolder" H 8138 3950 50  0001 C CNN
 F 3 "~" H 8100 4100 50  0001 C CNN
+F 4 "C14663" H 8100 4100 50  0001 C CNN "LCSC"
 	1    8100 4100
 	1    0    0    -1
@@
 L power:GND #PWR0126
 U 1 1 60256C31
-P 6850 3550
-F 0 "#PWR0126" H 6850 3300 50  0001 C CNN
-F 1 "GND" V 6855 3422 50  0000 R CNN
-F 2 "" H 6850 3550 50  0001 C CNN
-F 3 "" H 6850 3550 50  0001 C CNN
-	1    6850 3550
+P 7150 3550
+F 0 "#PWR0126" H 7150 3300 50  0001 C CNN
+F 1 "GND" V 7155 3422 50  0000 R CNN
+F 2 "" H 7150 3550 50  0001 C CNN
+F 3 "" H 7150 3550 50  0001 C CNN
+	1    7150 3550
 	0    1    1    0
 $EndComp
@@
 L power:GND #PWR0127
 U 1 1 602572F0
-P 6850 3450
-F 0 "#PWR0127" H 6850 3200 50  0001 C CNN
-F 1 "GND" V 6855 3322 50  0000 R CNN
-F 2 "" H 6850 3450 50  0001 C CNN
-F 3 "" H 6850 3450 50  0001 C CNN
-	1    6850 3450
+P 7150 3450
+F 0 "#PWR0127" H 7150 3200 50  0001 C CNN
+F 1 "GND" V 7155 3322 50  0000 R CNN
+F 2 "" H 7150 3450 50  0001 C CNN
+F 3 "" H 7150 3450 50  0001 C CNN
+	1    7150 3450
 	0    1    1    0
 $EndComp
@@
 F 2 "" H 7350 3600 50  0001 C CNN
 F 3 "" H 7350 3600 50  0001 C CNN
+F 4 "-" H 7600 3600 50  0001 C CNN "LCSC"
 	1    7600 3600
 	1    0    0    -1
@@
 Connection ~ 8100 3950
 Wire Wire Line
-	8000 3850 10000 3850
+	8000 3850 8250 3850
 Wire Wire Line
-	8000 3650 10000 3650
+	8000 3650 8250 3650
 Wire Wire Line
-	8000 3550 10000 3550
+	8000 3550 8250 3550
 Wire Wire Line
-	8000 3750 10000 3750
-$Comp
-L Device:R R?
-U 1 1 60259AC4
-P 7000 3450
-F 0 "R?" V 6793 3450 50  0000 C CNN
-F 1 "1k" V 6884 3450 50  0000 C CNN
-F 2 "" V 6930 3450 50  0001 C CNN
-F 3 "~" H 7000 3450 50  0001 C CNN
-	1    7000 3450
-	0    1    1    0
-$EndComp
-$Comp
-L Device:R R?
-U 1 1 6025A673
-P 7000 3550
-F 0 "R?" V 6793 3550 50  0000 C CNN
-F 1 "1k" V 6884 3550 50  0000 C CNN
-F 2 "" V 6930 3550 50  0001 C CNN
-F 3 "~" H 7000 3550 50  0001 C CNN
-	1    7000 3550
-	0    1    1    0
-$EndComp
+	8000 3750 8250 3750
 $EndSCHEMATC

Commit message: Hotová deska
Parts:
- 2209Br1: footprint (none) -> FinalExamThesis:TMC_2209_Breaout_Board
Changed lines of the file:
@@
 F 0 "2209Br1" H 7575 3027 50  0000 C CNN
 F 1 "TMC2209BreaoutBoard" H 7575 2936 50  0000 C CNN
-F 2 "" H 7350 3600 50  0001 C CNN
+F 2 "FinalExamThesis:TMC_2209_Breaout_Board" H 7350 3600 50  0001 C CNN
 F 3 "" H 7350 3600 50  0001 C CNN
 F 4 "-" H 7600 3600 50  0001 C CNN "LCSC"

Commit message: Nová Deska
Parts:
- added C3: 2,2mF, Capacitor_THT:CP_Radial_D10.0mm_P2.50mm, symbol Device:C
- 2209Br1: symbol Základní-deska-II-rescue:TMC2209BreaoutBoard-Tmc2209BreakoutBoard -> Základní-deska-II-rescue:TMC2209BreaoutBoard-Tmc2209BreakoutBoard-Základní-deska-II-rescue
Connections:
- wire segments 11 -> 15
Changed lines of the file:
@@
 L power:+10V #PWR0114
 U 1 1 60254170
-P 8000 3350
-F 0 "#PWR0114" H 8000 3200 50  0001 C CNN
-F 1 "+10V" V 8015 3478 50  0000 L CNN
-F 2 "" H 8000 3350 50  0001 C CNN
-F 3 "" H 8000 3350 50  0001 C CNN
-	1    8000 3350
+P 8200 3200
+F 0 "#PWR0114" H 8200 3050 50  0001 C CNN
+F 1 "+10V" V 8215 3328 50  0000 L CNN
+F 2 "" H 8200 3200 50  0001 C CNN
+F 3 "" H 8200 3200 50  0001 C CNN
+	1    8200 3200
 	0    1    1    0
 $EndComp
@@
 L power:GND #PWR0113
 U 1 1 60253955
-P 8000 3450
-F 0 "#PWR0113" H 8000 3200 50  0001 C CNN
-F 1 "GND" V 8005 3322 50  0000 R CNN
-F 2 "" H 8000 3450 50  0001 C CNN
-F 3 "" H 8000 3450 50  0001 C CNN
-	1    8000 3450
+P 8200 3500
+F 0 "#PWR0113" H 8200 3250 50  0001 C CNN
+F 1 "GND" V 8205 3372 50  0000 R CNN
+F 2 "" H 8200 3500 50  0001 C CNN
+F 3 "" H 8200 3500 50  0001 C CNN
+	1    8200 3500
 	0    -1   -1   0
 $EndComp
 $Comp
-L Základní-deska-II-rescue:TMC2209BreaoutBoard-Tmc2209BreakoutBoard 2209Br1
+L Základní-deska-II-rescue:TMC2209BreaoutBoard-Tmc2209BreakoutBoard-Základní-deska-II-rescue 2209Br1
 U 1 1 601F591C
 P 7600 3600
@@
 Wire Wire Line
 	8000 3750 8250 3750
+$Comp
+L Device:C C3
+U 1 1 602B2D07
+P 8200 3350
+F 0 "C3" H 8315 3396 50  0000 L CNN
+F 1 "2,2mF" H 8315 3305 50  0000 L CNN
+F 2 "Capacitor_THT:CP_Radial_D10.0mm_P2.50mm" H 8238 3200 50  0001 C CNN
+F 3 "~" H 8200 3350 50  0001 C CNN
+F 4 "C138489" H 8200 3350 50  0001 C CNN "LCSC"
+	1    8200 3350
+	1    0    0    -1
+$EndComp
+Wire Wire Line
+	8200 3500 8000 3500
+Wire Wire Line
+	8000 3500 8000 3450
+Connection ~ 8200 3500
+Wire Wire Line
+	8000 3350 8000 3200
+Wire Wire Line
+	8000 3200 8200 3200
+Connection ~ 8200 3200
 $EndSCHEMATC

Commit message: Deska 1.1
Parts:
- C3: value 2,2mF -> 470uF; LCSC C138489 -> C34642
Changed lines of the file:
@@
 P 8200 3350
 F 0 "C3" H 8315 3396 50  0000 L CNN
-F 1 "2,2mF" H 8315 3305 50  0000 L CNN
+F 1 "470uF" H 8315 3305 50  0000 L CNN
 F 2 "Capacitor_THT:CP_Radial_D10.0mm_P2.50mm" H 8238 3200 50  0001 C CNN
 F 3 "~" H 8200 3350 50  0001 C CNN
-F 4 "C138489" H 8200 3350 50  0001 C CNN "LCSC"
+F 4 "C34642" H 8200 3350 50  0001 C CNN "LCSC"
 	1    8200 3350
 	1    0    0    -1

Commit message: release candidate
Parts:
- C1: LCSC C14663 -> C1525
Changed lines of the file:
@@
 F 2 "Capacitor_SMD:C_0402_1005Metric_Pad0.74x0.62mm_HandSolder" H 8138 3950 50  0001 C CNN
 F 3 "~" H 8100 4100 50  0001 C CNN
-F 4 "C14663" H 8100 4100 50  0001 C CNN "LCSC"
+F 4 "C1525" H 8100 4100 50  0001 C CNN "LCSC"
 	1    8100 4100
 	1    0    0    -1

Commit message: Ordered
Parts:
- 2209Br1: symbol Základní-deska-II-rescue:TMC2209BreaoutBoard-Tmc2209BreakoutBoard-Základní-deska-II-rescue -> Zakladni_deska_II-rescue:TMC2209BreaoutBoard; JLCPCB_IGNORE (none) -> 1
- J7: JLCPCB_IGNORE (none) -> 1
Changed lines of the file:
@@
 F 3 "~" H 8450 3750 50  0001 C CNN
 F 4 "-" H 8450 3750 50  0001 C CNN "LCSC"
+F 5 "1" H 8450 3750 50  0001 C CNN "JLCPCB_IGNORE"
 	1    8450 3750
 	-1   0    0    1
@@
 $EndComp
 $Comp
-L Základní-deska-II-rescue:TMC2209BreaoutBoard-Tmc2209BreakoutBoard-Základní-deska-II-rescue 2209Br1
+L Zakladni_deska_II-rescue:TMC2209BreaoutBoard 2209Br1
 U 1 1 601F591C
 P 7600 3600
@@
 F 3 "" H 7350 3600 50  0001 C CNN
 F 4 "-" H 7600 3600 50  0001 C CNN "LCSC"
+F 5 "1" H 7600 3600 50  0001 C CNN "JLCPCB_IGNORE"
 	1    7600 3600
 	1    0    0    -1
