File: Krokovka2.sch (KiCad schematic (older format))
At the start: 9 parts, among them J10 Conn_01x01_Female, J12 Conn_01x02_Female, J13 Conn_01x08_Female, J14 Conn_01x04_Male, J8 Conn_01x08_Female

Commit message: Deska 0.5
Parts:
- removed J10: Conn_01x01_Female, symbol Connector:Conn_01x01_Female
- removed J12: Conn_01x02_Female, symbol Connector:Conn_01x02_Female
- removed J13, J8: Conn_01x08_Female, symbol Connector:Conn_01x08_Female
- added 2209Br2: TMC2209BreaoutBoard, symbol Tmc2209BreakoutBoard:TMC2209BreaoutBoard
Connections:
- net labels removed: A1, A2, B1, B2, CLK, DIAG, DIR, EN, INDEX, MS1, MS2, PDN_UART, STEP, VCC, VDD, VM, VREF
- wire segments 33 -> 17
Other:
- moved on the sheet: C6, C7, C8, C9, J14
