File: Krokovka2.sch (KiCad schematic (older format))
At the start: 6 parts, among them J14 Conn_01x04_Male

Commit message: Doplnen reset
Parts:
- added C?: 10nF, symbol Device:C
Connections:
- net labels added: VDD_2
- wire segments 17 -> 22
Changed lines of the file:
@@
 	6050 4300 6050 4200
-$Comp
-L power:+3V3 #PWR05
-U 1 1 6026F14F
-P 6900 4500
-F 0 "#PWR05" H 6900 4350 50  0001 C CNN
-F 1 "+3V3" V 6915 4628 50  0000 L CNN
-F 2 "" H 6900 4500 50  0001 C CNN
-F 3 "" H 6900 4500 50  0001 C CNN
-	1    6900 4500
-	0    1    1    0
-$EndComp
 $Comp
 L power:GND #PWR?
 U 1 1 60270539
-P 6900 4600
+P 7250 4800
 AR Path="/601BF914/60270539" Ref="#PWR?"  Part="1"
 AR Path="/601E7BA1/60270539" Ref="#PWR010"  Part="1"
-F 0 "#PWR010" H 6900 4350 50  0001 C CNN
-F 1 "GND" V 6905 4472 50  0000 R CNN
-F 2 "" H 6900 4600 50  0001 C CNN
-F 3 "" H 6900 4600 50  0001 C CNN
-	1    6900 4600
+F 0 "#PWR010" H 7250 4550 50  0001 C CNN
+F 1 "GND" V 7255 4672 50  0000 R CNN
+F 2 "" H 7250 4800 50  0001 C CNN
+F 3 "" H 7250 4800 50  0001 C CNN
+	1    7250 4800
 	0    -1   -1   0
 $EndComp
@@
 NoConn ~ 6050 4500
 NoConn ~ 6050 4600
+$Comp
+L Device:C C?
+U 1 1 6023D6D9
+P 7050 4650
+F 0 "C?" H 7165 4696 50  0000 L CNN
+F 1 "10nF" H 7165 4605 50  0000 L CNN
+F 2 "" H 7088 4500 50  0001 C CNN
+F 3 "~" H 7050 4650 50  0001 C CNN
+	1    7050 4650
+	1    0    0    -1
+$EndComp
+Wire Wire Line
+	6900 4500 7050 4500
+Wire Wire Line
+	7050 4500 7250 4500
+Connection ~ 7050 4500
+Wire Wire Line
+	6900 4600 6900 4800
+Wire Wire Line
+	6900 4800 7050 4800
+Wire Wire Line
+	7250 4800 7050 4800
+Connection ~ 7050 4800
+Text HLabel 7250 4500 2    50   Input ~ 0
+VDD_2
 $EndSCHEMATC

Commit message: Mosfet
Parts:
- gave numbers to parts that had none: 1
Changed lines of the file:
@@
 NoConn ~ 6050 4600
 $Comp
-L Device:C C?
+L Device:C C18
 U 1 1 6023D6D9
 P 7050 4650
-F 0 "C?" H 7165 4696 50  0000 L CNN
+F 0 "C18" H 7165 4696 50  0000 L CNN
 F 1 "10nF" H 7165 4605 50  0000 L CNN
 F 2 "" H 7088 4500 50  0001 C CNN

Commit message: Jirka upravy
Parts:
- removed C6, C7, C8, C9: 470pF, symbol Device:C
- added R? (x2): 1k, symbol Device:R
- C18: value 10nF -> 100nF
Connections:
- wire segments 22 -> 10
Changed lines of the file:
@@
 $EndDescr
-$Comp
-L Device:C C?
-U 1 1 6020C1DD
-P 7750 4950
-AR Path="/601BF914/6020C1DD" Ref="C?"  Part="1"
-AR Path="/601E7BA1/6020C1DD" Ref="C6"  Part="1"
-F 0 "C6" H 7865 4996 50  0000 L CNN
-F 1 "470pF" H 7865 4905 50  0000 L CNN
-F 2 "" H 7788 4800 50  0001 C CNN
-F 3 "~" H 7750 4950 50  0001 C CNN
-	1    7750 4950
-	1    0    0    -1
-$EndComp
-$Comp
-L Device:C C?
-U 1 1 6020C1E3
-P 8450 4950
-AR Path="/601BF914/6020C1E3" Ref="C?"  Part="1"
-AR Path="/601E7BA1/6020C1E3" Ref="C8"  Part="1"
-F 0 "C8" H 8565 4996 50  0000 L CNN
-F 1 "470pF" H 8565 4905 50  0000 L CNN
-F 2 "" H 8488 4800 50  0001 C CNN
-F 3 "~" H 8450 4950 50  0001 C CNN
-	1    8450 4950
-	1    0    0    -1
-$EndComp
-$Comp
-L Device:C C?
-U 1 1 6020C1E9
-P 8800 4950
-AR Path="/601BF914/6020C1E9" Ref="C?"  Part="1"
-AR Path="/601E7BA1/6020C1E9" Ref="C9"  Part="1"
-F 0 "C9" H 8915 4996 50  0000 L CNN
-F 1 "470pF" H 8915 4905 50  0000 L CNN
-F 2 "" H 8838 4800 50  0001 C CNN
-F 3 "~" H 8800 4950 50  0001 C CNN
-	1    8800 4950
-	1    0    0    -1
-$EndComp
 $Comp
 L Connector:Conn_01x04_Male J?
@@
 	1    9100 4300
 	-1   0    0    1
-$EndComp
-Wire Wire Line
-	6900 4400 7750 4400
-Wire Wire Line
-	6900 4300 8100 4300
-Wire Wire Line
-	6900 4200 8450 4200
-Wire Wire Line
-	6900 4100 8800 4100
-Wire Wire Line
-	7750 4800 7750 4400
-Connection ~ 7750 4400
-Wire Wire Line
-	7750 4400 8900 4400
-Connection ~ 8100 4300
-Wire Wire Line
-	8100 4300 8900 4300
-Wire Wire Line
-	8450 4800 8450 4200
-Connection ~ 8450 4200
-Wire Wire Line
-	8450 4200 8900 4200
-Wire Wire Line
-	8800 4800 8800 4100
-Connection ~ 8800 4100
-Wire Wire Line
-	8800 4100 8900 4100
-$Comp
-L power:GND #PWR?
-U 1 1 6020C20B
-P 7750 5200
-AR Path="/601BF914/6020C20B" Ref="#PWR?"  Part="1"
-AR Path="/601E7BA1/6020C20B" Ref="#PWR027"  Part="1"
-F 0 "#PWR027" H 7750 4950 50  0001 C CNN
-F 1 "GND" H 7755 5027 50  0000 C CNN
-F 2 "" H 7750 5200 50  0001 C CNN
-F 3 "" H 7750 5200 50  0001 C CNN
-	1    7750 5200
-	1    0    0    -1
-$EndComp
-$Comp
-L power:GND #PWR?
-U 1 1 6020C211
-P 8100 5200
-AR Path="/601BF914/6020C211" Ref="#PWR?"  Part="1"
-AR Path="/601E7BA1/6020C211" Ref="#PWR028"  Part="1"
-F 0 "#PWR028" H 8100 4950 50  0001 C CNN
-F 1 "GND" H 8105 5027 50  0000 C CNN
-F 2 "" H 8100 5200 50  0001 C CNN
-F 3 "" H 8100 5200 50  0001 C CNN
-	1    8100 5200
-	1    0    0    -1
-$EndComp
-$Comp
-L power:GND #PWR?
-U 1 1 6020C217
-P 8450 5200
-AR Path="/601BF914/6020C217" Ref="#PWR?"  Part="1"
-AR Path="/601E7BA1/6020C217" Ref="#PWR029"  Part="1"
-F 0 "#PWR029" H 8450 4950 50  0001 C CNN
-F 1 "GND" H 8455 5027 50  0000 C CNN
-F 2 "" H 8450 5200 50  0001 C CNN
-F 3 "" H 8450 5200 50  0001 C CNN
-	1    8450 5200
-	1    0    0    -1
-$EndComp
-$Comp
-L power:GND #PWR?
-U 1 1 6020C21D
-P 8800 5200
-AR Path="/601BF914/6020C21D" Ref="#PWR?"  Part="1"
-AR Path="/601E7BA1/6020C21D" Ref="#PWR030"  Part="1"
-F 0 "#PWR030" H 8800 4950 50  0001 C CNN
-F 1 "GND" H 8805 5027 50  0000 C CNN
-F 2 "" H 8800 5200 50  0001 C CNN
-F 3 "" H 8800 5200 50  0001 C CNN
-	1    8800 5200
-	1    0    0    -1
-$EndComp
-Wire Wire Line
-	7750 5100 7750 5200
-Wire Wire Line
-	8450 5100 8450 5200
-Wire Wire Line
-	8800 5100 8800 5200
-Wire Wire Line
-	8100 5100 8100 5200
-Wire Wire Line
-	8100 4800 8100 4300
-$Comp
-L Device:C C?
-U 1 1 6020C228
-P 8100 4950
-AR Path="/601BF914/6020C228" Ref="C?"  Part="1"
-AR Path="/601E7BA1/6020C228" Ref="C7"  Part="1"
-F 0 "C7" H 8215 4996 50  0000 L CNN
-F 1 "470pF" H 8215 4905 50  0000 L CNN
-F 2 "" H 8138 4800 50  0001 C CNN
-F 3 "~" H 8100 4950 50  0001 C CNN
-	1    8100 4950
-	1    0    0    -1
 $EndComp
 Text HLabel 6050 3900 0    50   Input ~ 0
@@
 L power:+3V3 #PWR0115
 U 1 1 601B777E
-P 6050 4000
-F 0 "#PWR0115" H 6050 3850 50  0001 C CNN
-F 1 "+3V3" V 6065 4128 50  0000 L CNN
-F 2 "" H 6050 4000 50  0001 C CNN
-F 3 "" H 6050 4000 50  0001 C CNN
-	1    6050 4000
+P 5750 4000
+F 0 "#PWR0115" H 5750 3850 50  0001 C CNN
+F 1 "+3V3" V 5765 4128 50  0000 L CNN
+F 2 "" H 5750 4000 50  0001 C CNN
+F 3 "" H 5750 4000 50  0001 C CNN
+	1    5750 4000
 	0    -1   -1   0
 $EndComp
@@
 L power:GND #PWR?
 U 1 1 60270903
-P 6050 4100
+P 5750 4100
 AR Path="/601BF914/60270903" Ref="#PWR?"  Part="1"
 AR Path="/601E7BA1/60270903" Ref="#PWR01"  Part="1"
-F 0 "#PWR01" H 6050 3850 50  0001 C CNN
-F 1 "GND" V 6055 3972 50  0000 R CNN
-F 2 "" H 6050 4100 50  0001 C CNN
-F 3 "" H 6050 4100 50  0001 C CNN
-	1    6050 4100
+F 0 "#PWR01" H 5750 3850 50  0001 C CNN
+F 1 "GND" V 5755 3972 50  0000 R CNN
+F 2 "" H 5750 4100 50  0001 C CNN
+F 3 "" H 5750 4100 50  0001 C CNN
+	1    5750 4100
 	0    1    1    0
 $EndComp
@@
 P 7050 4650
 F 0 "C18" H 7165 4696 50  0000 L CNN
-F 1 "10nF" H 7165 4605 50  0000 L CNN
+F 1 "100nF" H 7165 4605 50  0000 L CNN
 F 2 "" H 7088 4500 50  0001 C CNN
 F 3 "~" H 7050 4650 50  0001 C CNN
@@
 Text HLabel 7250 4500 2    50   Input ~ 0
 VDD_2
+Wire Wire Line
+	6900 4400 8900 4400
+Wire Wire Line
+	6900 4200 8900 4200
+Wire Wire Line
+	6900 4100 8900 4100
+Wire Wire Line
+	6900 4300 8900 4300
+$Comp
+L Device:R R?
+U 1 1 602577DF
+P 5900 4000
+F 0 "R?" V 5693 4000 50  0000 C CNN
+F 1 "1k" V 6100 4000 50  0000 C CNN
+F 2 "" V 5830 4000 50  0001 C CNN
+F 3 "~" H 5900 4000 50  0001 C CNN
+	1    5900 4000
+	0    1    1    0
+$EndComp
+$Comp
+L Device:R R?
+U 1 1 60258476
+P 5900 4100
+F 0 "R?" V 6050 4100 50  0000 C CNN
+F 1 "1k" V 5784 4100 50  0000 C CNN
+F 2 "" V 5830 4100 50  0001 C CNN
+F 3 "~" H 5900 4100 50  0001 C CNN
+	1    5900 4100
+	0    1    1    0
+$EndComp
 $EndSCHEMATC

Commit message: Hotové schéma
Parts:
- removed R?: 1k, symbol Device:R
- 2209Br2: LCSC (none) -> -
- C18: footprint (none) -> Capacitor_SMD:C_0402_1005Metric_Pad0.74x0.62mm_HandSolder; LCSC (none) -> C14663
- J14: footprint (none) -> Connector_PinHeader_2.54mm:PinHeader_1x04_P2.54mm_Vertical; LCSC (none) -> -
- R11: renamed from R?; footprint (none) -> Resistor_SMD:R_0805_2012Metric_Pad1.20x1.40mm_HandSolder; LCSC (none) -> C17513
Connections:
- wire segments 10 -> 14
Other:
- moved on the sheet: J14, R11
Changed lines of the file:
@@
 Comment4 ""
 $EndDescr
-$Comp
-L Connector:Conn_01x04_Male J?
-U 1 1 6020C1EF
-P 9100 4300
-AR Path="/601BF914/6020C1EF" Ref="J?"  Part="1"
-AR Path="/601E7BA1/6020C1EF" Ref="J14"  Part="1"
-F 0 "J14" H 9072 4182 50  0000 R CNN
-F 1 "Conn_01x04_Male" H 9072 4273 50  0000 R CNN
-F 2 "" H 9100 4300 50  0001 C CNN
-F 3 "~" H 9100 4300 50  0001 C CNN
-	1    9100 4300
-	-1   0    0    1
-$EndComp
 Text HLabel 6050 3900 0    50   Input ~ 0
 EN2
-Text HLabel 6050 4300 0    50   Input ~ 0
-PDN_2
-$Comp
-L power:GND #PWR?
-U 1 1 6020C23F
-P 6900 4000
-AR Path="/601BF914/6020C23F" Ref="#PWR?"  Part="1"
-AR Path="/601E7BA1/6020C23F" Ref="#PWR025"  Part="1"
-F 0 "#PWR025" H 6900 3750 50  0001 C CNN
-F 1 "GND" V 6905 3872 50  0000 R CNN
-F 2 "" H 6900 4000 50  0001 C CNN
-F 3 "" H 6900 4000 50  0001 C CNN
-	1    6900 4000
-	0    -1   -1   0
-$EndComp
-$Comp
-L power:+10V #PWR0117
-U 1 1 601A68DF
-P 6900 3900
-F 0 "#PWR0117" H 6900 3750 50  0001 C CNN
-F 1 "+10V" V 6915 4028 50  0000 L CNN
-F 2 "" H 6900 3900 50  0001 C CNN
-F 3 "" H 6900 3900 50  0001 C CNN
-	1    6900 3900
-	0    1    1    0
-$EndComp
 Text HLabel 6400 3500 1    50   Input ~ 0
 INDEX_2
-$Comp
-L power:+3V3 #PWR0115
-U 1 1 601B777E
-P 5750 4000
-F 0 "#PWR0115" H 5750 3850 50  0001 C CNN
-F 1 "+3V3" V 5765 4128 50  0000 L CNN
-F 2 "" H 5750 4000 50  0001 C CNN
-F 3 "" H 5750 4000 50  0001 C CNN
-	1    5750 4000
-	0    -1   -1   0
-$EndComp
-$Comp
-L Základní-deska-II-rescue:TMC2209BreaoutBoard-Tmc2209BreakoutBoard 2209Br2
-U 1 1 60267626
-P 6500 4150
-F 0 "2209Br2" H 6475 3577 50  0000 C CNN
-F 1 "TMC2209BreaoutBoard" H 6475 3486 50  0000 C CNN
-F 2 "" H 6250 4150 50  0001 C CNN
-F 3 "" H 6250 4150 50  0001 C CNN
-	1    6500 4150
-	1    0    0    -1
-$EndComp
-NoConn ~ 6300 3500
-NoConn ~ 6500 3500
-NoConn ~ 6050 4400
-Wire Wire Line
-	6050 4300 6050 4200
 $Comp
 L power:GND #PWR?
@@
 L power:GND #PWR?
 U 1 1 60270903
-P 5750 4100
+P 5300 4100
 AR Path="/601BF914/60270903" Ref="#PWR?"  Part="1"
 AR Path="/601E7BA1/60270903" Ref="#PWR01"  Part="1"
-F 0 "#PWR01" H 5750 3850 50  0001 C CNN
-F 1 "GND" V 5755 3972 50  0000 R CNN
-F 2 "" H 5750 4100 50  0001 C CNN
-F 3 "" H 5750 4100 50  0001 C CNN
-	1    5750 4100
+F 0 "#PWR01" H 5300 3850 50  0001 C CNN
+F 1 "GND" V 5305 3972 50  0000 R CNN
+F 2 "" H 5300 4100 50  0001 C CNN
+F 3 "" H 5300 4100 50  0001 C CNN
+	1    5300 4100
 	0    1    1    0
 $EndComp
-NoConn ~ 6050 4500
-NoConn ~ 6050 4600
 $Comp
 L Device:C C18
@@
 F 0 "C18" H 7165 4696 50  0000 L CNN
 F 1 "100nF" H 7165 4605 50  0000 L CNN
-F 2 "" H 7088 4500 50  0001 C CNN
+F 2 "Capacitor_SMD:C_0402_1005Metric_Pad0.74x0.62mm_HandSolder" H 7088 4500 50  0001 C CNN
 F 3 "~" H 7050 4650 50  0001 C CNN
+F 4 "C14663" H 7050 4650 50  0001 C CNN "LCSC"
 	1    7050 4650
 	1    0    0    -1
 $EndComp
 Wire Wire Line
-	6900 4500 7050 4500
-Wire Wire Line
 	7050 4500 7250 4500
 Connection ~ 7050 4500
-Wire Wire Line
-	6900 4600 6900 4800
 Wire Wire Line
 	6900 4800 7050 4800
@@
 Text HLabel 7250 4500 2    50   Input ~ 0
 VDD_2
+$Comp
+L Connector:Conn_01x04_Male J?
+U 1 1 6020C1EF
+P 7450 4300
+AR Path="/601BF914/6020C1EF" Ref="J?"  Part="1"
+AR Path="/601E7BA1/6020C1EF" Ref="J14"  Part="1"
+F 0 "J14" H 7422 4182 50  0000 R CNN
+F 1 "Conn_01x04_Male" H 7422 4273 50  0000 R CNN
+F 2 "Connector_PinHeader_2.54mm:PinHeader_1x04_P2.54mm_Vertical" H 7450 4300 50  0001 C CNN
+F 3 "~" H 7450 4300 50  0001 C CNN
+F 4 "-" H 7450 4300 50  0001 C CNN "LCSC"
+	1    7450 4300
+	-1   0    0    1
+$EndComp
+$Comp
+L power:+3V3 #PWR0115
+U 1 1 601B777E
+P 5300 4000
+F 0 "#PWR0115" H 5300 3850 50  0001 C CNN
+F 1 "+3V3" V 5315 4128 50  0000 L CNN
+F 2 "" H 5300 4000 50  0001 C CNN
+F 3 "" H 5300 4000 50  0001 C CNN
+	1    5300 4000
+	0    -1   -1   0
+$EndComp
+Text HLabel 6050 4300 0    50   Input ~ 0
+PDN_2
 Wire Wire Line
-	6900 4400 8900 4400
+	6900 4600 6900 4800
+NoConn ~ 6050 4600
+NoConn ~ 6050 4500
+NoConn ~ 6050 4400
 Wire Wire Line
-	6900 4200 8900 4200
+	6050 4300 6050 4200
 Wire Wire Line
-	6900 4100 8900 4100
-Wire Wire Line
-	6900 4300 8900 4300
+	5300 4100 6050 4100
+NoConn ~ 6500 3500
+NoConn ~ 6300 3500
 $Comp
-L Device:R R?
-U 1 1 602577DF
-P 5900 4000
-F 0 "R?" V 5693 4000 50  0000 C CNN
-F 1 "1k" V 6100 4000 50  0000 C CNN
-F 2 "" V 5830 4000 50  0001 C CNN
-F 3 "~" H 5900 4000 50  0001 C CNN
-	1    5900 4000
+L power:+10V #PWR0117
+U 1 1 601A68DF
+P 6900 3900
+F 0 "#PWR0117" H 6900 3750 50  0001 C CNN
+F 1 "+10V" V 6915 4028 50  0000 L CNN
+F 2 "" H 6900 3900 50  0001 C CNN
+F 3 "" H 6900 3900 50  0001 C CNN
+	1    6900 3900
 	0    1    1    0
 $EndComp
 $Comp
-L Device:R R?
-U 1 1 60258476
-P 5900 4100
-F 0 "R?" V 6050 4100 50  0000 C CNN
-F 1 "1k" V 5784 4100 50  0000 C CNN
-F 2 "" V 5830 4100 50  0001 C CNN
-F 3 "~" H 5900 4100 50  0001 C CNN
-	1    5900 4100
+L power:GND #PWR?
+U 1 1 6020C23F
+P 6900 4000
+AR Path="/601BF914/6020C23F" Ref="#PWR?"  Part="1"
+AR Path="/601E7BA1/6020C23F" Ref="#PWR025"  Part="1"
+F 0 "#PWR025" H 6900 3750 50  0001 C CNN
+F 1 "GND" V 6905 3872 50  0000 R CNN
+F 2 "" H 6900 4000 50  0001 C CNN
+F 3 "" H 6900 4000 50  0001 C CNN
+	1    6900 4000
+	0    -1   -1   0
+$EndComp
+Wire Wire Line
+	6900 4100 7250 4100
+Wire Wire Line
+	6900 4200 7250 4200
+Wire Wire Line
+	6900 4300 7250 4300
+Wire Wire Line
+	6900 4400 7250 4400
+Wire Wire Line
+	6900 4500 7050 4500
+$Comp
+L power:PWR_FLAG #FLG0103
+U 1 1 60227C9E
+P 5800 4000
+F 0 "#FLG0103" H 5800 4075 50  0001 C CNN
+F 1 "PWR_FLAG" H 5800 4173 50  0000 C CNN
+F 2 "" H 5800 4000 50  0001 C CNN
+F 3 "~" H 5800 4000 50  0001 C CNN
+	1    5800 4000
+	1    0    0    -1
+$EndComp
+$Comp
+L Základní-deska-II-rescue:TMC2209BreaoutBoard-Tmc2209BreakoutBoard 2209Br2
+U 1 1 60267626
+P 6500 4150
+F 0 "2209Br2" H 6475 3577 50  0000 C CNN
+F 1 "TMC2209BreaoutBoard" H 6475 3486 50  0000 C CNN
+F 2 "" H 6250 4150 50  0001 C CNN
+F 3 "" H 6250 4150 50  0001 C CNN
+F 4 "-" H 6500 4150 50  0001 C CNN "LCSC"
+	1    6500 4150
+	1    0    0    -1
+$EndComp
+$Comp
+L Device:R R11
+U 1 1 602577DF
+P 5600 4000
+F 0 "R11" V 5500 3850 50  0000 C CNN
+F 1 "1k" V 5600 4000 50  0000 C CNN
+F 2 "Resistor_SMD:R_0805_2012Metric_Pad1.20x1.40mm_HandSolder" V 5530 4000 50  0001 C CNN
+F 3 "~" H 5600 4000 50  0001 C CNN
+F 4 "C17513" H 5600 4000 50  0001 C CNN "LCSC"
+	1    5600 4000
 	0    1    1    0
 $EndComp
+Wire Wire Line
+	6050 4000 5800 4000
+Wire Wire Line
+	5800 4000 5750 4000
+Connection ~ 5800 4000
+Wire Wire Line
+	5450 4000 5300 4000
 $EndSCHEMATC

Commit message: Hotová deska
Parts:
- 2209Br2: footprint (none) -> FinalExamThesis:TMC_2209_Breaout_Board
Changed lines of the file:
@@
 F 0 "2209Br2" H 6475 3577 50  0000 C CNN
 F 1 "TMC2209BreaoutBoard" H 6475 3486 50  0000 C CNN
-F 2 "" H 6250 4150 50  0001 C CNN
+F 2 "FinalExamThesis:TMC_2209_Breaout_Board" H 6250 4150 50  0001 C CNN
 F 3 "" H 6250 4150 50  0001 C CNN
 F 4 "-" H 6500 4150 50  0001 C CNN "LCSC"

Commit message: Jirka
Parts:
- added C2: 300mF - electrolyt, Capacitor_SMD:C_0402_1005Metric_Pad0.74x0.62mm_HandSolder, symbol Device:C
Changed lines of the file:
@@
 Wire Wire Line
 	5450 4000 5300 4000
+$Comp
+L Device:C C2
+U 1 1 60311DC8
+P 7050 3600
+F 0 "C2" H 7165 3646 50  0000 L CNN
+F 1 "300mF - electrolyt" H 7165 3555 50  0000 L CNN
+F 2 "Capacitor_SMD:C_0402_1005Metric_Pad0.74x0.62mm_HandSolder" H 7088 3450 50  0001 C CNN
+F 3 "~" H 7050 3600 50  0001 C CNN
+F 4 "C14663" H 7050 3600 50  0001 C CNN "LCSC"
+	1    7050 3600
+	1    0    0    -1
+$EndComp
 $EndSCHEMATC

Commit message: Nová Deska
Parts:
- 2209Br2: symbol Základní-deska-II-rescue:TMC2209BreaoutBoard-Tmc2209BreakoutBoard -> Základní-deska-II-rescue:TMC2209BreaoutBoard-Tmc2209BreakoutBoard-Základní-deska-II-rescue
- C2: value 300mF - electrolyt -> 2,2mF; footprint Capacitor_SMD:C_0402_1005Metric_Pad0.74x0.62mm_HandSolder -> Capacitor_THT:CP_Radial_D10.0mm_P2.50mm; LCSC C14663 -> C138489
Connections:
- wire segments 14 -> 17
Changed lines of the file:
@@
 L power:+10V #PWR0117
 U 1 1 601A68DF
-P 6900 3900
-F 0 "#PWR0117" H 6900 3750 50  0001 C CNN
-F 1 "+10V" V 6915 4028 50  0000 L CNN
-F 2 "" H 6900 3900 50  0001 C CNN
-F 3 "" H 6900 3900 50  0001 C CNN
-	1    6900 3900
+P 7050 3700
+F 0 "#PWR0117" H 7050 3550 50  0001 C CNN
+F 1 "+10V" V 7065 3828 50  0000 L CNN
+F 2 "" H 7050 3700 50  0001 C CNN
+F 3 "" H 7050 3700 50  0001 C CNN
+	1    7050 3700
 	0    1    1    0
 $EndComp
@@
 L power:GND #PWR?
 U 1 1 6020C23F
-P 6900 4000
+P 7050 4000
 AR Path="/601BF914/6020C23F" Ref="#PWR?"  Part="1"
 AR Path="/601E7BA1/6020C23F" Ref="#PWR025"  Part="1"
-F 0 "#PWR025" H 6900 3750 50  0001 C CNN
-F 1 "GND" V 6905 3872 50  0000 R CNN
-F 2 "" H 6900 4000 50  0001 C CNN
-F 3 "" H 6900 4000 50  0001 C CNN
-	1    6900 4000
+F 0 "#PWR025" H 7050 3750 50  0001 C CNN
+F 1 "GND" V 7055 3872 50  0000 R CNN
+F 2 "" H 7050 4000 50  0001 C CNN
+F 3 "" H 7050 4000 50  0001 C CNN
+	1    7050 4000
 	0    -1   -1   0
 $EndComp
@@
 $EndComp
 $Comp
-L Základní-deska-II-rescue:TMC2209BreaoutBoard-Tmc2209BreakoutBoard 2209Br2
+L Základní-deska-II-rescue:TMC2209BreaoutBoard-Tmc2209BreakoutBoard-Základní-deska-II-rescue 2209Br2
 U 1 1 60267626
 P 6500 4150
@@
 	5450 4000 5300 4000
 $Comp
-L Device:C C2
-U 1 1 60311DC8
-P 7050 3600
-F 0 "C2" H 7165 3646 50  0000 L CNN
-F 1 "300mF - electrolyt" H 7165 3555 50  0000 L CNN
-F 2 "Capacitor_SMD:C_0402_1005Metric_Pad0.74x0.62mm_HandSolder" H 7088 3450 50  0001 C CNN
-F 3 "~" H 7050 3600 50  0001 C CNN
-F 4 "C14663" H 7050 3600 50  0001 C CNN "LCSC"
-	1    7050 3600
+L Device:C C?
+U 1 1 602B60C0
+P 7050 3850
+AR Path="/601BF914/602B60C0" Ref="C?"  Part="1"
+AR Path="/601E7BA1/602B60C0" Ref="C2"  Part="1"
+F 0 "C2" H 7165 3896 50  0000 L CNN
+F 1 "2,2mF" H 7165 3805 50  0000 L CNN
+F 2 "Capacitor_THT:CP_Radial_D10.0mm_P2.50mm" H 7088 3700 50  0001 C CNN
+F 3 "~" H 7050 3850 50  0001 C CNN
+F 4 "C138489" H 7050 3850 50  0001 C CNN "LCSC"
+	1    7050 3850
 	1    0    0    -1
 $EndComp
+Wire Wire Line
+	6900 4000 7050 4000
+Connection ~ 7050 4000
+Wire Wire Line
+	6900 3900 6900 3700
+Wire Wire Line
+	6900 3700 7050 3700
+Connection ~ 7050 3700
 $EndSCHEMATC

Commit message: Deska 1.1
Parts:
- C2: value 2,2mF -> 470uF; LCSC C138489 -> C34642
Changed lines of the file:
@@
 AR Path="/601E7BA1/602B60C0" Ref="C2"  Part="1"
 F 0 "C2" H 7165 3896 50  0000 L CNN
-F 1 "2,2mF" H 7165 3805 50  0000 L CNN
+F 1 "470uF" H 7165 3805 50  0000 L CNN
 F 2 "Capacitor_THT:CP_Radial_D10.0mm_P2.50mm" H 7088 3700 50  0001 C CNN
 F 3 "~" H 7050 3850 50  0001 C CNN
-F 4 "C138489" H 7050 3850 50  0001 C CNN "LCSC"
+F 4 "C34642" H 7050 3850 50  0001 C CNN "LCSC"
 	1    7050 3850
 	1    0    0    -1
