File: Krokovka2.sch (KiCad schematic (older format))
At the start: 5 parts, among them J14 Conn_01x04_Male

Commit message: release candidate
Parts:
- C18: LCSC C14663 -> C1525
Changed lines of the file:
@@
 F 2 "Capacitor_SMD:C_0402_1005Metric_Pad0.74x0.62mm_HandSolder" H 7088 4500 50  0001 C CNN
 F 3 "~" H 7050 4650 50  0001 C CNN
-F 4 "C14663" H 7050 4650 50  0001 C CNN "LCSC"
+F 4 "C1525" H 7050 4650 50  0001 C CNN "LCSC"
 	1    7050 4650
 	1    0    0    -1

Commit message: Ordered
Parts:
- 2209Br2: symbol Základní-deska-II-rescue:TMC2209BreaoutBoard-Tmc2209BreakoutBoard-Základní-deska-II-rescue -> Zakladni_deska_II-rescue:TMC2209BreaoutBoard; JLCPCB_IGNORE (none) -> 1
- J14: JLCPCB_IGNORE (none) -> 1
- R11: LCSC C17513 -> C17379
Changed lines of the file:
@@
 F 3 "~" H 7450 4300 50  0001 C CNN
 F 4 "-" H 7450 4300 50  0001 C CNN "LCSC"
+F 5 "1" H 7450 4300 50  0001 C CNN "JLCPCB_IGNORE"
 	1    7450 4300
 	-1   0    0    1
@@
 $EndComp
 $Comp
-L Základní-deska-II-rescue:TMC2209BreaoutBoard-Tmc2209BreakoutBoard-Základní-deska-II-rescue 2209Br2
+L Zakladni_deska_II-rescue:TMC2209BreaoutBoard 2209Br2
 U 1 1 60267626
 P 6500 4150
@@
 F 3 "" H 6250 4150 50  0001 C CNN
 F 4 "-" H 6500 4150 50  0001 C CNN "LCSC"
+F 5 "1" H 6500 4150 50  0001 C CNN "JLCPCB_IGNORE"
 	1    6500 4150
 	1    0    0    -1
@@
 F 2 "Resistor_SMD:R_0805_2012Metric_Pad1.20x1.40mm_HandSolder" V 5530 4000 50  0001 C CNN
 F 3 "~" H 5600 4000 50  0001 C CNN
-F 4 "C17513" H 5600 4000 50  0001 C CNN "LCSC"
+F 4 "C17379" H 5600 4000 50  0001 C CNN "LCSC"
 	1    5600 4000
 	0    1    1    0
