File: Krokovka3.sch (KiCad schematic (older format))
At the start: 9 parts, among them J15 Conn_01x08_Female, J17 Conn_01x01_Female, J19 Conn_01x02_Female, J20 Conn_01x08_Female, J21 Conn_01x04_Male

Commit message: Deska 0.5
Parts:
- removed J15, J20: Conn_01x08_Female, symbol Connector:Conn_01x08_Female
- removed J17: Conn_01x01_Female, symbol Connector:Conn_01x01_Female
- removed J19: Conn_01x02_Female, symbol Connector:Conn_01x02_Female
- added 2209Br3: TMC2209BreaoutBoard, symbol Tmc2209BreakoutBoard:TMC2209BreaoutBoard
Connections:
- net labels removed: A1, A2, B1, B2, CLK, DIAG, DIR, EN, INDEX, MS1, MS2, PDN_UART, STEP, VCC, VDD, VM, VREF
- wire segments 33 -> 17
Other:
- moved on the sheet: C10, C11, C12, C13, J21
