File: Krokovka3.sch (KiCad schematic (older format))
At the start: 6 parts, among them J21 Conn_01x04_Male

Commit message: Doplnen reset
Parts:
- added C?: 10nF, symbol Device:C
Connections:
- net labels added: VDD_3
- wire segments 17 -> 22
Changed lines of the file:
@@
-$EndComp
-$Comp
-L power:+3V3 #PWR0120
-U 1 1 601B12BE
-P 7700 3050
-F 0 "#PWR0120" H 7700 2900 50  0001 C CNN
-F 1 "+3V3" V 7715 3178 50  0000 L CNN
-F 2 "" H 7700 3050 50  0001 C CNN
-F 3 "" H 7700 3050 50  0001 C CNN
-	1    7700 3050
-	0    1    1    0
 $EndComp
 $Comp
@@
 L power:GND #PWR?
 U 1 1 6027C950
-P 7700 3150
+P 7950 3350
 AR Path="/601BF914/6027C950" Ref="#PWR?"  Part="1"
 AR Path="/601E7BA1/6027C950" Ref="#PWR?"  Part="1"
 AR Path="/60210E5F/6027C950" Ref="#PWR012"  Part="1"
-F 0 "#PWR012" H 7700 2900 50  0001 C CNN
-F 1 "GND" V 7705 3022 50  0000 R CNN
-F 2 "" H 7700 3150 50  0001 C CNN
-F 3 "" H 7700 3150 50  0001 C CNN
-	1    7700 3150
+F 0 "#PWR012" H 7950 3100 50  0001 C CNN
+F 1 "GND" V 7955 3222 50  0000 R CNN
+F 2 "" H 7950 3350 50  0001 C CNN
+F 3 "" H 7950 3350 50  0001 C CNN
+	1    7950 3350
 	0    -1   -1   0
 $EndComp
@@
 NoConn ~ 6850 3050
 NoConn ~ 6850 3150
+$Comp
+L Device:C C?
+U 1 1 602407B9
+P 7850 3200
+AR Path="/601BF914/602407B9" Ref="C?"  Part="1"
+AR Path="/601E7BA1/602407B9" Ref="C?"  Part="1"
+AR Path="/60210E5F/602407B9" Ref="C?"  Part="1"
+F 0 "C?" H 7800 3600 50  0000 L CNN
+F 1 "10nF" H 7750 3500 50  0000 L CNN
+F 2 "" H 7888 3050 50  0001 C CNN
+F 3 "~" H 7850 3200 50  0001 C CNN
+	1    7850 3200
+	-1   0    0    1
+$EndComp
+Wire Wire Line
+	7700 3150 7700 3350
+Wire Wire Line
+	7700 3350 7850 3350
+Wire Wire Line
+	7950 3350 7850 3350
+Connection ~ 7850 3350
+Text HLabel 8000 3050 2    50   Input ~ 0
+VDD_3
+Wire Wire Line
+	8000 3050 7850 3050
+Wire Wire Line
+	7850 3050 7700 3050
+Connection ~ 7850 3050
 $EndSCHEMATC

Commit message: Mosfet
Parts:
- gave numbers to parts that had none: 1
Changed lines of the file:
@@
 AR Path="/601BF914/602407B9" Ref="C?"  Part="1"
 AR Path="/601E7BA1/602407B9" Ref="C?"  Part="1"
-AR Path="/60210E5F/602407B9" Ref="C?"  Part="1"
-F 0 "C?" H 7800 3600 50  0000 L CNN
+AR Path="/60210E5F/602407B9" Ref="C20"  Part="1"
+F 0 "C20" H 7800 3600 50  0000 L CNN
 F 1 "10nF" H 7750 3500 50  0000 L CNN
 F 2 "" H 7888 3050 50  0001 C CNN

Commit message: Jirka upravy
Parts:
- removed C10, C11, C12, C13: 470pF, symbol Device:C
- added R? (x2): 1k, symbol Device:R
- C20: value 10nF -> 100nF
Connections:
- wire segments 22 -> 10
Changed lines of the file:
@@
 $EndDescr
-$Comp
-L Device:C C?
-U 1 1 60217BBA
-P 8550 3500
-AR Path="/601BF914/60217BBA" Ref="C?"  Part="1"
-AR Path="/601E7BA1/60217BBA" Ref="C?"  Part="1"
-AR Path="/60210E5F/60217BBA" Ref="C10"  Part="1"
-F 0 "C10" H 8665 3546 50  0000 L CNN
-F 1 "470pF" H 8665 3455 50  0000 L CNN
-F 2 "" H 8588 3350 50  0001 C CNN
-F 3 "~" H 8550 3500 50  0001 C CNN
-	1    8550 3500
-	1    0    0    -1
-$EndComp
-$Comp
-L Device:C C?
-U 1 1 60217BC0
-P 9250 3500
-AR Path="/601BF914/60217BC0" Ref="C?"  Part="1"
-AR Path="/601E7BA1/60217BC0" Ref="C?"  Part="1"
-AR Path="/60210E5F/60217BC0" Ref="C12"  Part="1"
-F 0 "C12" H 9365 3546 50  0000 L CNN
-F 1 "470pF" H 9365 3455 50  0000 L CNN
-F 2 "" H 9288 3350 50  0001 C CNN
-F 3 "~" H 9250 3500 50  0001 C CNN
-	1    9250 3500
-	1    0    0    -1
-$EndComp
-$Comp
-L Device:C C?
-U 1 1 60217BC6
-P 9600 3500
-AR Path="/601BF914/60217BC6" Ref="C?"  Part="1"
-AR Path="/601E7BA1/60217BC6" Ref="C?"  Part="1"
-AR Path="/60210E5F/60217BC6" Ref="C13"  Part="1"
-F 0 "C13" H 9715 3546 50  0000 L CNN
-F 1 "470pF" H 9715 3455 50  0000 L CNN
-F 2 "" H 9638 3350 50  0001 C CNN
-F 3 "~" H 9600 3500 50  0001 C CNN
-	1    9600 3500
-	1    0    0    -1
-$EndComp
 $Comp
 L Connector:Conn_01x04_Male J?
@@
 	1    9900 2850
 	-1   0    0    1
-$EndComp
-Wire Wire Line
-	7700 2950 8550 2950
-Wire Wire Line
-	7700 2850 8900 2850
-Wire Wire Line
-	7700 2750 9250 2750
-Wire Wire Line
-	7700 2650 9600 2650
-Wire Wire Line
-	8550 3350 8550 2950
-Connection ~ 8550 2950
-Wire Wire Line
-	8550 2950 9700 2950
-Connection ~ 8900 2850
-Wire Wire Line
-	8900 2850 9700 2850
-Wire Wire Line
-	9250 3350 9250 2750
-Connection ~ 9250 2750
-Wire Wire Line
-	9250 2750 9700 2750
-Wire Wire Line
-	9600 3350 9600 2650
-Connection ~ 9600 2650
-Wire Wire Line
-	9600 2650 9700 2650
-$Comp
-L power:GND #PWR?
-U 1 1 60217BE8
-P 8550 3750
-AR Path="/601BF914/60217BE8" Ref="#PWR?"  Part="1"
-AR Path="/601E7BA1/60217BE8" Ref="#PWR?"  Part="1"
-AR Path="/60210E5F/60217BE8" Ref="#PWR036"  Part="1"
-F 0 "#PWR036" H 8550 3500 50  0001 C CNN
-F 1 "GND" H 8555 3577 50  0000 C CNN
-F 2 "" H 8550 3750 50  0001 C CNN
-F 3 "" H 8550 3750 50  0001 C CNN
-	1    8550 3750
-	1    0    0    -1
-$EndComp
-$Comp
-L power:GND #PWR?
-U 1 1 60217BEE
-P 8900 3750
-AR Path="/601BF914/60217BEE" Ref="#PWR?"  Part="1"
-AR Path="/601E7BA1/60217BEE" Ref="#PWR?"  Part="1"
-AR Path="/60210E5F/60217BEE" Ref="#PWR037"  Part="1"
-F 0 "#PWR037" H 8900 3500 50  0001 C CNN
-F 1 "GND" H 8905 3577 50  0000 C CNN
-F 2 "" H 8900 3750 50  0001 C CNN
-F 3 "" H 8900 3750 50  0001 C CNN
-	1    8900 3750
-	1    0    0    -1
-$EndComp
-$Comp
-L power:GND #PWR?
-U 1 1 60217BF4
-P 9250 3750
-AR Path="/601BF914/60217BF4" Ref="#PWR?"  Part="1"
-AR Path="/601E7BA1/60217BF4" Ref="#PWR?"  Part="1"
-AR Path="/60210E5F/60217BF4" Ref="#PWR038"  Part="1"
-F 0 "#PWR038" H 9250 3500 50  0001 C CNN
-F 1 "GND" H 9255 3577 50  0000 C CNN
-F 2 "" H 9250 3750 50  0001 C CNN
-F 3 "" H 9250 3750 50  0001 C CNN
-	1    9250 3750
-	1    0    0    -1
-$EndComp
-$Comp
-L power:GND #PWR?
-U 1 1 60217BFA
-P 9600 3750
-AR Path="/601BF914/60217BFA" Ref="#PWR?"  Part="1"
-AR Path="/601E7BA1/60217BFA" Ref="#PWR?"  Part="1"
-AR Path="/60210E5F/60217BFA" Ref="#PWR039"  Part="1"
-F 0 "#PWR039" H 9600 3500 50  0001 C CNN
-F 1 "GND" H 9605 3577 50  0000 C CNN
-F 2 "" H 9600 3750 50  0001 C CNN
-F 3 "" H 9600 3750 50  0001 C CNN
-	1    9600 3750
-	1    0    0    -1
-$EndComp
-Wire Wire Line
-	8550 3650 8550 3750
-Wire Wire Line
-	9250 3650 9250 3750
-Wire Wire Line
-	9600 3650 9600 3750
-Wire Wire Line
-	8900 3650 8900 3750
-Wire Wire Line
-	8900 3350 8900 2850
-$Comp
-L Device:C C?
-U 1 1 60217C05
-P 8900 3500
-AR Path="/601BF914/60217C05" Ref="C?"  Part="1"
-AR Path="/601E7BA1/60217C05" Ref="C?"  Part="1"
-AR Path="/60210E5F/60217C05" Ref="C11"  Part="1"
-F 0 "C11" H 9015 3546 50  0000 L CNN
-F 1 "470pF" H 9015 3455 50  0000 L CNN
-F 2 "" H 8938 3350 50  0001 C CNN
-F 3 "~" H 8900 3500 50  0001 C CNN
-	1    8900 3500
-	1    0    0    -1
 $EndComp
 Text HLabel 6850 2450 0    50   Input ~ 0
@@
 L power:GND #PWR?
 U 1 1 601D625A
-P 6850 2650
+P 6550 2550
 AR Path="/601BF914/601D625A" Ref="#PWR?"  Part="1"
 AR Path="/601E7BA1/601D625A" Ref="#PWR?"  Part="1"
 AR Path="/60210E5F/601D625A" Ref="#PWR0119"  Part="1"
-F 0 "#PWR0119" H 6850 2400 50  0001 C CNN
-F 1 "GND" V 6855 2522 50  0000 R CNN
-F 2 "" H 6850 2650 50  0001 C CNN
-F 3 "" H 6850 2650 50  0001 C CNN
-	1    6850 2650
+F 0 "#PWR0119" H 6550 2300 50  0001 C CNN
+F 1 "GND" V 6555 2422 50  0000 R CNN
+F 2 "" H 6550 2550 50  0001 C CNN
+F 3 "" H 6550 2550 50  0001 C CNN
+	1    6550 2550
 	0    1    1    0
 $EndComp
@@
 L power:+3V3 #PWR0104
 U 1 1 601B5180
-P 6850 2550
-F 0 "#PWR0104" H 6850 2400 50  0001 C CNN
-F 1 "+3V3" V 6865 2678 50  0000 L CNN
-F 2 "" H 6850 2550 50  0001 C CNN
-F 3 "" H 6850 2550 50  0001 C CNN
-	1    6850 2550
+P 6550 2650
+F 0 "#PWR0104" H 6550 2500 50  0001 C CNN
+F 1 "+3V3" V 6565 2778 50  0000 L CNN
+F 2 "" H 6550 2650 50  0001 C CNN
+F 3 "" H 6550 2650 50  0001 C CNN
+	1    6550 2650
 	0    -1   -1   0
 $EndComp
@@
 AR Path="/60210E5F/602407B9" Ref="C20"  Part="1"
 F 0 "C20" H 7800 3600 50  0000 L CNN
-F 1 "10nF" H 7750 3500 50  0000 L CNN
+F 1 "100nF" H 7750 3500 50  0000 L CNN
 F 2 "" H 7888 3050 50  0001 C CNN
 F 3 "~" H 7850 3200 50  0001 C CNN
@@
 	7850 3050 7700 3050
 Connection ~ 7850 3050
+Wire Wire Line
+	7700 2950 9700 2950
+Wire Wire Line
+	7700 2750 9700 2750
+Wire Wire Line
+	7700 2650 9700 2650
+Wire Wire Line
+	7700 2850 9700 2850
+$Comp
+L Device:R R?
+U 1 1 6025D497
+P 6700 2650
+F 0 "R?" V 6493 2650 50  0000 C CNN
+F 1 "1k" V 6700 2600 50  0000 C CNN
+F 2 "" V 6630 2650 50  0001 C CNN
+F 3 "~" H 6700 2650 50  0001 C CNN
+	1    6700 2650
+	0    1    1    0
+$EndComp
+$Comp
+L Device:R R?
+U 1 1 6025DA6F
+P 6700 2550
+F 0 "R?" V 6493 2550 50  0000 C CNN
+F 1 "1k" V 6584 2550 50  0000 C CNN
+F 2 "" V 6630 2550 50  0001 C CNN
+F 3 "~" H 6700 2550 50  0001 C CNN
+	1    6700 2550
+	0    1    1    0
+$EndComp
 $EndSCHEMATC

Commit message: Hotové schéma
Parts:
- removed R?: 1k, symbol Device:R
- 2209Br3: LCSC (none) -> -
- C20: footprint (none) -> Capacitor_SMD:C_0402_1005Metric_Pad0.74x0.62mm_HandSolder; LCSC (none) -> C14663
- J21: footprint (none) -> Connector_PinHeader_2.54mm:PinHeader_1x04_P2.54mm_Vertical; LCSC (none) -> -
- R14: renamed from R?; footprint (none) -> Resistor_SMD:R_0805_2012Metric_Pad1.20x1.40mm_HandSolder; LCSC (none) -> C17513
Connections:
- wire segments 10 -> 11
Other:
- moved on the sheet: J21
Changed lines of the file:
@@
 L Connector:Conn_01x04_Male J?
 U 1 1 60217BCC
-P 9900 2850
+P 8250 2850
 AR Path="/601BF914/60217BCC" Ref="J?"  Part="1"
 AR Path="/601E7BA1/60217BCC" Ref="J?"  Part="1"
 AR Path="/60210E5F/60217BCC" Ref="J21"  Part="1"
-F 0 "J21" H 9872 2732 50  0000 R CNN
-F 1 "Conn_01x04_Male" H 9872 2823 50  0000 R CNN
-F 2 "" H 9900 2850 50  0001 C CNN
-F 3 "~" H 9900 2850 50  0001 C CNN
-	1    9900 2850
+F 0 "J21" H 8222 2732 50  0000 R CNN
+F 1 "Conn_01x04_Male" H 8222 2823 50  0000 R CNN
+F 2 "Connector_PinHeader_2.54mm:PinHeader_1x04_P2.54mm_Vertical" H 8250 2850 50  0001 C CNN
+F 3 "~" H 8250 2850 50  0001 C CNN
+F 4 "-" H 8250 2850 50  0001 C CNN "LCSC"
+	1    8250 2850
 	-1   0    0    1
 $EndComp
 Text HLabel 6850 2450 0    50   Input ~ 0
 EN3
-Text HLabel 6850 2750 0    50   Input ~ 0
+Text HLabel 6850 2850 0    50   Input ~ 0
 PDN_3
 $Comp
@@
 F 2 "" H 7050 2700 50  0001 C CNN
 F 3 "" H 7050 2700 50  0001 C CNN
+F 4 "-" H 7300 2700 50  0001 C CNN "LCSC"
 	1    7300 2700
 	1    0    0    -1
@@
 F 0 "C20" H 7800 3600 50  0000 L CNN
 F 1 "100nF" H 7750 3500 50  0000 L CNN
-F 2 "" H 7888 3050 50  0001 C CNN
+F 2 "Capacitor_SMD:C_0402_1005Metric_Pad0.74x0.62mm_HandSolder" H 7888 3050 50  0001 C CNN
 F 3 "~" H 7850 3200 50  0001 C CNN
+F 4 "C14663" H 7850 3200 50  0001 C CNN "LCSC"
 	1    7850 3200
 	-1   0    0    1
@@
 Connection ~ 7850 3050
 Wire Wire Line
-	7700 2950 9700 2950
+	7700 2950 8050 2950
 Wire Wire Line
-	7700 2750 9700 2750
+	7700 2750 8050 2750
 Wire Wire Line
-	7700 2650 9700 2650
+	7700 2650 8050 2650
 Wire Wire Line
-	7700 2850 9700 2850
+	7700 2850 8050 2850
 $Comp
-L Device:R R?
+L Device:R R14
 U 1 1 6025D497
 P 6700 2650
-F 0 "R?" V 6493 2650 50  0000 C CNN
-F 1 "1k" V 6700 2600 50  0000 C CNN
-F 2 "" V 6630 2650 50  0001 C CNN
+F 0 "R14" V 6700 2650 50  0000 C CNN
+F 1 "1k" V 6800 2650 50  0000 C CNN
+F 2 "Resistor_SMD:R_0805_2012Metric_Pad1.20x1.40mm_HandSolder" V 6630 2650 50  0001 C CNN
 F 3 "~" H 6700 2650 50  0001 C CNN
+F 4 "C17513" H 6700 2650 50  0001 C CNN "LCSC"
 	1    6700 2650
 	0    1    1    0
 $EndComp
+Wire Wire Line
+	6550 2550 6850 2550
 $Comp
-L Device:R R?
-U 1 1 6025DA6F
-P 6700 2550
-F 0 "R?" V 6493 2550 50  0000 C CNN
-F 1 "1k" V 6584 2550 50  0000 C CNN
-F 2 "" V 6630 2550 50  0001 C CNN
-F 3 "~" H 6700 2550 50  0001 C CNN
-	1    6700 2550
-	0    1    1    0
+L power:PWR_FLAG #FLG0102
+U 1 1 60224EB1
+P 6850 2650
+F 0 "#FLG0102" H 6850 2725 50  0001 C CNN
+F 1 "PWR_FLAG" H 6850 2823 50  0000 C CNN
+F 2 "" H 6850 2650 50  0001 C CNN
+F 3 "~" H 6850 2650 50  0001 C CNN
+	1    6850 2650
+	1    0    0    -1
 $EndComp
+Connection ~ 6850 2650
 $EndSCHEMATC

Commit message: Hotová deska
Parts:
- 2209Br3: footprint (none) -> FinalExamThesis:TMC_2209_Breaout_Board
Changed lines of the file:
@@
 F 0 "2209Br3" H 7275 2127 50  0000 C CNN
 F 1 "TMC2209BreaoutBoard" H 7275 2036 50  0000 C CNN
-F 2 "" H 7050 2700 50  0001 C CNN
+F 2 "FinalExamThesis:TMC_2209_Breaout_Board" H 7050 2700 50  0001 C CNN
 F 3 "" H 7050 2700 50  0001 C CNN
 F 4 "-" H 7300 2700 50  0001 C CNN "LCSC"

Commit message: Deska2
Parts:
- added R18, R19: 1k, Resistor_SMD:R_0805_2012Metric_Pad1.20x1.40mm_HandSolder, symbol Device:R
Connections:
- net labels added: DIR, STEP
- no-connect marks 5 -> 3
Changed lines of the file:
@@
 	1    0    0    -1
 $EndComp
-NoConn ~ 6850 3050
-NoConn ~ 6850 3150
 $Comp
 L Device:C C?
@@
 $EndComp
 Connection ~ 6850 2650
+$Comp
+L Device:R R18
+U 1 1 6029EFAD
+P 6700 3050
+F 0 "R18" V 6700 3050 50  0000 C CNN
+F 1 "1k" V 6600 3050 50  0000 C CNN
+F 2 "Resistor_SMD:R_0805_2012Metric_Pad1.20x1.40mm_HandSolder" V 6630 3050 50  0001 C CNN
+F 3 "~" H 6700 3050 50  0001 C CNN
+F 4 "C17513" H 6700 3050 50  0001 C CNN "LCSC"
+	1    6700 3050
+	0    1    1    0
+$EndComp
+$Comp
+L Device:R R19
+U 1 1 6029F320
+P 6700 3150
+F 0 "R19" V 6700 3150 50  0000 C CNN
+F 1 "1k" V 6800 3150 50  0000 C CNN
+F 2 "Resistor_SMD:R_0805_2012Metric_Pad1.20x1.40mm_HandSolder" V 6630 3150 50  0001 C CNN
+F 3 "~" H 6700 3150 50  0001 C CNN
+F 4 "C17513" H 6700 3150 50  0001 C CNN "LCSC"
+	1    6700 3150
+	0    1    1    0
+$EndComp
+Text HLabel 6550 3050 0    50   Input ~ 0
+STEP
+Text HLabel 6550 3150 0    50   Input ~ 0
+DIR
 $EndSCHEMATC

Commit message: Nová Deska
Parts:
- added C5: 2,2mF, Capacitor_THT:CP_Radial_D10.0mm_P2.50mm, symbol Device:C
- 2209Br3: symbol Základní-deska-II-rescue:TMC2209BreaoutBoard-Tmc2209BreakoutBoard -> Základní-deska-II-rescue:TMC2209BreaoutBoard-Tmc2209BreakoutBoard-Základní-deska-II-rescue
Connections:
- wire segments 11 -> 14
Changed lines of the file:
@@
 L power:GND #PWR?
 U 1 1 60217C1C
-P 7700 2550
+P 7850 2550
 AR Path="/601BF914/60217C1C" Ref="#PWR?"  Part="1"
 AR Path="/601E7BA1/60217C1C" Ref="#PWR?"  Part="1"
 AR Path="/60210E5F/60217C1C" Ref="#PWR034"  Part="1"
-F 0 "#PWR034" H 7700 2300 50  0001 C CNN
-F 1 "GND" V 7705 2422 50  0000 R CNN
-F 2 "" H 7700 2550 50  0001 C CNN
-F 3 "" H 7700 2550 50  0001 C CNN
-	1    7700 2550
+F 0 "#PWR034" H 7850 2300 50  0001 C CNN
+F 1 "GND" V 7855 2422 50  0000 R CNN
+F 2 "" H 7850 2550 50  0001 C CNN
+F 3 "" H 7850 2550 50  0001 C CNN
+	1    7850 2550
 	0    -1   -1   0
 $EndComp
@@
 L power:+10V #PWR0121
 U 1 1 601B18BE
-P 7700 2450
-F 0 "#PWR0121" H 7700 2300 50  0001 C CNN
-F 1 "+10V" V 7715 2578 50  0000 L CNN
-F 2 "" H 7700 2450 50  0001 C CNN
-F 3 "" H 7700 2450 50  0001 C CNN
-	1    7700 2450
+P 7850 2250
+F 0 "#PWR0121" H 7850 2100 50  0001 C CNN
+F 1 "+10V" V 7865 2378 50  0000 L CNN
+F 2 "" H 7850 2250 50  0001 C CNN
+F 3 "" H 7850 2250 50  0001 C CNN
+	1    7850 2250
 	0    1    1    0
 $EndComp
@@
 $EndComp
 $Comp
-L Základní-deska-II-rescue:TMC2209BreaoutBoard-Tmc2209BreakoutBoard 2209Br3
+L Základní-deska-II-rescue:TMC2209BreaoutBoard-Tmc2209BreakoutBoard-Základní-deska-II-rescue 2209Br3
 U 1 1 602743DD
 P 7300 2700
@@
 Text HLabel 6550 3150 0    50   Input ~ 0
 DIR
+Wire Wire Line
+	7700 2450 7700 2250
+Wire Wire Line
+	7700 2250 7850 2250
+Connection ~ 7850 2250
+Wire Wire Line
+	7850 2550 7700 2550
+Connection ~ 7850 2550
+$Comp
+L Device:C C?
+U 1 1 602B8941
+P 7850 2400
+AR Path="/601BF914/602B8941" Ref="C?"  Part="1"
+AR Path="/60210E5F/602B8941" Ref="C5"  Part="1"
+F 0 "C5" H 7965 2446 50  0000 L CNN
+F 1 "2,2mF" H 7965 2355 50  0000 L CNN
+F 2 "Capacitor_THT:CP_Radial_D10.0mm_P2.50mm" H 7888 2250 50  0001 C CNN
+F 3 "~" H 7850 2400 50  0001 C CNN
+F 4 "C138489" H 7850 2400 50  0001 C CNN "LCSC"
+	1    7850 2400
+	1    0    0    -1
+$EndComp
 $EndSCHEMATC

Commit message: Deska 1.1
Parts:
- C5: value 2,2mF -> 470uF; LCSC C138489 -> C34642
Changed lines of the file:
@@
 AR Path="/60210E5F/602B8941" Ref="C5"  Part="1"
 F 0 "C5" H 7965 2446 50  0000 L CNN
-F 1 "2,2mF" H 7965 2355 50  0000 L CNN
+F 1 "470uF" H 7965 2355 50  0000 L CNN
 F 2 "Capacitor_THT:CP_Radial_D10.0mm_P2.50mm" H 7888 2250 50  0001 C CNN
 F 3 "~" H 7850 2400 50  0001 C CNN
-F 4 "C138489" H 7850 2400 50  0001 C CNN "LCSC"
+F 4 "C34642" H 7850 2400 50  0001 C CNN "LCSC"
 	1    7850 2400
 	1    0    0    -1
