File: Krokovka3.sch (KiCad schematic (older format))
At the start: 7 parts, among them J21 Conn_01x04_Male

Commit message: release candidate
Parts:
- C20: LCSC C14663 -> C1525
Changed lines of the file:
@@
 F 2 "Capacitor_SMD:C_0402_1005Metric_Pad0.74x0.62mm_HandSolder" H 7888 3050 50  0001 C CNN
 F 3 "~" H 7850 3200 50  0001 C CNN
-F 4 "C14663" H 7850 3200 50  0001 C CNN "LCSC"
+F 4 "C1525" H 7850 3200 50  0001 C CNN "LCSC"
 	1    7850 3200
 	-1   0    0    1

Commit message: Ordered
Parts:
- 2209Br3: symbol Základní-deska-II-rescue:TMC2209BreaoutBoard-Tmc2209BreakoutBoard-Základní-deska-II-rescue -> Zakladni_deska_II-rescue:TMC2209BreaoutBoard; JLCPCB_IGNORE (none) -> 1
- J21: JLCPCB_IGNORE (none) -> 1
- R14, R18, R19: LCSC C17513 -> C17379
Changed lines of the file:
@@
 F 3 "~" H 8250 2850 50  0001 C CNN
 F 4 "-" H 8250 2850 50  0001 C CNN "LCSC"
+F 5 "1" H 8250 2850 50  0001 C CNN "JLCPCB_IGNORE"
 	1    8250 2850
 	-1   0    0    1
@@
 $EndComp
 $Comp
-L Základní-deska-II-rescue:TMC2209BreaoutBoard-Tmc2209BreakoutBoard-Základní-deska-II-rescue 2209Br3
+L Zakladni_deska_II-rescue:TMC2209BreaoutBoard 2209Br3
 U 1 1 602743DD
 P 7300 2700
@@
 F 3 "" H 7050 2700 50  0001 C CNN
 F 4 "-" H 7300 2700 50  0001 C CNN "LCSC"
+F 5 "1" H 7300 2700 50  0001 C CNN "JLCPCB_IGNORE"
 	1    7300 2700
 	1    0    0    -1
@@
 F 2 "Resistor_SMD:R_0805_2012Metric_Pad1.20x1.40mm_HandSolder" V 6630 2650 50  0001 C CNN
 F 3 "~" H 6700 2650 50  0001 C CNN
-F 4 "C17513" H 6700 2650 50  0001 C CNN "LCSC"
+F 4 "C17379" H 6700 2650 50  0001 C CNN "LCSC"
 	1    6700 2650
 	0    1    1    0
@@
 	1    0    0    -1
 $EndComp
-Connection ~ 6850 2650
 $Comp
 L Device:R R18
@@
 F 2 "Resistor_SMD:R_0805_2012Metric_Pad1.20x1.40mm_HandSolder" V 6630 3050 50  0001 C CNN
 F 3 "~" H 6700 3050 50  0001 C CNN
-F 4 "C17513" H 6700 3050 50  0001 C CNN "LCSC"
+F 4 "C17379" H 6700 3050 50  0001 C CNN "LCSC"
 	1    6700 3050
 	0    1    1    0
@@
 F 2 "Resistor_SMD:R_0805_2012Metric_Pad1.20x1.40mm_HandSolder" V 6630 3150 50  0001 C CNN
 F 3 "~" H 6700 3150 50  0001 C CNN
-F 4 "C17513" H 6700 3150 50  0001 C CNN "LCSC"
+F 4 "C17379" H 6700 3150 50  0001 C CNN "LCSC"
 	1    6700 3150
 	0    1    1    0
