File: Napajeni.sch (KiCad schematic (older format))
At the start: 16 parts, among them Q1 BS250, Q2 NTR2101P, Q3 NTR2101P, Q4 BS250, Q5 NTR2101P, SW1 SW_MEC_5G, SW2 SW_MEC_5G

Commit message: Deska 0.5
Parts:
- removed H1, H2: MountingHole_Pad, symbol Mechanical:MountingHole_Pad
- added PL1, PL2: Plate, symbol Tmc2209BreakoutBoard:Plate
Connections:
- net GND: now also PL2.1 (PWR)
- net at F1.2: now also PL1.1 (PWR)
Other:
- moved on the sheet: C1, F1, Q1, Q2, Q3, Q4, Q5, R1, R2, R3, R4, R5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
