File: Napajeni.sch (KiCad schematic (older format))
At the start: 8 parts, among them Q2 2N7002

Commit message: Nová Deska
Parts:
- PL1, PL2: symbol Základní-deska-II-rescue:Plate-Tmc2209BreakoutBoard -> Základní-deska-II-rescue:Plate-Tmc2209BreakoutBoard-Základní-deska-II-rescue
- iQ1, iQ2: footprint (none) -> FinalExamThesis:NCE20P45Q; symbol NCE20P45Q:NCE20P45Q -> Základní-deska-II-rescue:NCE20P45Q-NCE20P45Q
Changed lines of the file:
@@
 	7600 3400 7600 3500
 $Comp
-L Základní-deska-II-rescue:Plate-Tmc2209BreakoutBoard PL2
+L Základní-deska-II-rescue:Plate-Tmc2209BreakoutBoard-Základní-deska-II-rescue PL2
 U 1 1 601FAA1F
 P 3200 2600
+AR Path="/601FAA1F" Ref="PL2"  Part="1"
+AR Path="/60188778/601FAA1F" Ref="PL2"  Part="1"
 F 0 "PL2" V 3300 2600 50  0000 C CNN
 F 1 "Plate" V 3400 2600 50  0000 C CNN
@@
 $EndComp
 $Comp
-L NCE20P45Q:NCE20P45Q iQ2
+L Základní-deska-II-rescue:NCE20P45Q-NCE20P45Q iQ2
 U 1 1 60300EC1
 P 5050 2250
+AR Path="/60300EC1" Ref="iQ2"  Part="1"
+AR Path="/60188778/60300EC1" Ref="iQ2"  Part="1"
 F 0 "iQ2" H 5050 2900 50  0000 C CNN
 F 1 "NCE20P45Q" H 5050 1550 50  0000 C CNN
-F 2 "" H 4950 2350 50  0001 C CNN
+F 2 "FinalExamThesis:NCE20P45Q" H 4950 2350 50  0001 C CNN
 F 3 "" H 4950 2350 50  0001 C CNN
 	1    5050 2250
@@
 	8750 1900 8750 2100
 $Comp
-L NCE20P45Q:NCE20P45Q iQ1
+L Základní-deska-II-rescue:NCE20P45Q-NCE20P45Q iQ1
 U 1 1 602FAA88
 P 7850 2250
+AR Path="/602FAA88" Ref="iQ1"  Part="1"
+AR Path="/60188778/602FAA88" Ref="iQ1"  Part="1"
 F 0 "iQ1" H 7850 2900 50  0000 C CNN
 F 1 "NCE20P45Q" H 7850 1600 50  0000 C CNN
-F 2 "" H 7750 2350 50  0001 C CNN
+F 2 "FinalExamThesis:NCE20P45Q" H 7750 2350 50  0001 C CNN
 F 3 "" H 7750 2350 50  0001 C CNN
 	1    7850 2250
@@
 	4500 2100 3400 2100
 $Comp
-L Základní-deska-II-rescue:Plate-Tmc2209BreakoutBoard PL1
+L Základní-deska-II-rescue:Plate-Tmc2209BreakoutBoard-Základní-deska-II-rescue PL1
 U 1 1 601FA68F
 P 3200 2100
+AR Path="/601FA68F" Ref="PL1"  Part="1"
+AR Path="/60188778/601FA68F" Ref="PL1"  Part="1"
 F 0 "PL1" V 2975 2112 50  0000 C CNN
 F 1 "Plate" V 3066 2112 50  0000 C CNN

Commit message: Deska 1.1
Parts:
- iQ1, iQ2: symbol Základní-deska-II-rescue:NCE20P45Q-NCE20P45Q -> Základní-deska-II-rescue:NCE20P45Q-NCE20P45Q-Základní-deska-II-rescue
Changed lines of the file:
@@
 $EndComp
 $Comp
-L Základní-deska-II-rescue:NCE20P45Q-NCE20P45Q iQ2
+L Základní-deska-II-rescue:NCE20P45Q-NCE20P45Q-Základní-deska-II-rescue iQ2
 U 1 1 60300EC1
 P 5050 2250
 AR Path="/60300EC1" Ref="iQ2"  Part="1"
-AR Path="/60188778/60300EC1" Ref="iQ2"  Part="1"
-F 0 "iQ2" H 5050 2900 50  0000 C CNN
+AR Path="/60188778/60300EC1" Ref="Q1"  Part="1"
+F 0 "Q1" H 5050 2900 50  0000 C CNN
 F 1 "NCE20P45Q" H 5050 1550 50  0000 C CNN
 F 2 "FinalExamThesis:NCE20P45Q" H 4950 2350 50  0001 C CNN
@@
 Wire Wire Line
 	8750 1900 8750 2100
-$Comp
-L Základní-deska-II-rescue:NCE20P45Q-NCE20P45Q iQ1
-U 1 1 602FAA88
-P 7850 2250
-AR Path="/602FAA88" Ref="iQ1"  Part="1"
-AR Path="/60188778/602FAA88" Ref="iQ1"  Part="1"
-F 0 "iQ1" H 7850 2900 50  0000 C CNN
-F 1 "NCE20P45Q" H 7850 1600 50  0000 C CNN
-F 2 "FinalExamThesis:NCE20P45Q" H 7750 2350 50  0001 C CNN
-F 3 "" H 7750 2350 50  0001 C CNN
-	1    7850 2250
-	1    0    0    -1
-$EndComp
 Wire Wire Line
 	5550 2100 5550 2400
@@
 	5950 2100 7350 2100
 Connection ~ 5950 2100
-Wire Wire Line
-	7350 2700 7350 2400
-Connection ~ 7350 2100
-Connection ~ 7350 2400
-Wire Wire Line
-	7350 2400 7350 2100
 Wire Wire Line
 	5550 2100 5950 2100
@@
 Connection ~ 8400 2100
 Wire Wire Line
-	8400 2100 8400 2400
-Connection ~ 8400 2400
+	5550 1850 5800 1850
+Wire Wire Line
+	5800 1850 5800 3500
 Wire Wire Line
 	8400 2400 8400 2700
 Wire Wire Line
-	5550 1850 5800 1850
+	8400 2100 8400 2400
+Connection ~ 8400 2400
+Connection ~ 7350 2100
 Wire Wire Line
-	5800 1850 5800 3500
+	7350 2400 7350 2100
+Wire Wire Line
+	7350 2700 7350 2400
+Connection ~ 7350 2400
+$Comp
+L Základní-deska-II-rescue:NCE20P45Q-NCE20P45Q-Základní-deska-II-rescue iQ1
+U 1 1 602FAA88
+P 7850 2250
+AR Path="/602FAA88" Ref="iQ1"  Part="1"
+AR Path="/60188778/602FAA88" Ref="Q3"  Part="1"
+F 0 "Q3" H 7850 2900 50  0000 C CNN
+F 1 "NCE20P45Q" H 7850 1600 50  0000 C CNN
+F 2 "FinalExamThesis:NCE20P45Q" H 7750 2350 50  0001 C CNN
+F 3 "" H 7750 2350 50  0001 C CNN
+	1    7850 2250
+	1    0    0    -1
+$EndComp
 $EndSCHEMATC

Commit message: release candidate
Parts:
- PL1, PL2: LCSC (none) -> -
- iQ1, iQ2: LCSC (none) -> C193354
Changed lines of the file:
@@
 F 2 "FinalExamThesis:Plate" H 3200 2600 50  0001 C CNN
 F 3 "" H 3200 2600 50  0001 C CNN
+F 4 "-" H 3200 2600 50  0001 C CNN "LCSC"
 	1    3200 2600
 	0    1    1    0
@@
 F 2 "FinalExamThesis:NCE20P45Q" H 4950 2350 50  0001 C CNN
 F 3 "" H 4950 2350 50  0001 C CNN
+F 4 "C193354" H 5050 2250 50  0001 C CNN "LCSC"
 	1    5050 2250
 	-1   0    0    -1
@@
 F 2 "FinalExamThesis:Plate" H 3200 2100 50  0001 C CNN
 F 3 "" H 3200 2100 50  0001 C CNN
+F 4 "-" H 3200 2100 50  0001 C CNN "LCSC"
 	1    3200 2100
 	0    1    1    0
@@
 F 2 "FinalExamThesis:NCE20P45Q" H 7750 2350 50  0001 C CNN
 F 3 "" H 7750 2350 50  0001 C CNN
+F 4 "C193354" H 7850 2250 50  0001 C CNN "LCSC"
 	1    7850 2250
 	1    0    0    -1

Commit message: Ordered
Parts:
- removed iQ1, iQ2: NCE20P45Q, FinalExamThesis:NCE20P45Q, symbol Základní-deska-II-rescue:NCE20P45Q-NCE20P45Q-Základní-deska-II-rescue
- added Q1, Q3: NCE2301, Package_TO_SOT_SMD:SOT-23, symbol Zakladni_deska_II-rescue:NCE2301
- PL1, PL2: symbol Základní-deska-II-rescue:Plate-Tmc2209BreakoutBoard-Základní-deska-II-rescue -> Zakladni_deska_II-rescue:Plate-Tmc2209BreakoutBoard; JLCPCB_IGNORE (none) -> 1
- Q2: JLCPCB_CORRECTION (none) -> 0;0;180
- R15: LCSC C17407 -> C17422
- R5: LCSC C17414 -> C17429
Connections:
- net +10V: now also Q3.3 (D)
- net GND: now also Q1.1 (G)
- net at PL1.1: now also Q1.3 (D)
- net at R15.1: now also Q1.2 (S), Q3.2 (S)
- net at Q2.3 (D), R15.2: now also Q3.1 (G)
Other:
- moved on the sheet: R15
Changed lines of the file:
@@
 L power:GND #PWR04
 U 1 1 6018E3FD
-P 5800 3500
-F 0 "#PWR04" H 5800 3250 50  0001 C CNN
-F 1 "GND" H 5805 3327 50  0000 C CNN
-F 2 "" H 5800 3500 50  0001 C CNN
-F 3 "" H 5800 3500 50  0001 C CNN
-	1    5800 3500
+P 4950 3525
+F 0 "#PWR04" H 4950 3275 50  0001 C CNN
+F 1 "GND" H 4955 3352 50  0000 C CNN
+F 2 "" H 4950 3525 50  0001 C CNN
+F 3 "" H 4950 3525 50  0001 C CNN
+	1    4950 3525
 	1    0    0    -1
 $EndComp
@@
 L power:GND #PWR09
 U 1 1 601B5E05
-P 7200 3500
-F 0 "#PWR09" H 7200 3250 50  0001 C CNN
-F 1 "GND" H 7205 3327 50  0000 C CNN
-F 2 "" H 7200 3500 50  0001 C CNN
-F 3 "" H 7200 3500 50  0001 C CNN
-	1    7200 3500
-	1    0    0    -1
-$EndComp
-Wire Wire Line
-	7200 3200 7200 3500
+P 7200 3525
+F 0 "#PWR09" H 7200 3275 50  0001 C CNN
+F 1 "GND" H 7205 3352 50  0000 C CNN
+F 2 "" H 7200 3525 50  0001 C CNN
+F 3 "" H 7200 3525 50  0001 C CNN
+	1    7200 3525
+	1    0    0    -1
+$EndComp
+Wire Wire Line
+	7200 3200 7200 3525
 $Comp
 L Device:R R5
@@
 F 2 "Resistor_SMD:R_0805_2012Metric_Pad1.20x1.40mm_HandSolder" V 7530 3250 50  0001 C CNN
 F 3 "~" H 7600 3250 50  0001 C CNN
-F 4 "C17414	" H 7600 3250 50  0001 C CNN "LCSC"
+F 4 "C17429" H 7600 3250 50  0001 C CNN "LCSC"
 	1    7600 3250
 	1    0    0    -1
@@
 L power:GND #PWR011
 U 1 1 601BC6CA
-P 7600 3500
-F 0 "#PWR011" H 7600 3250 50  0001 C CNN
-F 1 "GND" H 7605 3327 50  0000 C CNN
-F 2 "" H 7600 3500 50  0001 C CNN
-F 3 "" H 7600 3500 50  0001 C CNN
-	1    7600 3500
+P 7600 3525
+F 0 "#PWR011" H 7600 3275 50  0001 C CNN
+F 1 "GND" H 7605 3352 50  0000 C CNN
+F 2 "" H 7600 3525 50  0001 C CNN
+F 3 "" H 7600 3525 50  0001 C CNN
+	1    7600 3525
 	1    0    0    -1
 $EndComp
@@
 F 3 "https://www.onsemi.com/pub/Collateral/NDS7002A-D.PDF" H 7300 3000 50  0001 L CNN
 F 4 "C8545" H 7300 3000 50  0001 C CNN "LCSC"
+F 5 "0;0;180" H 7300 3000 50  0001 C CNN "JLCPCB_CORRECTION"
 	1    7300 3000
 	-1   0    0    -1
@@
 L Device:R R15
 U 1 1 60230BAA
-P 6900 2450
-F 0 "R15" H 6830 2404 50  0000 R CNN
-F 1 "100k" H 6830 2495 50  0000 R CNN
-F 2 "Resistor_SMD:R_0805_2012Metric_Pad1.20x1.40mm_HandSolder" V 6830 2450 50  0001 C CNN
-F 3 "~" H 6900 2450 50  0001 C CNN
-F 4 "C17407" H 6900 2450 50  0001 C CNN "LCSC"
-	1    6900 2450
-	0    -1   -1   0
-$EndComp
-Wire Wire Line
-	6750 2450 5950 2450
+P 6500 2450
+F 0 "R15" H 6430 2404 50  0000 R CNN
+F 1 "100k" H 6430 2495 50  0000 R CNN
+F 2 "Resistor_SMD:R_0805_2012Metric_Pad1.20x1.40mm_HandSolder" V 6430 2450 50  0001 C CNN
+F 3 "~" H 6500 2450 50  0001 C CNN
+F 4 "C17422" H 6500 2450 50  0001 C CNN "LCSC"
+	1    6500 2450
+	0    -1   -1   0
+$EndComp
+Wire Wire Line
+	6350 2450 5950 2450
 Wire Wire Line
 	5950 2450 5950 2100
 Wire Wire Line
-	7050 2450 7200 2450
+	6650 2450 7200 2450
 Wire Wire Line
 	7200 2450 7200 2800
@@
 	7600 3000 7650 3000
 Wire Wire Line
-	7600 3400 7600 3500
-$Comp
-L Základní-deska-II-rescue:Plate-Tmc2209BreakoutBoard-Základní-deska-II-rescue PL2
+	7600 3400 7600 3525
+$Comp
+L Zakladni_deska_II-rescue:Plate-Tmc2209BreakoutBoard PL2
 U 1 1 601FAA1F
 P 3200 2600
@@
 F 3 "" H 3200 2600 50  0001 C CNN
 F 4 "-" H 3200 2600 50  0001 C CNN "LCSC"
+F 5 "1" H 3200 2600 50  0001 C CNN "JLCPCB_IGNORE"
 	1    3200 2600
 	0    1    1    0
 $EndComp
-$Comp
-L Základní-deska-II-rescue:NCE20P45Q-NCE20P45Q-Základní-deska-II-rescue iQ2
-U 1 1 60300EC1
-P 5050 2250
-AR Path="/60300EC1" Ref="iQ2"  Part="1"
-AR Path="/60188778/60300EC1" Ref="Q1"  Part="1"
-F 0 "Q1" H 5050 2900 50  0000 C CNN
-F 1 "NCE20P45Q" H 5050 1550 50  0000 C CNN
-F 2 "FinalExamThesis:NCE20P45Q" H 4950 2350 50  0001 C CNN
-F 3 "" H 4950 2350 50  0001 C CNN
-F 4 "C193354" H 5050 2250 50  0001 C CNN "LCSC"
-	1    5050 2250
-	-1   0    0    -1
-$EndComp
-Wire Wire Line
-	8400 2100 8750 2100
 Wire Wire Line
 	8750 1650 8750 1900
-Connection ~ 8750 1900
-Wire Wire Line
-	8750 1900 8750 2100
-Wire Wire Line
-	5550 2100 5550 2400
-Connection ~ 5550 2400
-Wire Wire Line
-	5550 2400 5550 2700
-Wire Wire Line
-	7200 2450 7200 1850
-Wire Wire Line
-	7200 1850 7350 1850
+Wire Wire Line
+	7200 2450 7200 2400
 Connection ~ 7200 2450
-Wire Wire Line
-	5950 2100 7350 2100
 Connection ~ 5950 2100
 Wire Wire Line
-	5550 2100 5950 2100
-Connection ~ 5550 2100
-Wire Wire Line
-	4500 2700 4500 2400
-Connection ~ 4500 2100
-Wire Wire Line
-	4500 2100 4500 1850
-Connection ~ 4500 2400
-Wire Wire Line
-	4500 2400 4500 2100
-Wire Wire Line
-	4500 2100 3400 2100
-$Comp
-L Základní-deska-II-rescue:Plate-Tmc2209BreakoutBoard-Základní-deska-II-rescue PL1
+	4750 2100 3400 2100
+$Comp
+L Zakladni_deska_II-rescue:Plate-Tmc2209BreakoutBoard PL1
 U 1 1 601FA68F
 P 3200 2100
@@
 F 3 "" H 3200 2100 50  0001 C CNN
 F 4 "-" H 3200 2100 50  0001 C CNN "LCSC"
+F 5 "1" H 3200 2100 50  0001 C CNN "JLCPCB_IGNORE"
 	1    3200 2100
 	0    1    1    0
 $EndComp
 Wire Wire Line
-	8400 1850 8400 2100
-Connection ~ 8400 2100
-Wire Wire Line
-	5550 1850 5800 1850
-Wire Wire Line
-	5800 1850 5800 3500
-Wire Wire Line
-	8400 2400 8400 2700
-Wire Wire Line
-	8400 2100 8400 2400
-Connection ~ 8400 2400
-Connection ~ 7350 2100
-Wire Wire Line
-	7350 2400 7350 2100
-Wire Wire Line
-	7350 2700 7350 2400
-Connection ~ 7350 2400
-$Comp
-L Základní-deska-II-rescue:NCE20P45Q-NCE20P45Q-Základní-deska-II-rescue iQ1
-U 1 1 602FAA88
-P 7850 2250
-AR Path="/602FAA88" Ref="iQ1"  Part="1"
-AR Path="/60188778/602FAA88" Ref="Q3"  Part="1"
-F 0 "Q3" H 7850 2900 50  0000 C CNN
-F 1 "NCE20P45Q" H 7850 1600 50  0000 C CNN
-F 2 "FinalExamThesis:NCE20P45Q" H 7750 2350 50  0001 C CNN
-F 3 "" H 7750 2350 50  0001 C CNN
-F 4 "C193354" H 7850 2250 50  0001 C CNN "LCSC"
-	1    7850 2250
-	1    0    0    -1
-$EndComp
+	4950 2400 4950 3525
+Connection ~ 8750 1900
+Wire Wire Line
+	8750 1900 8750 2100
+$Comp
+L Zakladni_deska_II-rescue:NCE2301 Q1
+U 1 1 602E74FB
+P 4950 2200
+F 0 "Q1" V 5292 2200 50  0000 C CNN
+F 1 "NCE2301" V 5201 2200 50  0000 C CNN
+F 2 "Package_TO_SOT_SMD:SOT-23" H 5150 2125 50  0001 L CIN
+F 3 "http://www.vishay.com/docs/70209/70209.pdf" H 4950 2200 50  0001 L CNN
+F 4 "C113201" H 4950 2200 50  0001 C CNN "LCSC"
+F 5 "0;0;180" H 4950 2200 50  0001 C CNN "JLCPCB_CORRECTION"
+	1    4950 2200
+	0    -1   -1   0
+$EndComp
+Wire Wire Line
+	5150 2100 5950 2100
+$Comp
+L Zakladni_deska_II-rescue:NCE2301 Q3
+U 1 1 602EC88A
+P 7200 2200
+F 0 "Q3" V 7542 2200 50  0000 C CNN
+F 1 "NCE2301" V 7451 2200 50  0000 C CNN
+F 2 "Package_TO_SOT_SMD:SOT-23" H 7400 2125 50  0001 L CIN
+F 3 "http://www.vishay.com/docs/70209/70209.pdf" H 7200 2200 50  0001 L CNN
+F 4 "C113201" H 7200 2200 50  0001 C CNN "LCSC"
+F 5 "0;0;180" H 7200 2200 50  0001 C CNN "JLCPCB_CORRECTION"
+	1    7200 2200
+	0    1    -1   0
+$EndComp
+Wire Wire Line
+	5950 2100 7000 2100
+Wire Wire Line
+	7400 2100 8750 2100
 $EndSCHEMATC
