File: Základní deska II.sch (KiCad schematic (older format))
At the start: 7 parts, among them J5 Conn_01x04_Male, U1 ESP32-DEVKITC-32D

Commit message: Doplnen reset
Parts:
- added J1, J2: Conn_01x04_Male, symbol Connector:Conn_01x04_Male
- added R1: 1k, symbol Device:R
- added R2: 100k, symbol Device:R
- added SW1, SW3, SW4, SW5: SW_MEC_5G, symbol Switch:SW_MEC_5G
Connections:
- net labels added: VDD_1, VDD_2, VDD_3, VDD_4, Čte
- wire segments 54 -> 80
- no-connect marks 12 -> 17
Other:
- moved on the sheet: J5

Commit message: Jirka upravy
Parts:
- added R4: 330, symbol Device:R
Connections:
- net labels added: Řídí
- wire segments 80 -> 81
Changed lines of the file:
@@
 Connection ~ 5950 2100
 Wire Wire Line
-	3450 2200 5650 2200
+	3450 2200 5200 2200
 Wire Wire Line
 	3450 2100 5200 2100
@@
 Text GLabel 9500 5950 0    50   Input ~ 0
 VDD_4
+$Comp
+L power:PWR_FLAG #FLG02
+U 1 1 6024A163
+P 1850 2000
+F 0 "#FLG02" H 1850 2075 50  0001 C CNN
+F 1 "PWR_FLAG" H 1850 2173 50  0000 C CNN
+F 2 "" H 1850 2000 50  0001 C CNN
+F 3 "~" H 1850 2000 50  0001 C CNN
+	1    1850 2000
+	1    0    0    -1
+$EndComp
+Connection ~ 1850 2000
+Text Label 3850 2100 0    50   ~ 0
+Řídí
+$Comp
+L Device:R R?
+U 1 1 6024CA84
+P 5350 2200
+AR Path="/601BF914/6024CA84" Ref="R?"  Part="1"
+AR Path="/6024CA84" Ref="R4"  Part="1"
+F 0 "R4" V 5550 2200 50  0000 C CNN
+F 1 "330" V 5450 2200 50  0000 C CNN
+F 2 "" V 5280 2200 50  0001 C CNN
+F 3 "~" H 5350 2200 50  0001 C CNN
+	1    5350 2200
+	0    1    1    0
+$EndComp
+Wire Wire Line
+	5500 2200 5650 2200
 $EndSCHEMATC

Commit message: Hotové schéma
Parts:
- added H1, H2, H3, H4: MountingHole, symbol Mechanical:MountingHole
- J1, J2, J5: footprint (none) -> Connector_PinHeader_2.54mm:PinHeader_1x04_P2.54mm_Vertical; LCSC (none) -> -
- R1, R10, R6, R7, R8, R9: footprint (none) -> Resistor_SMD:R_0805_2012Metric_Pad1.20x1.40mm_HandSolder; LCSC (none) -> C17513
- R2: footprint (none) -> Resistor_SMD:R_0805_2012Metric_Pad1.20x1.40mm_HandSolder; LCSC (none) -> C17407
- R4: footprint (none) -> Resistor_SMD:R_0805_2012Metric_Pad1.20x1.40mm_HandSolder; LCSC (none) -> C17617
- SW1, SW3, SW4, SW5: footprint (none) -> Connector_PinHeader_2.54mm:PinHeader_1x02_P2.54mm_Vertical; LCSC (none) -> -
- U1: footprint MODULE_ESP32-DEVKITC-32D -> FinalExamThesis:MODULE_ESP32-DEVKITC-32D; LCSC (none) -> -
Changed lines of the file:
@@
 F0 "Napajeni" 50
 F1 "Napajeni.sch" 50
-F2 "SW_OFF" I L 9500 1050 50
+F2 "SW_CTRL" I L 9500 1050 50
 $EndSheet
 $Sheet
@@
 F 0 "R6" V 3693 3000 50  0000 C CNN
 F 1 "1k" V 3784 3000 50  0000 C CNN
-F 2 "" V 3830 3000 50  0001 C CNN
+F 2 "Resistor_SMD:R_0805_2012Metric_Pad1.20x1.40mm_HandSolder" V 3830 3000 50  0001 C CNN
 F 3 "~" H 3900 3000 50  0001 C CNN
+F 4 "C17513" H 3900 3000 50  0001 C CNN "LCSC"
 	1    3900 3000
 	0    1    1    0
@@
 F 0 "U1" H 2650 4067 50  0000 C CNN
 F 1 "ESP32-DEVKITC-32D" H 2650 3976 50  0000 C CNN
-F 2 "MODULE_ESP32-DEVKITC-32D" H 2650 2900 50  0001 L BNN
+F 2 "FinalExamThesis:MODULE_ESP32-DEVKITC-32D" H 2650 2900 50  0001 L BNN
 F 3 "" H 2650 2900 50  0001 L BNN
 F 4 "4" H 2650 2900 50  0001 L BNN "PARTREV"
 F 5 "Espressif Systems" H 2650 2900 50  0001 L BNN "MANUFACTURER"
+F 6 "-" H 2650 2900 50  0001 C CNN "LCSC"
 	1    2650 2900
 	1    0    0    -1
@@
 F 0 "R10" V 8743 6250 50  0000 C CNN
 F 1 "1k" V 8834 6250 50  0000 C CNN
-F 2 "" V 8880 6250 50  0001 C CNN
+F 2 "Resistor_SMD:R_0805_2012Metric_Pad1.20x1.40mm_HandSolder" V 8880 6250 50  0001 C CNN
 F 3 "~" H 8950 6250 50  0001 C CNN
+F 4 "C17513" H 8950 6250 50  0001 C CNN "LCSC"
 	1    8950 6250
 	0    1    1    0
@@
 F 0 "R9" V 8743 4650 50  0000 C CNN
 F 1 "1k" V 8834 4650 50  0000 C CNN
-F 2 "" V 8880 4650 50  0001 C CNN
+F 2 "Resistor_SMD:R_0805_2012Metric_Pad1.20x1.40mm_HandSolder" V 8880 4650 50  0001 C CNN
 F 3 "~" H 8950 4650 50  0001 C CNN
+F 4 "C17513" H 8950 4650 50  0001 C CNN "LCSC"
 	1    8950 4650
 	0    1    1    0
@@
 F 0 "R8" V 8743 3850 50  0000 C CNN
 F 1 "1k" V 8834 3850 50  0000 C CNN
-F 2 "" V 8880 3850 50  0001 C CNN
+F 2 "Resistor_SMD:R_0805_2012Metric_Pad1.20x1.40mm_HandSolder" V 8880 3850 50  0001 C CNN
 F 3 "~" H 8950 3850 50  0001 C CNN
+F 4 "C17513" H 8950 3850 50  0001 C CNN "LCSC"
 	1    8950 3850
 	0    1    1    0
@@
 F 0 "R7" V 8743 2950 50  0000 C CNN
 F 1 "1k" V 8834 2950 50  0000 C CNN
-F 2 "" V 8880 2950 50  0001 C CNN
+F 2 "Resistor_SMD:R_0805_2012Metric_Pad1.20x1.40mm_HandSolder" V 8880 2950 50  0001 C CNN
 F 3 "~" H 8950 2950 50  0001 C CNN
+F 4 "C17513" H 8950 2950 50  0001 C CNN "LCSC"
 	1    8950 2950
 	0    1    1    0
@@
 F3 "PDN_1" I L 9500 2600 50
 F4 "INDEX_1" I L 9500 2950 50
-F5 "VDD" I L 9500 2750 50
+F5 "VDD_1" I L 9500 2750 50
 $EndSheet
 $Sheet
@@
 F 0 "J2" V 2800 5100 50  0000 R CNN
 F 1 "Conn_01x04_Male" V 2900 5400 50  0000 R CNN
-F 2 "" H 2950 5150 50  0001 C CNN
+F 2 "Connector_PinHeader_2.54mm:PinHeader_1x04_P2.54mm_Vertical" H 2950 5150 50  0001 C CNN
 F 3 "~" H 2950 5150 50  0001 C CNN
+F 4 "-" H 2950 5150 50  0001 C CNN "LCSC"
 	1    2950 5150
 	0    1    1    0
@@
 F 0 "J1" V 700 4300 50  0000 R CNN
 F 1 "Conn_01x04_Male" V 800 4600 50  0000 R CNN
-F 2 "" H 850 4350 50  0001 C CNN
+F 2 "Connector_PinHeader_2.54mm:PinHeader_1x04_P2.54mm_Vertical" H 850 4350 50  0001 C CNN
 F 3 "~" H 850 4350 50  0001 C CNN
+F 4 "-" H 850 4350 50  0001 C CNN "LCSC"
 	1    850  4350
 	0    -1   -1   0
@@
 F 0 "J5" V 2100 5100 50  0000 R CNN
 F 1 "Conn_01x04_Male" V 2200 5400 50  0000 R CNN
-F 2 "" H 2250 5150 50  0001 C CNN
+F 2 "Connector_PinHeader_2.54mm:PinHeader_1x04_P2.54mm_Vertical" H 2250 5150 50  0001 C CNN
 F 3 "~" H 2250 5150 50  0001 C CNN
+F 4 "-" H 2250 5150 50  0001 C CNN "LCSC"
 	1    2250 5150
 	0    1    1    0
@@
 F 0 "SW1" H 5950 2085 50  0000 C CNN
 F 1 "SW_MEC_5G" H 5950 1994 50  0000 C CNN
-F 2 "" H 5950 2000 50  0001 C CNN
+F 2 "Connector_PinHeader_2.54mm:PinHeader_1x02_P2.54mm_Vertical" H 5950 2000 50  0001 C CNN
 F 3 "http://www.apem.com/int/index.php?controller=attachment&id_attachment=488" H 5950 2000 50  0001 C CNN
+F 4 "-" H 5950 1800 50  0001 C CNN "LCSC"
 	1    5950 1800
 	0    1    1    0
@@
 F 0 "R2" H 5720 1846 50  0000 L CNN
 F 1 "100k" H 5720 1755 50  0000 L CNN
-F 2 "" V 5580 1800 50  0001 C CNN
+F 2 "Resistor_SMD:R_0805_2012Metric_Pad1.20x1.40mm_HandSolder" V 5580 1800 50  0001 C CNN
 F 3 "~" H 5650 1800 50  0001 C CNN
+F 4 "C17407" H 5650 1800 50  0001 C CNN "LCSC"
 	1    5650 1800
 	1    0    0    -1
@@
 F 0 "R1" V 5143 2100 50  0000 C CNN
 F 1 "1k" V 5234 2100 50  0000 C CNN
-F 2 "" V 5280 2100 50  0001 C CNN
+F 2 "Resistor_SMD:R_0805_2012Metric_Pad1.20x1.40mm_HandSolder" V 5280 2100 50  0001 C CNN
 F 3 "~" H 5350 2100 50  0001 C CNN
+F 4 "C17513" H 5350 2100 50  0001 C CNN "LCSC"
 	1    5350 2100
 	0    1    1    0
@@
 F 0 "SW3" H 6300 2085 50  0000 C CNN
 F 1 "SW_MEC_5G" H 6300 1994 50  0000 C CNN
-F 2 "" H 6300 2000 50  0001 C CNN
+F 2 "Connector_PinHeader_2.54mm:PinHeader_1x02_P2.54mm_Vertical" H 6300 2000 50  0001 C CNN
 F 3 "http://www.apem.com/int/index.php?controller=attachment&id_attachment=488" H 6300 2000 50  0001 C CNN
+F 4 "-" H 6300 1800 50  0001 C CNN "LCSC"
 	1    6300 1800
 	0    1    1    0
@@
 F 0 "SW4" H 6650 2085 50  0000 C CNN
 F 1 "SW_MEC_5G" H 6650 1994 50  0000 C CNN
-F 2 "" H 6650 2000 50  0001 C CNN
+F 2 "Connector_PinHeader_2.54mm:PinHeader_1x02_P2.54mm_Vertical" H 6650 2000 50  0001 C CNN
 F 3 "http://www.apem.com/int/index.php?controller=attachment&id_attachment=488" H 6650 2000 50  0001 C CNN
+F 4 "-" H 6650 1800 50  0001 C CNN "LCSC"
 	1    6650 1800
 	0    1    1    0
@@
 F 0 "SW5" H 7050 2085 50  0000 C CNN
 F 1 "SW_MEC_5G" H 7050 1994 50  0000 C CNN
-F 2 "" H 7050 2000 50  0001 C CNN
+F 2 "Connector_PinHeader_2.54mm:PinHeader_1x02_P2.54mm_Vertical" H 7050 2000 50  0001 C CNN
 F 3 "http://www.apem.com/int/index.php?controller=attachment&id_attachment=488" H 7050 2000 50  0001 C CNN
+F 4 "-" H 7050 1800 50  0001 C CNN "LCSC"
 	1    7050 1800
 	0    1    1    0
@@
 F 0 "R4" V 5550 2200 50  0000 C CNN
 F 1 "330" V 5450 2200 50  0000 C CNN
-F 2 "" V 5280 2200 50  0001 C CNN
+F 2 "Resistor_SMD:R_0805_2012Metric_Pad1.20x1.40mm_HandSolder" V 5280 2200 50  0001 C CNN
 F 3 "~" H 5350 2200 50  0001 C CNN
+F 4 "C17617" H 5350 2200 50  0001 C CNN "LCSC"
 	1    5350 2200
 	0    1    1    0
@@
 Wire Wire Line
 	5500 2200 5650 2200
+$Comp
+L Mechanical:MountingHole H1
+U 1 1 6022FB89
+P 650 650
+F 0 "H1" H 750 696 50  0000 L CNN
+F 1 "MountingHole" H 750 605 50  0000 L CNN
+F 2 "" H 650 650 50  0001 C CNN
+F 3 "~" H 650 650 50  0001 C CNN
+	1    650  650
+	1    0    0    -1
+$EndComp
+$Comp
+L Mechanical:MountingHole H2
+U 1 1 60230021
+P 650 850
+F 0 "H2" H 750 896 50  0000 L CNN
+F 1 "MountingHole" H 750 805 50  0000 L CNN
+F 2 "" H 650 850 50  0001 C CNN
+F 3 "~" H 650 850 50  0001 C CNN
+	1    650  850
+	1    0    0    -1
+$EndComp
+$Comp
+L Mechanical:MountingHole H3
+U 1 1 602300F2
+P 650 1050
+F 0 "H3" H 750 1096 50  0000 L CNN
+F 1 "MountingHole" H 750 1005 50  0000 L CNN
+F 2 "" H 650 1050 50  0001 C CNN
+F 3 "~" H 650 1050 50  0001 C CNN
+	1    650  1050
+	1    0    0    -1
+$EndComp
+$Comp
+L Mechanical:MountingHole H4
+U 1 1 602301EA
+P 650 1300
+F 0 "H4" H 750 1346 50  0000 L CNN
+F 1 "MountingHole" H 750 1255 50  0000 L CNN
+F 2 "" H 650 1300 50  0001 C CNN
+F 3 "~" H 650 1300 50  0001 C CNN
+	1    650  1300
+	1    0    0    -1
+$EndComp
 $EndSCHEMATC

Commit message: Hotová deska
Parts:
- H1, H2, H3, H4: footprint (none) -> MountingHole:MountingHole_3mm
Changed lines of the file:
@@
 F 0 "H1" H 750 696 50  0000 L CNN
 F 1 "MountingHole" H 750 605 50  0000 L CNN
-F 2 "" H 650 650 50  0001 C CNN
+F 2 "MountingHole:MountingHole_3mm" H 650 650 50  0001 C CNN
 F 3 "~" H 650 650 50  0001 C CNN
 	1    650  650
@@
 F 0 "H2" H 750 896 50  0000 L CNN
 F 1 "MountingHole" H 750 805 50  0000 L CNN
-F 2 "" H 650 850 50  0001 C CNN
+F 2 "MountingHole:MountingHole_3mm" H 650 850 50  0001 C CNN
 F 3 "~" H 650 850 50  0001 C CNN
 	1    650  850
@@
 F 0 "H3" H 750 1096 50  0000 L CNN
 F 1 "MountingHole" H 750 1005 50  0000 L CNN
-F 2 "" H 650 1050 50  0001 C CNN
+F 2 "MountingHole:MountingHole_3mm" H 650 1050 50  0001 C CNN
 F 3 "~" H 650 1050 50  0001 C CNN
 	1    650  1050
@@
 F 0 "H4" H 750 1346 50  0000 L CNN
 F 1 "MountingHole" H 750 1255 50  0000 L CNN
-F 2 "" H 650 1300 50  0001 C CNN
+F 2 "MountingHole:MountingHole_3mm" H 650 1300 50  0001 C CNN
 F 3 "~" H 650 1300 50  0001 C CNN
 	1    650  1300

Commit message: Deska2
Parts:
- removed SW1, SW3, SW4, SW5: SW_MEC_5G, Connector_PinHeader_2.54mm:PinHeader_1x02_P2.54mm_Vertical, symbol Switch:SW_MEC_5G
- added J3, J4, J6, J8, J9: Conn_01x02_Male, Connector_PinHeader_2.54mm:PinHeader_1x02_P2.54mm_Vertical, symbol Connector:Conn_01x02_Male
- added R16, R17: 330, Resistor_SMD:R_0805_2012Metric_Pad1.20x1.40mm_HandSolder, symbol Device:R
Connections:
- wire segments 81 -> 86
- no-connect marks 17 -> 13
Changed lines of the file:
@@
 U 1 1 602202EC
 P 3900 3000
-F 0 "R6" V 3693 3000 50  0000 C CNN
-F 1 "1k" V 3784 3000 50  0000 C CNN
+F 0 "R6" V 3900 3000 50  0000 C CNN
+F 1 "1k" V 3950 2850 50  0000 C CNN
 F 2 "Resistor_SMD:R_0805_2012Metric_Pad1.20x1.40mm_HandSolder" V 3830 3000 50  0001 C CNN
 F 3 "~" H 3900 3000 50  0001 C CNN
@@
 F4 "INDEX_3" I L 9500 4650 50
 F5 "VDD_3" I L 9500 5000 50
+F6 "STEP" I L 9500 5100 50
+F7 "DIR" I L 9500 5200 50
 $EndSheet
 Wire Wire Line
@@
 F 4 "-" H 2250 5150 50  0001 C CNN "LCSC"
 	1    2250 5150
-	0    1    1    0
-$EndComp
-$Comp
-L Switch:SW_MEC_5G SW?
-U 1 1 601E6C8F
-P 5950 1800
-AR Path="/60188778/601E6C8F" Ref="SW?"  Part="1"
-AR Path="/601BF914/601E6C8F" Ref="SW?"  Part="1"
-AR Path="/601E6C8F" Ref="SW1"  Part="1"
-F 0 "SW1" H 5950 2085 50  0000 C CNN
-F 1 "SW_MEC_5G" H 5950 1994 50  0000 C CNN
-F 2 "Connector_PinHeader_2.54mm:PinHeader_1x02_P2.54mm_Vertical" H 5950 2000 50  0001 C CNN
-F 3 "http://www.apem.com/int/index.php?controller=attachment&id_attachment=488" H 5950 2000 50  0001 C CNN
-F 4 "-" H 5950 1800 50  0001 C CNN "LCSC"
-	1    5950 1800
 	0    1    1    0
 $EndComp
@@
 Wire Wire Line
 	5650 1550 5950 1550
-Wire Wire Line
-	5950 1550 5950 1600
 Connection ~ 5650 1550
 Wire Wire Line
 	5650 2100 5950 2100
-Wire Wire Line
-	5950 2100 5950 2000
 Connection ~ 5650 2100
 Wire Wire Line
@@
 	0    1    1    0
 $EndComp
-$Comp
-L Switch:SW_MEC_5G SW?
-U 1 1 601F7428
-P 6300 1800
-AR Path="/60188778/601F7428" Ref="SW?"  Part="1"
-AR Path="/601BF914/601F7428" Ref="SW?"  Part="1"
-AR Path="/601F7428" Ref="SW3"  Part="1"
-F 0 "SW3" H 6300 2085 50  0000 C CNN
-F 1 "SW_MEC_5G" H 6300 1994 50  0000 C CNN
-F 2 "Connector_PinHeader_2.54mm:PinHeader_1x02_P2.54mm_Vertical" H 6300 2000 50  0001 C CNN
-F 3 "http://www.apem.com/int/index.php?controller=attachment&id_attachment=488" H 6300 2000 50  0001 C CNN
-F 4 "-" H 6300 1800 50  0001 C CNN "LCSC"
-	1    6300 1800
-	0    1    1    0
-$EndComp
-$Comp
-L Switch:SW_MEC_5G SW?
-U 1 1 601F76BE
-P 6650 1800
-AR Path="/60188778/601F76BE" Ref="SW?"  Part="1"
-AR Path="/601BF914/601F76BE" Ref="SW?"  Part="1"
-AR Path="/601F76BE" Ref="SW4"  Part="1"
-F 0 "SW4" H 6650 2085 50  0000 C CNN
-F 1 "SW_MEC_5G" H 6650 1994 50  0000 C CNN
-F 2 "Connector_PinHeader_2.54mm:PinHeader_1x02_P2.54mm_Vertical" H 6650 2000 50  0001 C CNN
-F 3 "http://www.apem.com/int/index.php?controller=attachment&id_attachment=488" H 6650 2000 50  0001 C CNN
-F 4 "-" H 6650 1800 50  0001 C CNN "LCSC"
-	1    6650 1800
-	0    1    1    0
-$EndComp
-$Comp
-L Switch:SW_MEC_5G SW?
-U 1 1 601F78CA
-P 7050 1800
-AR Path="/60188778/601F78CA" Ref="SW?"  Part="1"
-AR Path="/601BF914/601F78CA" Ref="SW?"  Part="1"
-AR Path="/601F78CA" Ref="SW5"  Part="1"
-F 0 "SW5" H 7050 2085 50  0000 C CNN
-F 1 "SW_MEC_5G" H 7050 1994 50  0000 C CNN
-F 2 "Connector_PinHeader_2.54mm:PinHeader_1x02_P2.54mm_Vertical" H 7050 2000 50  0001 C CNN
-F 3 "http://www.apem.com/int/index.php?controller=attachment&id_attachment=488" H 7050 2000 50  0001 C CNN
-F 4 "-" H 7050 1800 50  0001 C CNN "LCSC"
-	1    7050 1800
-	0    1    1    0
-$EndComp
 Wire Wire Line
 	5950 1550 6300 1550
-Wire Wire Line
-	7050 1550 7050 1600
 Connection ~ 5950 1550
-Wire Wire Line
-	6300 1550 6300 1600
 Connection ~ 6300 1550
 Wire Wire Line
 	6300 1550 6650 1550
-Wire Wire Line
-	6650 1550 6650 1600
 Connection ~ 6650 1550
 Wire Wire Line
@@
 	5950 2100 6300 2100
 Wire Wire Line
-	6300 2100 6300 2000
-Wire Wire Line
 	6300 2100 6650 2100
-Wire Wire Line
-	6650 2100 6650 2000
 Connection ~ 6300 2100
 Wire Wire Line
 	6650 2100 7050 2100
-Wire Wire Line
-	7050 2100 7050 2000
 Connection ~ 6650 2100
 Text Label 3850 2200 0    50   ~ 0
@@
 NoConn ~ 1500 3100
 Wire Wire Line
-	3450 2900 3650 2900
-Wire Wire Line
-	3450 2500 3650 2500
-NoConn ~ 3650 2500
-NoConn ~ 3650 2900
-Wire Wire Line
-	3450 3200 3650 3200
-NoConn ~ 3650 3200
-Wire Wire Line
 	4300 3750 9500 3750
 Wire Wire Line
@@
 Wire Wire Line
 	3450 2700 3700 2700
-NoConn ~ 3700 2700
 Text GLabel 9500 2750 0    50   Input ~ 0
 VDD_1
@@
 	1    0    0    -1
 $EndComp
+$Comp
+L Connector:Conn_01x02_Male J3
+U 1 1 60299CC2
+P 4200 2600
+F 0 "J3" H 4172 2482 50  0000 R CNN
+F 1 "Conn_01x02_Male" H 4172 2573 50  0000 R CNN
+F 2 "Connector_PinHeader_2.54mm:PinHeader_1x02_P2.54mm_Vertical" H 4200 2600 50  0001 C CNN
+F 3 "~" H 4200 2600 50  0001 C CNN
+	1    4200 2600
+	-1   0    0    1
+$EndComp
+Wire Wire Line
+	3450 2500 3700 2500
+Wire Wire Line
+	3700 2700 3700 2600
+Wire Wire Line
+	5000 2900 5000 5100
+Wire Wire Line
+	5000 5100 9500 5100
+Wire Wire Line
+	3450 2900 5000 2900
+Wire Wire Line
+	4900 5200 9500 5200
+Wire Wire Line
+	3450 3200 4900 3200
+Wire Wire Line
+	4900 3200 4900 5200
+$Comp
+L Device:R R17
+U 1 1 602A877F
+P 3850 2600
+F 0 "R17" V 3850 2600 50  0000 C CNN
+F 1 "330" V 3950 2600 50  0000 C CNN
+F 2 "Resistor_SMD:R_0805_2012Metric_Pad1.20x1.40mm_HandSolder" V 3780 2600 50  0001 C CNN
+F 3 "~" H 3850 2600 50  0001 C CNN
+F 4 "C17513" H 3850 2600 50  0001 C CNN "LCSC"
+	1    3850 2600
+	0    1    1    0
+$EndComp
+$Comp
+L Device:R R16
+U 1 1 602A8C46
+P 3850 2500
+F 0 "R16" V 3850 2500 50  0000 C CNN
+F 1 "330" V 3750 2500 50  0000 C CNN
+F 2 "Resistor_SMD:R_0805_2012Metric_Pad1.20x1.40mm_HandSolder" V 3780 2500 50  0001 C CNN
+F 3 "~" H 3850 2500 50  0001 C CNN
+F 4 "C17513" H 3850 2500 50  0001 C CNN "LCSC"
+	1    3850 2500
+	0    1    1    0
+$EndComp
+$Comp
+L Connector:Conn_01x02_Male J4
+U 1 1 602E4ED5
+P 6150 1850
+F 0 "J4" H 6122 1732 50  0000 R CNN
+F 1 "Conn_01x02_Male" H 6500 2200 50  0000 R CNN
+F 2 "Connector_PinHeader_2.54mm:PinHeader_1x02_P2.54mm_Vertical" H 6150 1850 50  0001 C CNN
+F 3 "~" H 6150 1850 50  0001 C CNN
+	1    6150 1850
+	-1   0    0    1
+$EndComp
+$Comp
+L Connector:Conn_01x02_Male J8
+U 1 1 602E56CE
+P 6850 1850
+F 0 "J8" H 6822 1732 50  0000 R CNN
+F 1 "Conn_01x02_Male" H 7150 2200 50  0000 R CNN
+F 2 "Connector_PinHeader_2.54mm:PinHeader_1x02_P2.54mm_Vertical" H 6850 1850 50  0001 C CNN
+F 3 "~" H 6850 1850 50  0001 C CNN
+	1    6850 1850
+	-1   0    0    1
+$EndComp
+$Comp
+L Connector:Conn_01x02_Male J9
+U 1 1 602E585C
+P 7250 1850
+F 0 "J9" H 7222 1732 50  0000 R CNN
+F 1 "Conn_01x02_Male" H 7750 1450 50  0000 R CNN
+F 2 "Connector_PinHeader_2.54mm:PinHeader_1x02_P2.54mm_Vertical" H 7250 1850 50  0001 C CNN
+F 3 "~" H 7250 1850 50  0001 C CNN
+	1    7250 1850
+	-1   0    0    1
+$EndComp
+$Comp
+L Connector:Conn_01x02_Male J6
+U 1 1 602E5ED6
+P 6500 1850
+F 0 "J6" H 6472 1732 50  0000 R CNN
+F 1 "Conn_01x02_Male" H 7000 1450 50  0000 R CNN
+F 2 "Connector_PinHeader_2.54mm:PinHeader_1x02_P2.54mm_Vertical" H 6500 1850 50  0001 C CNN
+F 3 "~" H 6500 1850 50  0001 C CNN
+	1    6500 1850
+	-1   0    0    1
+$EndComp
+Wire Wire Line
+	5950 1550 5950 1750
+Wire Wire Line
+	5950 1850 5950 2100
+Wire Wire Line
+	6300 1550 6300 1750
+Wire Wire Line
+	6300 1850 6300 2100
+Wire Wire Line
+	6650 1550 6650 1750
+Wire Wire Line
+	6650 1850 6650 2100
+Wire Wire Line
+	7050 1550 7050 1750
+Wire Wire Line
+	7050 1850 7050 2100
 $EndSCHEMATC

Commit message: Deska 1.1
Parts:
- H1, H2, H3, H4: footprint MountingHole:MountingHole_3mm -> MountingHole:MountingHole_2mm
Changed lines of the file:
@@
 F 0 "H1" H 750 696 50  0000 L CNN
 F 1 "MountingHole" H 750 605 50  0000 L CNN
-F 2 "MountingHole:MountingHole_3mm" H 650 650 50  0001 C CNN
+F 2 "MountingHole:MountingHole_2mm" H 650 650 50  0001 C CNN
 F 3 "~" H 650 650 50  0001 C CNN
 	1    650  650
@@
 F 0 "H2" H 750 896 50  0000 L CNN
 F 1 "MountingHole" H 750 805 50  0000 L CNN
-F 2 "MountingHole:MountingHole_3mm" H 650 850 50  0001 C CNN
+F 2 "MountingHole:MountingHole_2mm" H 650 850 50  0001 C CNN
 F 3 "~" H 650 850 50  0001 C CNN
 	1    650  850
@@
 F 0 "H3" H 750 1096 50  0000 L CNN
 F 1 "MountingHole" H 750 1005 50  0000 L CNN
-F 2 "MountingHole:MountingHole_3mm" H 650 1050 50  0001 C CNN
+F 2 "MountingHole:MountingHole_2mm" H 650 1050 50  0001 C CNN
 F 3 "~" H 650 1050 50  0001 C CNN
 	1    650  1050
@@
 F 0 "H4" H 750 1346 50  0000 L CNN
 F 1 "MountingHole" H 750 1255 50  0000 L CNN
-F 2 "MountingHole:MountingHole_3mm" H 650 1300 50  0001 C CNN
+F 2 "MountingHole:MountingHole_2mm" H 650 1300 50  0001 C CNN
 F 3 "~" H 650 1300 50  0001 C CNN
 	1    650  1300

Commit message: release candidate
Parts:
- added H5, H6, H7: ToolingHole, FinalExamThesis:Tooling_Hole_2, symbol Mechanical:MountingHole
- H1, H2, H3, H4, J3, J4, J6, J8, J9: LCSC (none) -> -
- R16, R17: LCSC C17513 -> C17617
Changed lines of the file:
@@
 F 2 "MountingHole:MountingHole_2mm" H 650 650 50  0001 C CNN
 F 3 "~" H 650 650 50  0001 C CNN
+F 4 "-" H 650 650 50  0001 C CNN "LCSC"
 	1    650  650
 	1    0    0    -1
@@
 F 2 "MountingHole:MountingHole_2mm" H 650 850 50  0001 C CNN
 F 3 "~" H 650 850 50  0001 C CNN
+F 4 "-" H 650 850 50  0001 C CNN "LCSC"
 	1    650  850
 	1    0    0    -1
@@
 F 2 "MountingHole:MountingHole_2mm" H 650 1050 50  0001 C CNN
 F 3 "~" H 650 1050 50  0001 C CNN
+F 4 "-" H 650 1050 50  0001 C CNN "LCSC"
 	1    650  1050
 	1    0    0    -1
@@
 F 2 "MountingHole:MountingHole_2mm" H 650 1300 50  0001 C CNN
 F 3 "~" H 650 1300 50  0001 C CNN
+F 4 "-" H 650 1300 50  0001 C CNN "LCSC"
 	1    650  1300
 	1    0    0    -1
@@
 F 2 "Connector_PinHeader_2.54mm:PinHeader_1x02_P2.54mm_Vertical" H 4200 2600 50  0001 C CNN
 F 3 "~" H 4200 2600 50  0001 C CNN
+F 4 "-" H 4200 2600 50  0001 C CNN "LCSC"
 	1    4200 2600
 	-1   0    0    1
@@
 F 2 "Resistor_SMD:R_0805_2012Metric_Pad1.20x1.40mm_HandSolder" V 3780 2600 50  0001 C CNN
 F 3 "~" H 3850 2600 50  0001 C CNN
-F 4 "C17513" H 3850 2600 50  0001 C CNN "LCSC"
+F 4 "C17617" H 3850 2600 50  0001 C CNN "LCSC"
 	1    3850 2600
 	0    1    1    0
@@
 F 2 "Resistor_SMD:R_0805_2012Metric_Pad1.20x1.40mm_HandSolder" V 3780 2500 50  0001 C CNN
 F 3 "~" H 3850 2500 50  0001 C CNN
-F 4 "C17513" H 3850 2500 50  0001 C CNN "LCSC"
+F 4 "C17617" H 3850 2500 50  0001 C CNN "LCSC"
 	1    3850 2500
 	0    1    1    0
@@
 F 2 "Connector_PinHeader_2.54mm:PinHeader_1x02_P2.54mm_Vertical" H 6150 1850 50  0001 C CNN
 F 3 "~" H 6150 1850 50  0001 C CNN
+F 4 "-" H 6150 1850 50  0001 C CNN "LCSC"
 	1    6150 1850
 	-1   0    0    1
@@
 F 2 "Connector_PinHeader_2.54mm:PinHeader_1x02_P2.54mm_Vertical" H 6850 1850 50  0001 C CNN
 F 3 "~" H 6850 1850 50  0001 C CNN
+F 4 "-" H 6850 1850 50  0001 C CNN "LCSC"
 	1    6850 1850
 	-1   0    0    1
@@
 F 2 "Connector_PinHeader_2.54mm:PinHeader_1x02_P2.54mm_Vertical" H 7250 1850 50  0001 C CNN
 F 3 "~" H 7250 1850 50  0001 C CNN
+F 4 "-" H 7250 1850 50  0001 C CNN "LCSC"
 	1    7250 1850
 	-1   0    0    1
@@
 F 2 "Connector_PinHeader_2.54mm:PinHeader_1x02_P2.54mm_Vertical" H 6500 1850 50  0001 C CNN
 F 3 "~" H 6500 1850 50  0001 C CNN
+F 4 "-" H 6500 1850 50  0001 C CNN "LCSC"
 	1    6500 1850
 	-1   0    0    1
@@
 Wire Wire Line
 	7050 1850 7050 2100
+$Comp
+L Mechanical:MountingHole H5
+U 1 1 602DE9AD
+P 11100 600
+F 0 "H5" H 10900 600 50  0000 L CNN
+F 1 "ToolingHole" H 10650 450 50  0000 L CNN
+F 2 "FinalExamThesis:Tooling_Hole_2" H 11100 600 50  0001 C CNN
+F 3 "~" H 11100 600 50  0001 C CNN
+	1    11100 600
+	1    0    0    -1
+$EndComp
+$Comp
+L Mechanical:MountingHole H6
+U 1 1 602DF5CD
+P 11100 850
+F 0 "H6" H 10900 850 50  0000 L CNN
+F 1 "ToolingHole" H 10650 700 50  0000 L CNN
+F 2 "FinalExamThesis:Tooling_Hole_2" H 11100 850 50  0001 C CNN
+F 3 "~" H 11100 850 50  0001 C CNN
+	1    11100 850
+	1    0    0    -1
+$EndComp
+$Comp
+L Mechanical:MountingHole H7
+U 1 1 602DF825
+P 11100 1100
+F 0 "H7" H 10900 1100 50  0000 L CNN
+F 1 "ToolingHole" H 10650 950 50  0000 L CNN
+F 2 "FinalExamThesis:Tooling_Hole_2" H 11100 1100 50  0001 C CNN
+F 3 "~" H 11100 1100 50  0001 C CNN
+	1    11100 1100
+	1    0    0    -1
+$EndComp
 $EndSCHEMATC
