File: Základní deska II.kicad_pcb (KiCad board)
At the start: 2 copper layers, 34 parts, among them J1 Conn_01x04_Male, J14 Conn_01x04_Male, J2 Conn_01x04_Male, J21 Conn_01x04_Male, J28 Conn_01x04_Male, J5 Conn_01x04_Male, J7 Conn_01x04_Male, Q1 BS250, Q2 2N7000, Q4 BS250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

Commit message: Drobná úprava
Parts:
- moved R3 9.14 mm to (95.5, 139.7)
Changed lines of the file:
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@@
   )
   (module Resistor_SMD:R_0805_2012Metric_Pad1.20x1.40mm_HandSolder (layer F.Cu)
-    (at 98.79 131.17)
+    (at 95.52 139.7)
     (descr "Resistor SMD 0805 (2012 Metric), square (rectangular) end terminal, IPC_7351 nominal with elongated pad for handsoldering. (Body size source: IPC-SM-782 page 72, https://www.pcb-3d.com/wordpress/wp-content/uploads/ipc-sm-782a_amendment_1_and_2.pdf), generated with kicad-footprint-generator")
     (tags "resistor handsolder")
