File: Zakladni_deska_II.sch (KiCad schematic (older format))
At the start: 26 parts, among them J1 Conn_01x04_Male, J2 Conn_01x04_Male, J3 Conn_01x02_Male, J4 Conn_01x02_Male, J5 Conn_01x04_Male, J6 Conn_01x02_Male, J8 Conn_01x02_Male, J9 Conn_01x02_Male, U1 ESP32-DEVKITC-32D

Commit message: Ordered
Parts:
- H1, H2, H3, H4, J1, J2, J3, J4, J5, J6, J8, J9: JLCPCB_IGNORE (none) -> 1
- H5, H6, H7: JLCPCB_IGNORE (none) -> 1; LCSC (none) -> -
- R1, R10, R6, R7, R8, R9: LCSC C17513 -> C17379
- R2: LCSC C17407 -> C17422
- U1: symbol ESP32-DEVKITC-32D:ESP32-DEVKITC-32D -> Zakladni_deska_II-rescue:ESP32-DEVKITC-32D-ESP32-DEVKITC-32D; JLCPCB_IGNORE (none) -> 1
Changed lines of the file:
@@
 F 2 "Resistor_SMD:R_0805_2012Metric_Pad1.20x1.40mm_HandSolder" V 3830 3000 50  0001 C CNN
 F 3 "~" H 3900 3000 50  0001 C CNN
-F 4 "C17513" H 3900 3000 50  0001 C CNN "LCSC"
+F 4 "C17379" H 3900 3000 50  0001 C CNN "LCSC"
 	1    3900 3000
 	0    1    1    0
@@
 $EndComp
 $Comp
-L ESP32-DEVKITC-32D:ESP32-DEVKITC-32D U1
+L Zakladni_deska_II-rescue:ESP32-DEVKITC-32D-ESP32-DEVKITC-32D U1
 U 1 1 601D8F66
 P 2650 2900
@@
 F 5 "Espressif Systems" H 2650 2900 50  0001 L BNN "MANUFACTURER"
 F 6 "-" H 2650 2900 50  0001 C CNN "LCSC"
+F 7 "1" H 2650 2900 50  0001 C CNN "JLCPCB_IGNORE"
 	1    2650 2900
 	1    0    0    -1
@@
 F 2 "Resistor_SMD:R_0805_2012Metric_Pad1.20x1.40mm_HandSolder" V 8880 6250 50  0001 C CNN
 F 3 "~" H 8950 6250 50  0001 C CNN
-F 4 "C17513" H 8950 6250 50  0001 C CNN "LCSC"
+F 4 "C17379" H 8950 6250 50  0001 C CNN "LCSC"
 	1    8950 6250
 	0    1    1    0
@@
 F 2 "Resistor_SMD:R_0805_2012Metric_Pad1.20x1.40mm_HandSolder" V 8880 4650 50  0001 C CNN
 F 3 "~" H 8950 4650 50  0001 C CNN
-F 4 "C17513" H 8950 4650 50  0001 C CNN "LCSC"
+F 4 "C17379" H 8950 4650 50  0001 C CNN "LCSC"
 	1    8950 4650
 	0    1    1    0
@@
 F 2 "Resistor_SMD:R_0805_2012Metric_Pad1.20x1.40mm_HandSolder" V 8880 3850 50  0001 C CNN
 F 3 "~" H 8950 3850 50  0001 C CNN
-F 4 "C17513" H 8950 3850 50  0001 C CNN "LCSC"
+F 4 "C17379" H 8950 3850 50  0001 C CNN "LCSC"
 	1    8950 3850
 	0    1    1    0
@@
 F 2 "Resistor_SMD:R_0805_2012Metric_Pad1.20x1.40mm_HandSolder" V 8880 2950 50  0001 C CNN
 F 3 "~" H 8950 2950 50  0001 C CNN
-F 4 "C17513" H 8950 2950 50  0001 C CNN "LCSC"
+F 4 "C17379" H 8950 2950 50  0001 C CNN "LCSC"
 	1    8950 2950
 	0    1    1    0
@@
 F 3 "~" H 2950 5150 50  0001 C CNN
 F 4 "-" H 2950 5150 50  0001 C CNN "LCSC"
+F 5 "1" H 2950 5150 50  0001 C CNN "JLCPCB_IGNORE"
 	1    2950 5150
 	0    1    1    0
@@
 F 3 "~" H 850 4350 50  0001 C CNN
 F 4 "-" H 850 4350 50  0001 C CNN "LCSC"
+F 5 "1" H 850 4350 50  0001 C CNN "JLCPCB_IGNORE"
 	1    850  4350
 	0    -1   -1   0
@@
 F 3 "~" H 2250 5150 50  0001 C CNN
 F 4 "-" H 2250 5150 50  0001 C CNN "LCSC"
+F 5 "1" H 2250 5150 50  0001 C CNN "JLCPCB_IGNORE"
 	1    2250 5150
 	0    1    1    0
@@
 F 2 "Resistor_SMD:R_0805_2012Metric_Pad1.20x1.40mm_HandSolder" V 5580 1800 50  0001 C CNN
 F 3 "~" H 5650 1800 50  0001 C CNN
-F 4 "C17407" H 5650 1800 50  0001 C CNN "LCSC"
+F 4 "C17422" H 5650 1800 50  0001 C CNN "LCSC"
 	1    5650 1800
 	1    0    0    -1
@@
 F 2 "Resistor_SMD:R_0805_2012Metric_Pad1.20x1.40mm_HandSolder" V 5280 2100 50  0001 C CNN
 F 3 "~" H 5350 2100 50  0001 C CNN
-F 4 "C17513" H 5350 2100 50  0001 C CNN "LCSC"
+F 4 "C17379" H 5350 2100 50  0001 C CNN "LCSC"
 	1    5350 2100
 	0    1    1    0
@@
 	1    0    0    -1
 $EndComp
-Connection ~ 1850 2000
 Text Label 3850 2100 0    50   ~ 0
 Řídí
@@
 F 3 "~" H 650 650 50  0001 C CNN
 F 4 "-" H 650 650 50  0001 C CNN "LCSC"
+F 5 "1" H 650 650 50  0001 C CNN "JLCPCB_IGNORE"
 	1    650  650
 	1    0    0    -1
@@
 F 3 "~" H 650 850 50  0001 C CNN
 F 4 "-" H 650 850 50  0001 C CNN "LCSC"
+F 5 "1" H 650 850 50  0001 C CNN "JLCPCB_IGNORE"
 	1    650  850
 	1    0    0    -1
@@
 F 3 "~" H 650 1050 50  0001 C CNN
 F 4 "-" H 650 1050 50  0001 C CNN "LCSC"
+F 5 "1" H 650 1050 50  0001 C CNN "JLCPCB_IGNORE"
 	1    650  1050
 	1    0    0    -1
@@
 F 3 "~" H 650 1300 50  0001 C CNN
 F 4 "-" H 650 1300 50  0001 C CNN "LCSC"
+F 5 "1" H 650 1300 50  0001 C CNN "JLCPCB_IGNORE"
 	1    650  1300
 	1    0    0    -1
@@
 F 3 "~" H 4200 2600 50  0001 C CNN
 F 4 "-" H 4200 2600 50  0001 C CNN "LCSC"
+F 5 "1" H 4200 2600 50  0001 C CNN "JLCPCB_IGNORE"
 	1    4200 2600
 	-1   0    0    1
@@
 F 3 "~" H 6150 1850 50  0001 C CNN
 F 4 "-" H 6150 1850 50  0001 C CNN "LCSC"
+F 5 "1" H 6150 1850 50  0001 C CNN "JLCPCB_IGNORE"
 	1    6150 1850
 	-1   0    0    1
@@
 F 3 "~" H 6850 1850 50  0001 C CNN
 F 4 "-" H 6850 1850 50  0001 C CNN "LCSC"
+F 5 "1" H 6850 1850 50  0001 C CNN "JLCPCB_IGNORE"
 	1    6850 1850
 	-1   0    0    1
@@
 F 3 "~" H 7250 1850 50  0001 C CNN
 F 4 "-" H 7250 1850 50  0001 C CNN "LCSC"
+F 5 "1" H 7250 1850 50  0001 C CNN "JLCPCB_IGNORE"
 	1    7250 1850
 	-1   0    0    1
@@
 F 3 "~" H 6500 1850 50  0001 C CNN
 F 4 "-" H 6500 1850 50  0001 C CNN "LCSC"
+F 5 "1" H 6500 1850 50  0001 C CNN "JLCPCB_IGNORE"
 	1    6500 1850
 	-1   0    0    1
@@
 F 2 "FinalExamThesis:Tooling_Hole_2" H 11100 600 50  0001 C CNN
 F 3 "~" H 11100 600 50  0001 C CNN
+F 4 "1" H 11100 600 50  0001 C CNN "JLCPCB_IGNORE"
+F 5 "-" H 11100 600 50  0001 C CNN "LCSC"
 	1    11100 600
 	1    0    0    -1
@@
 F 2 "FinalExamThesis:Tooling_Hole_2" H 11100 850 50  0001 C CNN
 F 3 "~" H 11100 850 50  0001 C CNN
+F 4 "1" H 11100 850 50  0001 C CNN "JLCPCB_IGNORE"
+F 5 "-" H 11100 850 50  0001 C CNN "LCSC"
 	1    11100 850
 	1    0    0    -1
@@
 F 2 "FinalExamThesis:Tooling_Hole_2" H 11100 1100 50  0001 C CNN
 F 3 "~" H 11100 1100 50  0001 C CNN
+F 4 "1" H 11100 1100 50  0001 C CNN "JLCPCB_IGNORE"
+F 5 "-" H 11100 1100 50  0001 C CNN "LCSC"
 	1    11100 1100
 	1    0    0    -1
