File: STEP-DIR/Krokovka1.sch (KiCad schematic (older format))
At the start: 6 parts, among them J7 Conn_01x04_Male

Commit message: DIR STEP ven
Parts:
- 2209Br1: symbol Základní-deska-II-rescue:TMC2209BreaoutBoard-Tmc2209BreakoutBoard -> Tmc2209BreakoutBoard:TMC2209BreaoutBoard
Connections:
- net STEP1: now reaches 2209Br1.7 (STEP)
- net DIR1: now reaches 2209Br1.8 (DIR)
- no-connect marks 5 -> 3
Changed lines of the file:
@@
 $Descr A4 11693 8268
 encoding utf-8
-Sheet 5 6
+Sheet 3 6
 Title ""
 Date ""
@@
 Text HLabel 7150 3650 0    50   Input ~ 0
 PDN_1
+Text HLabel 7150 3950 0    50   Input ~ 0
+STEP1
+Text HLabel 7150 4050 0    50   Input ~ 0
+DIR1
 $Comp
 L power:GND #PWR0109
@@
 INDEX_1
 $Comp
-L Základní-deska-II-rescue:TMC2209BreaoutBoard-Tmc2209BreakoutBoard 2209Br1
+L Tmc2209BreakoutBoard:TMC2209BreaoutBoard 2209Br1
 U 1 1 601F591C
 P 7600 3600
@@
 Wire Wire Line
 	7500 2950 7500 2850
-NoConn ~ 7150 3950
-NoConn ~ 7150 4050
 $EndSCHEMATC
