File: STEP-DIR/Krokovka2.sch (KiCad schematic (older format))
At the start: 6 parts, among them J14 Conn_01x04_Male

Commit message: DIR STEP ven
Parts:
- 2209Br2: symbol Základní-deska-II-rescue:TMC2209BreaoutBoard-Tmc2209BreakoutBoard -> Tmc2209BreakoutBoard:TMC2209BreaoutBoard
Connections:
- net STEP2: now reaches 2209Br2.7 (STEP)
- net DIR2: now reaches 2209Br2.8 (DIR)
- no-connect marks 5 -> 3
Changed lines of the file:
@@
 $Descr A4 11693 8268
 encoding utf-8
-Sheet 3 6
+Sheet 4 6
 Title ""
 Date ""
@@
 Text HLabel 6050 4300 0    50   Input ~ 0
 PDN_2
+Text HLabel 6050 4500 0    50   Input ~ 0
+STEP2
+Text HLabel 6050 4600 0    50   Input ~ 0
+DIR2
 $Comp
 L power:GND #PWR?
@@
 $EndComp
 $Comp
-L Základní-deska-II-rescue:TMC2209BreaoutBoard-Tmc2209BreakoutBoard 2209Br2
+L Tmc2209BreakoutBoard:TMC2209BreaoutBoard 2209Br2
 U 1 1 60267626
 P 6500 4150
@@
 	0    1    1    0
 $EndComp
-NoConn ~ 6050 4500
-NoConn ~ 6050 4600
 $EndSCHEMATC
