File: STEP-DIR/Krokovka3.sch (KiCad schematic (older format))
At the start: 6 parts, among them J21 Conn_01x04_Male

Commit message: DIR STEP ven
Parts:
- 2209Br3: symbol Základní-deska-II-rescue:TMC2209BreaoutBoard-Tmc2209BreakoutBoard -> Tmc2209BreakoutBoard:TMC2209BreaoutBoard
Connections:
- net STEP3: now reaches 2209Br3.7 (STEP)
- net DIR3: now reaches 2209Br3.8 (DIR)
- no-connect marks 5 -> 3
Changed lines of the file:
@@
 $Descr A4 11693 8268
 encoding utf-8
-Sheet 6 6
+Sheet 5 6
 Title ""
 Date ""
@@
 Text HLabel 6850 2750 0    50   Input ~ 0
 PDN_3
+Text HLabel 6850 3050 0    50   Input ~ 0
+STEP3
+Text HLabel 6850 3150 0    50   Input ~ 0
+DIR3
 $Comp
 L power:GND #PWR?
@@
 	0    -1   -1   0
 $EndComp
+$Comp
+L Tmc2209BreakoutBoard:TMC2209BreaoutBoard 2209Br3
+U 1 1 602743DD
+P 7300 2700
+F 0 "2209Br3" H 7275 2127 50  0000 C CNN
+F 1 "TMC2209BreaoutBoard" H 7275 2036 50  0000 C CNN
+F 2 "" H 7050 2700 50  0001 C CNN
+F 3 "" H 7050 2700 50  0001 C CNN
+	1    7300 2700
+	1    0    0    -1
+$EndComp
 NoConn ~ 7100 2050
 NoConn ~ 7300 2050
@@
 	0    -1   -1   0
 $EndComp
-$Comp
-L Základní-deska-II-rescue:TMC2209BreaoutBoard-Tmc2209BreakoutBoard 2209Br3
-U 1 1 602743DD
-P 7300 2700
-F 0 "2209Br3" H 7275 2127 50  0000 C CNN
-F 1 "TMC2209BreaoutBoard" H 7275 2036 50  0000 C CNN
-F 2 "" H 7050 2700 50  0001 C CNN
-F 3 "" H 7050 2700 50  0001 C CNN
-	1    7300 2700
-	1    0    0    -1
-$EndComp
-NoConn ~ 6850 3050
-NoConn ~ 6850 3150
 $EndSCHEMATC
