File: STEP-DIR/Napajeni.sch (KiCad schematic (older format))
At the start: 16 parts, among them Q1 BS250, Q2 NTR2101P, Q3 NTR2101P, Q4 BS250, Q5 NTR2101P, SW1 SW_MEC_5G, SW2 SW_MEC_5G

Commit message: DIR STEP ven
Parts:
- PL1, PL2: symbol Základní-deska-II-rescue:Plate-Tmc2209BreakoutBoard -> Tmc2209BreakoutBoard:Plate
Changed lines of the file:
@@
 	4950 2100 4950 2200
 $Comp
-L Základní-deska-II-rescue:Plate-Tmc2209BreakoutBoard PL1
+L Tmc2209BreakoutBoard:Plate PL1
 U 1 1 601FA68F
 P 4250 2100
@@
 $EndComp
 $Comp
-L Základní-deska-II-rescue:Plate-Tmc2209BreakoutBoard PL2
+L Tmc2209BreakoutBoard:Plate PL2
 U 1 1 601FAA1F
 P 4250 2500
