File: STEP-DIR/Základní deska II.sch (KiCad schematic (older format))
At the start: 7 parts, among them J5 Conn_01x04_Male, U1 ESP32-DEVKITC-32D

Commit message: DIR STEP ven
Connections:
- net Krokovka3/STEP3: now reaches U1.10 (IO26)
- net Krokovka 4/DIR4: now reaches U1.11 (IO27)
- net Krokovka 4/STEP4: now reaches U1.12 (IO14)
- net Krokovka1/STEP1: now reaches U1.22 (IO22)
- net Krokovka1/DIR1: now reaches U1.25 (IO21)
- net Krokovka2/STEP2: now reaches U1.29 (IO5)
- net Krokovka2/DIR2: now reaches U1.32 (IO4)
- net Krokovka3/DIR3: now reaches U1.9 (IO25)
Changed lines of the file:
@@
+$EndSheet
+$Sheet
+S 9500 2350 1000 750
+U 601BF914
+F0 "Krokovka1" 50
+F1 "Krokovka1.sch" 50
+F2 "EN1" I L 9500 2500 50
+F3 "PDN_1" I L 9500 2600 50
+F4 "STEP1" I L 9500 2750 50
+F5 "DIR1" I L 9500 2850 50
+F6 "INDEX_1" I L 9500 2950 50
 $EndSheet
 $Sheet
@@
 F2 "EN2" I L 9500 3600 50
 F3 "PDN_2" I L 9500 3750 50
-F4 "INDEX_2" I L 9500 3850 50
+F4 "STEP2" I L 9500 3950 50
+F5 "DIR2" I L 9500 4100 50
+F6 "INDEX_2" I L 9500 3850 50
+$EndSheet
+$Sheet
+S 9500 4600 800  700
+U 60210E5F
+F0 "Krokovka3" 50
+F1 "Krokovka3.sch" 50
+F2 "EN3" I L 9500 4750 50
+F3 "PDN_3" I L 9500 4900 50
+F4 "STEP3" I L 9500 5050 50
+F5 "DIR3" I L 9500 5200 50
+F6 "INDEX_3" I L 9500 4650 50
 $EndSheet
 $Sheet
@@
 F2 "EN4" I L 9500 5750 50
 F3 "PDN_4" I L 9500 5850 50
-F4 "INDEX_4" I L 9500 6250 50
+F4 "STEP4" I L 9500 6000 50
+F5 "DIR4" I L 9500 6150 50
+F6 "INDEX_4" I L 9500 6250 50
 $EndSheet
 $Comp
@@
 Connection ~ 5950 3600
 Connection ~ 5950 4750
+Wire Wire Line
+	9500 2750 5800 2750
+Wire Wire Line
+	9500 2850 5700 2850
+Wire Wire Line
+	9500 3950 5450 3950
+Wire Wire Line
+	9500 4100 5350 4100
 Wire Wire Line
 	3450 3000 3750 3000
@@
 	1050 2500 1850 2500
 Wire Wire Line
+	5800 2750 5800 2200
+Wire Wire Line
+	5800 2200 3450 2200
+Wire Wire Line
+	3450 2500 5700 2500
+Wire Wire Line
+	5700 2500 5700 2850
+Wire Wire Line
 	3450 2700 5650 2700
 Wire Wire Line
@@
 	5550 2800 5550 3850
 Wire Wire Line
+	3450 2900 5450 2900
+Wire Wire Line
+	5450 2900 5450 3950
+Wire Wire Line
 	4300 3000 4300 4900
+Wire Wire Line
+	3450 3200 5350 3200
+Wire Wire Line
+	5350 3200 5350 4100
 NoConn ~ 3450 3800
 NoConn ~ 3450 3600
@@
 Wire Wire Line
 	1500 1150 9500 1150
+Wire Wire Line
+	1850 2800 1350 2800
+Wire Wire Line
+	1350 2800 1350 5200
+Wire Wire Line
+	1350 5200 9500 5200
+Wire Wire Line
+	1450 5050 1450 2900
+Wire Wire Line
+	1450 2900 1850 2900
+Wire Wire Line
+	1450 5050 9500 5050
 NoConn ~ 1850 3700
 NoConn ~ 1850 3600
 NoConn ~ 1850 3500
+Wire Wire Line
+	1650 6000 1650 3100
+Wire Wire Line
+	1650 3100 1850 3100
+Wire Wire Line
+	1650 6000 9500 6000
+Wire Wire Line
+	1550 6150 1550 3000
+Wire Wire Line
+	1550 3000 1850 3000
+Wire Wire Line
+	1550 6150 9500 6150
 Wire Wire Line
 	1850 3400 1750 3400
@@
 Wire Wire Line
 	8800 2950 4550 2950
-$Sheet
-S 9500 2350 1000 750
-U 601BF914
-F0 "Krokovka1" 50
-F1 "Krokovka1.sch" 50
-F2 "EN1" I L 9500 2500 50
-F3 "PDN_1" I L 9500 2600 50
-F4 "INDEX_1" I L 9500 2950 50
-$EndSheet
-$Sheet
-S 9500 4600 800  700
-U 60210E5F
-F0 "Krokovka3" 50
-F1 "Krokovka3.sch" 50
-F2 "EN3" I L 9500 4750 50
-F3 "PDN_3" I L 9500 4900 50
-F4 "INDEX_3" I L 9500 4650 50
-$EndSheet
 $EndSCHEMATC
